File: motherboard/buttons.kicad_sch (KiCad schematic)
At the start: 16 parts, among them J10 DEBUG UART, J11 PWR ON MODE, J7 RTC BATTERY, SW1 PWR, SW2 RESET, SW3 MASK, SW4 RECOVERY

Commit message: wip with pcie2.0 e key, ethernet, buttons and more
Parts:
- added C32: 10uF, symbol Device:C_Small
- added J12: 5V FAN, symbol Connector_Generic:Conn_01x02
- added Q10: 2SK3018W, Package_TO_SOT_SMD:SOT-323_SC-70, symbol Transistor_FET:BSS214NW
- added Q11: Q_PMOS_GSD, symbol Device:Q_PMOS_GSD
- added R45: 10k, symbol Device:R_Small
- added R46: 100R, symbol Device:R_Small
- added R47: 1k, symbol Device:R_Small
- added R48: 470R, symbol Device:R_Small
- added R49: 2.2R, symbol Device:R_Small
Connections:
- net GND: now also C32.2, J12.2 (Pin_2), Q10.2 (S)
- new net: C32.1, J12.1 (Pin_1), R49.2
- new net: Q10.1 (G), R46.2
- new net: Q10.3 (D), R47.2
- new net: Q11.1 (G), R47.1, R48.2
- new net: Q11.3 (D), R49.1
- new net +1V8: R45.1
- new net +5V: Q11.2 (S), R48.1
- new net GPIO1_D3/PWM1_M1: R45.2, R46.1
