File: motherboard/ethernet.kicad_sch (KiCad schematic)
At the start: 13 parts, among them U15 LPJM4938GENL, U16 TPD4EUSB30, U17 TPD4EUSB30

Commit message: synchronizing hierarchical pins
Parts:
- C35, C36: footprint (none) -> Capacitor_SMD:C_0402_1005Metric
Connections:
- net P25G_MDIN0: no longer U16.2 (D1-)
- net P25G_MDIN1: no longer U16.5 (D2-)
- net P25G_MDIN2: no longer U17.2 (D1-)
- net P25G_MDIN3: no longer U17.5 (D2-)
- net P25G_MDIP0: no longer U16.1 (D1+)
- net P25G_MDIP1: no longer U16.4 (D2+)
- net P25G_MDIP2: no longer U17.1 (D1+)
- net P25G_MDIP3: no longer U17.4 (D2+)
- net N2: now reaches CMC9.3, U15.6 (TD3-)
- net N2: now also U16.2 (D1-)
- net P2: now reaches CMC9.4, U15.5 (TD3+)
- net P2: now also U16.1 (D1+)
- net N1: now reaches CMC8.3, U15.4 (TD2-)
- net N1: now also U17.5 (D2-)
- net P1: now reaches CMC8.4, U15.3 (TD2+)
- net P1: now also U17.4 (D2+)
- net P0: now reaches CMC7.4, U15.1 (TD1+)
- net P0: now also U17.1 (D1+)
- net N0: now reaches CMC7.3, U15.2 (TD1-)
- net N0: now also U17.2 (D1-)
- net P3: now reaches CMC10.4, U15.7 (TD4+)
- net P3: now also U16.4 (D2+)
- net N3: now reaches CMC10.3, U15.8 (TD4-)
- net N3: now also U16.5 (D2-)
Changed lines of the file:
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@@
+		)
+	)
+	(label "N0"
+		(at 90.17 119.38 180)
+		(fields_autoplaced yes)
+		(effects
+			(font
+				(size 1.27 1.27)
+			)
+			(justify right bottom)
+		)
+	)
+	(label "P3"
+		(at 171.45 114.3 0)
+		(fields_autoplaced yes)
+		(effects
+			(font
+				(size 1.27 1.27)
+			)
+			(justify left bottom)
+		)
+	)
+	(label "P1"
+		(at 111.76 77.47 0)
+		(fields_autoplaced yes)
+		(effects
+			(font
+				(size 1.27 1.27)
+			)
+			(justify left bottom)
+		)
+	)
+	(label "N3"
+		(at 171.45 119.38 0)
+		(fields_autoplaced yes)
+		(effects
+			(font
+				(size 1.27 1.27)
+			)
+			(justify left bottom)
+		)
+	)
+	(label "P2"
+		(at 111.76 82.55 0)
+		(fields_autoplaced yes)
+		(effects
+			(font
+				(size 1.27 1.27)
+			)
+			(justify left bottom)
+		)
+	)
+	(label "P1"
+		(at 115.57 114.3 0)
+		(fields_autoplaced yes)
+		(effects
+			(font
+				(size 1.27 1.27)
+			)
+			(justify left bottom)
+		)
+	)
+	(label "P0"
+		(at 111.76 72.39 0)
+		(fields_autoplaced yes)
+		(effects
+			(font
+				(size 1.27 1.27)
+			)
+			(justify left bottom)
+		)
+	)
+	(label "P0"
+		(at 90.17 114.3 180)
+		(fields_autoplaced yes)
+		(effects
+			(font
+				(size 1.27 1.27)
+			)
+			(justify right bottom)
+		)
+	)
+	(label "P3"
+		(at 111.76 87.63 0)
+		(fields_autoplaced yes)
+		(effects
+			(font
+				(size 1.27 1.27)
+			)
+			(justify left bottom)
+		)
+	)
+	(label "N0"
+		(at 111.76 74.93 0)
+		(fields_autoplaced yes)
+		(effects
+			(font
+				(size 1.27 1.27)
+			)
+			(justify left bottom)
+		)
+	)
+	(label "N2"
+		(at 111.76 85.09 0)
+		(fields_autoplaced yes)
+		(effects
+			(font
+				(size 1.27 1.27)
+			)
+			(justify left bottom)
+		)
+	)
+	(label "N1"
+		(at 115.57 119.38 0)
+		(fields_autoplaced yes)
+		(effects
+			(font
+				(size 1.27 1.27)
+			)
+			(justify left bottom)
+		)
+	)
+	(label "N3"
+		(at 111.76 90.17 0)
+		(fields_autoplaced yes)
+		(effects
+			(font
+				(size 1.27 1.27)
+			)
+			(justify left bottom)
+		)
+	)
+	(label "N2"
+		(at 146.05 119.38 180)
+		(fields_autoplaced yes)
+		(effects
+			(font
+				(size 1.27 1.27)
+			)
+			(justify right bottom)
+		)
+	)
+	(label "N1"
+		(at 111.76 80.01 0)
+		(fields_autoplaced yes)
+		(effects
+			(font
+				(size 1.27 1.27)
+			)
+			(justify left bottom)
+		)
+	)
+	(label "P2"
+		(at 146.05 114.3 180)
+		(fields_autoplaced yes)
+		(effects
+			(font
+				(size 1.27 1.27)
+			)
+			(justify right bottom)
 		)
 	)
@@
 		)
 	)
-	(hierarchical_label "P25G_MDIP2"
-		(shape input)
-		(at 90.17 114.3 180)
-		(fields_autoplaced yes)
-		(effects
-			(font
-				(size 1.27 1.27)
-			)
-			(justify right)
-		)
-	)
-	(hierarchical_label "P25G_MDIN3"
-		(shape input)
-		(at 115.57 119.38 0)
-		(fields_autoplaced yes)
-		(effects
-			(font
-				(size 1.27 1.27)
-			)
-			(justify left)
-		)
-	)
 	(hierarchical_label "P25G_MDIN2"
 		(shape input)
@@
 		)
 	)
-	(hierarchical_label "P25G_MDIP3"
-		(shape input)
-		(at 115.57 114.3 0)
-		(fields_autoplaced yes)
-		(effects
-			(font
-				(size 1.27 1.27)
-			)
-			(justify left)
-		)
-	)
 	(hierarchical_label "P25G_MDIP2"
 		(shape input)
@@
 		)
 	)
-	(hierarchical_label "P25G_MDIP1"
-		(shape input)
-		(at 171.45 114.3 0)
-		(fields_autoplaced yes)
-		(effects
-			(font
-				(size 1.27 1.27)
-			)
-			(justify left)
-		)
-	)
 	(hierarchical_label "P25G_MDIP3"
 		(shape input)
@@
 		)
 	)
-	(hierarchical_label "P25G_MDIN1"
-		(shape input)
-		(at 171.45 119.38 0)
-		(fields_autoplaced yes)
-		(effects
-			(font
-				(size 1.27 1.27)
-			)
-			(justify left)
-		)
-	)
-	(hierarchical_label "P25G_MDIN2"
-		(shape input)
-		(at 90.17 119.38 180)
-		(fields_autoplaced yes)
-		(effects
-			(font
-				(size 1.27 1.27)
-			)
-			(justify right)
-		)
-	)
-	(hierarchical_label "P25G_MDIN0"
-		(shape input)
-		(at 146.05 119.38 180)
-		(fields_autoplaced yes)
-		(effects
-			(font
-				(size 1.27 1.27)
-			)
-			(justify right)
-		)
-	)
 	(hierarchical_label "P25G_MDIN0"
 		(shape input)
@@
 		(shape input)
 		(at 100.33 80.01 180)
-		(fields_autoplaced yes)
-		(effects
-			(font
-				(size 1.27 1.27)
-			)
-			(justify right)
-		)
-	)
-	(hierarchical_label "P25G_MDIP0"
-		(shape input)
-		(at 146.05 114.3 180)
 		(fields_autoplaced yes)
 		(effects
@@
 			)
 		)
-		(property "Footprint" ""
+		(property "Footprint" "Capacitor_SMD:C_0402_1005Metric"
 			(at 144.78 85.09 0)
 			(effects
@@
 			)
 		)
-		(property "Footprint" ""
+		(property "Footprint" "Capacitor_SMD:C_0402_1005Metric"
 			(at 149.86 85.09 0)
 			(effects
