File: motherboard/ethernet.kicad_sch (KiCad schematic)
At the start: 14 parts, among them J23 L829-1J1T-JM, U16 TPD4E02B04, U17 TPD4E02B04

Commit message: removed 2.5G ethernet
Parts:
- removed C94, C95, C96, C97: 100nF/100V, Capacitor_SMD:C_0805_2012Metric, symbol Device:C_Small
- removed CMC10, CMC7, CMC8, CMC9: ACM2012, ACM2012:FIL_ACM2012-900-2P-T001, symbol library:ACM2012_Common_Mode_Choke
- removed J23: L829-1J1T-JM, Ethernet:BEL_L829-1J1T-JM, symbol Ethernet:L829-1J1T-JM
- removed R53, R54: 1k, Resistor_SMD:R_0402_1005Metric, symbol Device:R_Small
- removed TP1: RJ45 ORANGE LED, TestPoint:TestPoint_Pad_D2.0mm, symbol Connector:TestPoint_Alt
- removed U16, U17: TPD4E02B04, Package_SON:USON-10_2.5x1.0mm_P0.5mm, symbol Power_Protection:TPD4EUSB30
