File: motherboard/USBC1.kicad_sch (KiCad schematic)
At the start: 34 parts, among them J1 USB_C_Receptacle, U10 TPD4EUSB30, U6 SY6280AAC, U7 FUSB302BMPX, U8 TPD4EUSB30, U9 TPD4EUSB30

Commit message: cost optimizations for jlc
Parts:
- R12, R13: footprint Resistor_SMD:R_0402_1005Metric -> Resistor_SMD:R_0603_1608Metric
Changed lines of the file:
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@@
 			)
 		)
-		(property "Footprint" "Resistor_SMD:R_0402_1005Metric"
+		(property "Footprint" "Resistor_SMD:R_0603_1608Metric"
 			(at 91.44 52.07 0)
 			(effects
@@
 			)
 		)
-		(property "Description" "Unpolarized capacitor, small symbol"
+		(property "Description" "C527590"
 			(at 125.73 40.64 0)
 			(effects
@@
 			)
 		)
-		(property "Footprint" "Resistor_SMD:R_0402_1005Metric"
+		(property "Footprint" "Resistor_SMD:R_0603_1608Metric"
 			(at 91.44 54.61 0)
 			(effects
@@
 			)
 		)
-		(property "Description" "Unpolarized capacitor, small symbol"
+		(property "Description" "C527590"
 			(at 180.34 77.47 0)
 			(effects
@@
 			)
 		)
-		(property "Description" "Unpolarized capacitor, small symbol"
+		(property "Description" "C527590"
 			(at 152.4 77.47 0)
 			(effects
@@
 			)
 		)
-		(property "Description" "Unpolarized capacitor, small symbol"
+		(property "Description" "C527590"
 			(at 120.65 40.64 0)
 			(effects
@@
 			)
 		)
-		(property "Description" "Unpolarized capacitor, small symbol"
+		(property "Description" "C527590"
 			(at 132.08 109.22 0)
 			(effects

Commit message: component placement of I/O
Connections:
- net at J1.A7 (D-), J1.B7 (D-): now also CMC2.2; no longer CMC2.1
- net at J1.A6 (D+), J1.B6 (D+): now also CMC2.1; no longer CMC2.2
- net at CMC2.3: now also R12.1; no longer R13.1
- net at CMC2.4: now also R13.1; no longer R12.1
Changed lines of the file:
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@@
 			)
 		)
-		(property "Description" "C527590"
+		(property "Description" "Unpolarized capacitor, small symbol"
 			(at 125.73 40.64 0)
 			(effects
@@
 			)
 		)
-		(property "Description" "C527590"
+		(property "Description" "Unpolarized capacitor, small symbol"
 			(at 180.34 77.47 0)
 			(effects
@@
 			)
 		)
-		(property "Description" "C527590"
+		(property "Description" "Unpolarized capacitor, small symbol"
 			(at 152.4 77.47 0)
 			(effects
@@
 			)
 		)
-		(property "Description" "C527590"
+		(property "Description" "Unpolarized capacitor, small symbol"
 			(at 120.65 40.64 0)
 			(effects
@@
 			)
 		)
-		(property "Description" "C527590"
+		(property "Description" "Unpolarized capacitor, small symbol"
 			(at 132.08 109.22 0)
 			(effects

Commit message: placement roughly halfway done
Parts:
- removed C17, C18, C21, C22: 100nF, Capacitor_SMD:C_0402_1005Metric, symbol Device:C_Small
- removed D2: LESD8D5.0CB1T5G, Diode_SMD:D_SOD-882, symbol Device:D_TVS_Small_Filled
- removed R12, R13: 2.2R, Resistor_SMD:R_0603_1608Metric, symbol Device:R_Small
- removed R14, R15, R16, R17: 0R, Resistor_SMD:R_0402_1005Metric, symbol Device:R_Small
- added U29: TVS2200DRV, Package_SON:WSON-6-1EP_2x2mm_P0.65mm_EP1x1.6mm, symbol Power_Protection:TVS2200DRV
- C14: value 100nF -> 100nF (+25V)
- C15, C16: value 10uF -> 10uF (C913517); footprint Capacitor_SMD:C_0402_1005Metric -> Capacitor_SMD:C_0603_1608Metric
- U10, U8, U9: value TPD4EUSB30 -> TPD4E02B04
Connections:
- net D+: now also CMC2.4
- net D-: now also CMC2.3
- net GND: now also U29.4 (IN), U29.5 (IN), U29.6 (IN)
- net RX1+: now also J1.B11 (RX1+)
- net RX1-: now also J1.B10 (RX1-)
- net RX2+: now also J1.A11 (RX2+)
- net RX2-: now also J1.A10 (RX2-)
- net TX1+: now also J1.A2 (TX1+)
- net TX1-: now also J1.A3 (TX1-)
- net TX2+: now also J1.B2 (TX2+)
- net TX2-: now also J1.B3 (TX2-)
- net VBUS: now also U29.1 (GND), U29.2 (GND), U29.3 (GND), U29.7 (GND)
