File: motherboard/motherboard.kicad_pcb (KiCad board)
At the start: 0 parts

Commit message: linked all footprints
Parts:
- added C1: 100nF, Capacitor_SMD:C_0402_1005Metric, F.Cu at (126.8, 142.3)
- added C10: 10uF, Capacitor_SMD:C_0402_1005Metric, F.Cu at (129.6, 150.2)
- added C11: 10uF, Capacitor_SMD:C_0402_1005Metric, F.Cu at (132.5, 142.3)
- added C12: 10uF, Capacitor_SMD:C_0402_1005Metric, F.Cu at (132.5, 144.3)
- added C13: 10uF, Capacitor_SMD:C_0402_1005Metric, F.Cu at (132.5, 146.2)
- added C14: 100nF, Capacitor_SMD:C_0402_1005Metric, F.Cu at (126.8, 120.8)
- added C15: 10uF, Capacitor_SMD:C_0402_1005Metric, F.Cu at (126.8, 122.8)
- added C16: 10uF, Capacitor_SMD:C_0402_1005Metric, F.Cu at (126.8, 124.8)
- added C17: 100nF, Capacitor_SMD:C_0402_1005Metric, F.Cu at (126.8, 126.8)
- added C18: 100nF, Capacitor_SMD:C_0402_1005Metric, F.Cu at (126.8, 128.7)
- added C19: 10uF, Capacitor_SMD:C_0402_1005Metric, F.Cu at (129.6, 120.8)
- added C2: 220pF, Capacitor_SMD:C_0402_1005Metric, F.Cu at (126.8, 144.3)
- added C20: 10uF, Capacitor_SMD:C_0402_1005Metric, F.Cu at (129.6, 122.8)
- added C21: 100nF, Capacitor_SMD:C_0402_1005Metric, F.Cu at (129.6, 124.8)
- added C22: 100nF, Capacitor_SMD:C_0402_1005Metric, F.Cu at (129.6, 126.8)
- added C23: 100nF, Capacitor_SMD:C_0402_1005Metric, F.Cu at (129.6, 128.7)
- added C24: 10uF, Capacitor_SMD:C_0402_1005Metric, F.Cu at (132.5, 120.8)
- added C25: 220pF, Capacitor_SMD:C_0402_1005Metric, F.Cu at (132.5, 122.8)
- added C26: 220pF, Capacitor_SMD:C_0402_1005Metric, F.Cu at (132.5, 124.8)
- added C27: 1uF, Capacitor_SMD:C_0402_1005Metric, F.Cu at (143.5, 111.2)
- added C28: 1nF, Capacitor_SMD:C_0402_1005Metric, F.Cu at (153.9, 76.9)
- added C29: 1nF, Capacitor_SMD:C_0402_1005Metric, F.Cu at (153.9, 78.8)
- added C3: 220pF, Capacitor_SMD:C_0402_1005Metric, F.Cu at (126.8, 146.2)
- added C30: 1nF, Capacitor_SMD:C_0402_1005Metric, F.Cu at (153.9, 80.8)
- added C31: 1nF, Capacitor_SMD:C_0402_1005Metric, F.Cu at (153.9, 82.8)
- added C32: 10uF, Capacitor_SMD:C_0402_1005Metric, F.Cu at (153.9, 84.8)
- added C33: 100nF, Capacitor_SMD:C_0402_1005Metric, F.Cu at (173.9, 126.4)
- added C34: 100nF, Capacitor_SMD:C_0402_1005Metric, F.Cu at (173.9, 128.4)
- added C35: 100nF, Capacitor_SMD:C_0402_1005Metric, F.Cu at (166.1, 126.5)
- added C36: 100nF, Capacitor_SMD:C_0402_1005Metric, F.Cu at (166.1, 128.5)
- added C37: 220nF, Capacitor_SMD:C_0402_1005Metric, F.Cu at (96.5, 122.6)
- added C38: 220nF, Capacitor_SMD:C_0402_1005Metric, F.Cu at (96.5, 124.5)
- added C39: 220nF, Capacitor_SMD:C_0402_1005Metric, F.Cu at (96.5, 126.5)
- added C4: 100nF, Capacitor_SMD:C_0402_1005Metric, F.Cu at (126.8, 148.2)
- added C40: 220nF, Capacitor_SMD:C_0402_1005Metric, F.Cu at (96.5, 128.5)
- added C41: 220nF, Capacitor_SMD:C_0402_1005Metric, F.Cu at (96.5, 130.4)
- added C42: 220nF, Capacitor_SMD:C_0402_1005Metric, F.Cu at (96.5, 132.4)
- added C43: 220nF, Capacitor_SMD:C_0402_1005Metric, F.Cu at (99.4, 122.6)
- added C44: 220nF, Capacitor_SMD:C_0402_1005Metric, F.Cu at (99.4, 124.5)
- added C45: 22uF, Capacitor_SMD:C_0402_1005Metric, F.Cu at (99.4, 126.5)
- added C46: 22uF, Capacitor_SMD:C_0402_1005Metric, F.Cu at (99.4, 128.5)
- added C47: 1uF, Capacitor_SMD:C_0402_1005Metric, F.Cu at (99.4, 130.4)
- added C48: 0.1uF, Capacitor_SMD:C_0402_1005Metric, F.Cu at (99.4, 132.4)
- added C49: 100nF, Capacitor_SMD:C_0402_1005Metric, F.Cu at (102.2, 122.6)
- added C5: 100nF, Capacitor_SMD:C_0402_1005Metric, F.Cu at (126.8, 150.2)
- added C50: 10uF, Capacitor_SMD:C_1206_3216Metric, F.Cu at (86.2, 135.2)
- added C51: 1uF, Capacitor_SMD:C_1206_3216Metric, F.Cu at (86.2, 138.5)
- added C52: 22uF, Capacitor_SMD:C_0603_1608Metric, F.Cu at (91.1, 134.8)
- added C53: 8.2nF, Capacitor_SMD:C_0603_1608Metric, F.Cu at (91.1, 137.3)
- added C54: 1nF, Capacitor_SMD:C_0402_1005Metric, F.Cu at (102.2, 124.5)
- added C55: 10pF, Capacitor_SMD:C_0402_1005Metric, F.Cu at (102.2, 126.5)
- added C56: 100nF, Capacitor_SMD:C_0402_1005Metric, F.Cu at (102.2, 128.5)
- added C57: 1uF, Capacitor_SMD:C_0402_1005Metric, F.Cu at (102.2, 130.4)
- added C58: 15pF, Capacitor_SMD:C_0402_1005Metric, F.Cu at (102.2, 132.4)
- added C59: 15pF, Capacitor_SMD:C_0402_1005Metric, F.Cu at (105.1, 122.6)
- added C6: 100nF, Capacitor_SMD:C_0402_1005Metric, F.Cu at (129.6, 142.3)
- added C60: 1uF, Capacitor_SMD:C_0402_1005Metric, F.Cu at (105.1, 124.5)
- added C61: 100nF, Capacitor_SMD:C_0402_1005Metric, F.Cu at (105.1, 126.5)
- added C62: 1uF, Capacitor_SMD:C_0402_1005Metric, F.Cu at (105.1, 128.5)
- added C63: 1uF, Capacitor_SMD:C_0402_1005Metric, F.Cu at (105.1, 130.4)
- added C64: 15pF, Capacitor_SMD:C_0402_1005Metric, F.Cu at (183.4, 53.0)
- added C65: 15pF, Capacitor_SMD:C_0402_1005Metric, F.Cu at (183.4, 55.0)
- added C66: 0.1uF, Capacitor_SMD:C_0402_1005Metric, F.Cu at (183.4, 56.9)
- added C67: 10uF, Capacitor_SMD:C_0402_1005Metric, F.Cu at (183.4, 58.9)
- added C68: 1uF, Capacitor_SMD:C_0402_1005Metric, F.Cu at (183.4, 60.9)
- added C7: 100nF, Capacitor_SMD:C_0402_1005Metric, F.Cu at (129.6, 144.3)
- added C8: 100nF, Capacitor_SMD:C_0402_1005Metric, F.Cu at (129.6, 146.2)
- added C9: 10uF, Capacitor_SMD:C_0402_1005Metric, F.Cu at (129.6, 148.2)
- added CMC1: ACM2012, ACM2012:FIL_ACM2012-900-2P-T001, F.Cu at (136.2, 142.6)
- added CMC10: ACM2012, ACM2012:FIL_ACM2012-900-2P-T001, F.Cu at (164.1, 124.3)
- added CMC2: ACM2012, ACM2012:FIL_ACM2012-900-2P-T001, F.Cu at (136.2, 121.1)
- added CMC3: ACM2012, ACM2012:FIL_ACM2012-900-2P-T001, F.Cu at (167.7, 89.1)
- added CMC4: ACM2012, ACM2012:FIL_ACM2012-900-2P-T001, F.Cu at (167.7, 91.7)
- added CMC5: ACM2012, ACM2012:FIL_ACM2012-900-2P-T001, F.Cu at (167.7, 94.2)
- added CMC6: ACM2012, ACM2012:FIL_ACM2012-900-2P-T001, F.Cu at (167.7, 96.8)
- added CMC7: ACM2012, ACM2012:FIL_ACM2012-900-2P-T001, F.Cu at (164.1, 116.6)
- added CMC8: ACM2012, ACM2012:FIL_ACM2012-900-2P-T001, F.Cu at (164.1, 119.2)
- added CMC9: ACM2012, ACM2012:FIL_ACM2012-900-2P-T001, F.Cu at (164.1, 121.7)
- added D1: LESD8D5.0CB1T5G, Diode_SMD:D_SOD-882, F.Cu at (135.3, 145.0)
- added D2: LESD8D5.0CB1T5G, Diode_SMD:D_SOD-882, F.Cu at (135.3, 123.6)
- added D3: LRB521S-30T1G, Diode_SMD:D_SOD-523, F.Cu at (152.5, 111.7)
- added D4: LRB521S-30T1G, Diode_SMD:D_SOD-523, F.Cu at (168.5, 83.7)
- added D5: SS54, Diode_SMD:D_SMA, F.Cu at (110.6, 112.6)
- added IC1: PI6C557-05BLE, SOP65P640X120-20N:SOP65P640X120-20N, F.Cu at (99.5, 137.5)
- added J1: USB_C_Receptacle, USB-C:USB-C-SMD_TYPE-C-24P-QT, F.Cu at (122.0, 114.0)
- added J10: DEBUG UART, Connector_PinHeader_2.54mm:PinHeader_1x03_P2.54mm_Vertical, F.Cu at (150.2, 78.2)
- added J12: 5V FAN, Connector_PinHeader_2.54mm:PinHeader_1x02_P2.54mm_Vertical, F.Cu at (157.7, 78.2)
- added J13: Bus_M.2_Socket_E, WIRELESS_E_KEY:CONN-SMD_APCI0147-P001A, F.Cu at (181.1, 120.4)
- added J14: Micro_SD_Card_Det1, microSD_Card:TF-SMD_TF-CARD-H1.8, F.Cu at (180.9, 94.2)
- added J15: Bus_M.2_Socket_M, NVME_M_KEY:CONN-SMD_AS0BC21-S30BM-7H, F.Cu at (95.0, 116.6)
- added J16: USB, 6P_05mm_FPC:FPC-SMD_6P-P0.50_XUNPU_FPC-05F-6PH20, F.Cu at (177.5, 54.4)
- added J17: USB, 6P_05mm_FPC:FPC-SMD_6P-P0.50_XUNPU_FPC-05F-6PH20, F.Cu at (177.5, 61.4)
- added J18: USB, 6P_05mm_FPC:FPC-SMD_6P-P0.50_XUNPU_FPC-05F-6PH20, F.Cu at (177.5, 68.3)
- added J19: USB, 6P_05mm_FPC:FPC-SMD_6P-P0.50_XUNPU_FPC-05F-6PH20, F.Cu at (177.5, 75.3)
- added J2: 20455-040E-76 OLED IPEX, eDP_Connector:IPEX_20455-040E-76, F.Cu at (156.9, 45.9)
- added J20: CM3588 Hirose Connector, Library:CM3588, F.Cu at (111.5, 72.3)
- added J5: USB_C_Receptacle, USB-C:USB-C-SMD_TYPE-C-24P-QT, F.Cu at (122.0, 135.4)
- added J7: RTC BATTERY, Connector_RJ:RJ45_Wuerth_7499111446_Horizontal, F.Cu at (146.2, 55.1)
- added J8: HDMI_A, Connector_Video:HDMI_A_Molex_208658-1001_Horizontal, F.Cu at (147.6, 96.9)
- added L1: 3.3uH, Inductor_SMD:L_Vishay_IHLP-1616, F.Cu at (110.2, 124.4)
- added Q1: 2SK3018W, Package_TO_SOT_SMD:SOT-323_SC-70, F.Cu at (158.9, 103.8)
- added Q10: 2SK3018W, Package_TO_SOT_SMD:SOT-323_SC-70, F.Cu at (168.9, 80.6)
- added Q11: AO3415A, Package_TO_SOT_SMD:SOT-23, F.Cu at (164.2, 81.0)
- added Q2: 2SK3018W, Package_TO_SOT_SMD:SOT-323_SC-70, F.Cu at (158.9, 107.7)
- added Q3: L2N7002WT1G, Package_TO_SOT_SMD:SOT-323_SC-70, F.Cu at (158.9, 111.5)
- added Q4: 2SK3018W, Package_TO_SOT_SMD:SOT-323_SC-70, F.Cu at (163.4, 103.8)
- added Q5: 2SK3018W, Package_TO_SOT_SMD:SOT-323_SC-70, F.Cu at (163.4, 107.7)
- added Q6: WNM6002-3/TR, Package_TO_SOT_SMD:SOT-323_SC-70, F.Cu at (163.4, 111.5)
- added Q7: WNM6002-3/TR, Package_TO_SOT_SMD:SOT-323_SC-70, F.Cu at (167.8, 103.8)
- added Q8: WNM6002-3/TR, Package_TO_SOT_SMD:SOT-323_SC-70, F.Cu at (167.8, 107.7)
- added Q9: WNM6002-3/TR, Package_TO_SOT_SMD:SOT-323_SC-70, F.Cu at (167.8, 111.5)
- added R1: 1M, Resistor_SMD:R_0402_1005Metric, F.Cu at (118.1, 142.3)
- added R10: 6.8k, Resistor_SMD:R_0402_1005Metric, F.Cu at (121.0, 150.3)
- added R11: 100k, Resistor_SMD:R_0402_1005Metric, F.Cu at (123.9, 142.3)
- added R12: 2.2R, Resistor_SMD:R_0402_1005Metric, F.Cu at (118.1, 120.9)
- added R13: 2.2R, Resistor_SMD:R_0402_1005Metric, F.Cu at (118.1, 122.8)
- added R14: 0R, Resistor_SMD:R_0402_1005Metric, F.Cu at (118.1, 124.8)
- added R15: 0R, Resistor_SMD:R_0402_1005Metric, F.Cu at (118.1, 126.8)
- added R16: 0R, Resistor_SMD:R_0402_1005Metric, F.Cu at (118.1, 128.8)
- added R17: 0R, Resistor_SMD:R_0402_1005Metric, F.Cu at (121.0, 120.9)
- added R18: 0R, Resistor_SMD:R_0402_1005Metric, F.Cu at (121.0, 122.8)
- added R19: 100k, Resistor_SMD:R_0402_1005Metric, F.Cu at (121.0, 124.8)
- added R2: 2.2k, Resistor_SMD:R_0402_1005Metric, F.Cu at (118.1, 144.3)
- added R20: 1M, Resistor_SMD:R_0402_1005Metric, F.Cu at (121.0, 126.8)
- added R21: 2.2k, Resistor_SMD:R_0402_1005Metric, F.Cu at (121.0, 128.8)
- added R22: 2.2k, Resistor_SMD:R_0402_1005Metric, F.Cu at (123.9, 120.9)
- added R23: 27k, Resistor_SMD:R_0402_1005Metric, F.Cu at (158.2, 88.8)
- added R24: 1.8k, Resistor_SMD:R_0402_1005Metric, F.Cu at (158.2, 90.8)
- added R25: 10k, Resistor_SMD:R_0402_1005Metric, F.Cu at (158.2, 92.8)
- added R26: 1.8k, Resistor_SMD:R_0402_1005Metric, F.Cu at (158.2, 94.8)
- added R27: 10k, Resistor_SMD:R_0402_1005Metric, F.Cu at (158.2, 96.8)
- added R28: 1k, Resistor_SMD:R_0402_1005Metric, F.Cu at (158.2, 98.8)
- added R29: 1.8k, Resistor_SMD:R_0402_1005Metric, F.Cu at (158.2, 100.8)
- added R3: 2.2k, Resistor_SMD:R_0402_1005Metric, F.Cu at (118.1, 146.3)
- added R30: 47k, Resistor_SMD:R_0402_1005Metric, F.Cu at (161.1, 88.8)
- added R31: 10k, Resistor_SMD:R_0402_1005Metric, F.Cu at (161.1, 90.8)
- added R32: 10k, Resistor_SMD:R_0402_1005Metric, F.Cu at (161.1, 92.8)
- added R33: 499R, Resistor_SMD:R_0402_1005Metric, F.Cu at (161.1, 94.8)
- added R34: 499R, Resistor_SMD:R_0402_1005Metric, F.Cu at (161.1, 96.8)
- added R35: 499R, Resistor_SMD:R_0402_1005Metric, F.Cu at (161.1, 98.8)
- added R36: 499R, Resistor_SMD:R_0402_1005Metric, F.Cu at (161.1, 100.8)
- added R37: 499R, Resistor_SMD:R_0402_1005Metric, F.Cu at (164.0, 88.8)
- added R38: 499R, Resistor_SMD:R_0402_1005Metric, F.Cu at (164.0, 90.8)
- added R39: 499R, Resistor_SMD:R_0402_1005Metric, F.Cu at (164.0, 92.8)
- added R4: 0R, Resistor_SMD:R_0402_1005Metric, F.Cu at (118.1, 148.3)
- added R40: 499R, Resistor_SMD:R_0402_1005Metric, F.Cu at (164.0, 94.8)
- added R41: 100R, Resistor_SMD:R_0402_1005Metric, F.Cu at (143.5, 76.9)
- added R42: 100R, Resistor_SMD:R_0402_1005Metric, F.Cu at (143.5, 78.9)
- added R43: 100R, Resistor_SMD:R_0402_1005Metric, F.Cu at (143.5, 80.9)
- added R44: 100R, Resistor_SMD:R_0402_1005Metric, F.Cu at (143.5, 82.9)
- added R45: 10k, Resistor_SMD:R_0402_1005Metric, F.Cu at (143.5, 84.8)
- added R46: 100R, Resistor_SMD:R_0402_1005Metric, F.Cu at (146.4, 76.9)
- added R47: 1k, Resistor_SMD:R_0402_1005Metric, F.Cu at (146.4, 78.9)
- added R48: 470R, Resistor_SMD:R_0402_1005Metric, F.Cu at (146.4, 80.9)
- added R49: 2.2R, Resistor_SMD:R_0402_1005Metric, F.Cu at (146.4, 82.9)
- added R5: 0R, Resistor_SMD:R_0402_1005Metric, F.Cu at (118.1, 150.3)
- added R50: 0R, Resistor_SMD:R_0402_1005Metric, F.Cu at (171.0, 126.4)
- added R51: 0R, Resistor_SMD:R_0402_1005Metric, F.Cu at (171.0, 128.4)
- added R52: 2.2k, Resistor_SMD:R_0402_1005Metric, F.Cu at (171.0, 130.4)
- added R53: 560R, Resistor_SMD:R_0402_1005Metric, F.Cu at (163.2, 126.5)
- added R54: 560R, Resistor_SMD:R_0402_1005Metric, F.Cu at (163.2, 128.5)
- added R55: 560R, Resistor_SMD:R_0402_1005Metric, F.Cu at (163.2, 130.5)
- added R56: 560R, Resistor_SMD:R_0402_1005Metric, F.Cu at (163.2, 132.5)
- added R57: 33R, Resistor_SMD:R_0402_1005Metric, F.Cu at (191.2, 88.8)
- added R58: 33R, Resistor_SMD:R_0402_1005Metric, F.Cu at (191.2, 90.8)
- added R59: 33R, Resistor_SMD:R_0402_1005Metric, F.Cu at (191.2, 92.8)
- added R6: 0R, Resistor_SMD:R_0402_1005Metric, F.Cu at (121.0, 142.3)
- added R60: 33R, Resistor_SMD:R_0402_1005Metric, F.Cu at (191.2, 94.8)
- added R61: 33R, Resistor_SMD:R_0402_1005Metric, F.Cu at (191.2, 96.8)
- added R62: 33R, Resistor_SMD:R_0402_1005Metric, F.Cu at (191.2, 98.8)
- added R63: 10k, Resistor_SMD:R_0402_1005Metric, F.Cu at (84.9, 122.6)
- added R64: 3.3k, Resistor_SMD:R_0402_1005Metric, F.Cu at (84.9, 124.6)
- added R65: 13k, Resistor_SMD:R_0402_1005Metric, F.Cu at (84.9, 126.5)
- added R66: 13k, Resistor_SMD:R_0402_1005Metric, F.Cu at (84.9, 128.5)
- added R67: 4.7k, Resistor_SMD:R_0402_1005Metric, F.Cu at (84.9, 130.5)
- added R68: NC, Resistor_SMD:R_0402_1005Metric, F.Cu at (84.9, 132.5)
- added R69: NC, Resistor_SMD:R_0402_1005Metric, F.Cu at (87.8, 122.6)
- added R7: 0R, Resistor_SMD:R_0402_1005Metric, F.Cu at (121.0, 144.3)
- added R70: 10k, Resistor_SMD:R_0402_1005Metric, F.Cu at (87.8, 124.6)
- added R71: 10k, Resistor_SMD:R_0402_1005Metric, F.Cu at (87.8, 126.5)
- added R72: 470R, Resistor_SMD:R_0402_1005Metric, F.Cu at (87.8, 128.5)
- added R73: 100R, Resistor_SMD:R_0402_1005Metric, F.Cu at (87.8, 130.5)
- added R74: 33R, Resistor_SMD:R_0402_1005Metric, F.Cu at (87.8, 132.5)
- added R75: 33R, Resistor_SMD:R_0402_1005Metric, F.Cu at (90.7, 122.6)
- added R76: 49.9R, Resistor_SMD:R_0402_1005Metric, F.Cu at (90.7, 124.6)
- added R77: 49.9R, Resistor_SMD:R_0402_1005Metric, F.Cu at (90.7, 126.5)
- added R78: 33R, Resistor_SMD:R_0402_1005Metric, F.Cu at (90.7, 128.5)
- added R79: 33R, Resistor_SMD:R_0402_1005Metric, F.Cu at (90.7, 130.5)
- added R8: 2.2R, Resistor_SMD:R_0402_1005Metric, F.Cu at (121.0, 146.3)
- added R80: 49.9R, Resistor_SMD:R_0402_1005Metric, F.Cu at (90.7, 132.5)
- added R81: 49.9R, Resistor_SMD:R_0402_1005Metric, F.Cu at (93.6, 122.6)
- added R82: 33R, Resistor_SMD:R_0402_1005Metric, F.Cu at (93.6, 124.6)
- added R83: 33R, Resistor_SMD:R_0402_1005Metric, F.Cu at (93.6, 126.5)
- added R84: 49.9R, Resistor_SMD:R_0402_1005Metric, F.Cu at (93.6, 128.5)
- added R85: 49.9R, Resistor_SMD:R_0402_1005Metric, F.Cu at (93.6, 130.5)
- added R86: 0R, Resistor_SMD:R_0402_1005Metric, F.Cu at (146.4, 84.8)
- added R87: 6.8k, Resistor_SMD:R_0402_1005Metric, F.Cu at (123.9, 144.3)
- added R88: 0R, Resistor_SMD:R_0402_1005Metric, F.Cu at (123.9, 146.3)
- added R89: 6.8k, Resistor_SMD:R_0402_1005Metric, F.Cu at (123.9, 122.8)
- added R9: 2.2R, Resistor_SMD:R_0402_1005Metric, F.Cu at (121.0, 148.3)
- added R90: 6.8k, Resistor_SMD:R_0402_1005Metric, F.Cu at (123.9, 124.8)
- added SW1: PWR, Button_Switch_SMD:SW_Push_1P1T_XKB_TS-1187A, F.Cu at (166.0, 55.3)
- added SW2: RESET, Button_Switch_SMD:SW_Push_1P1T_XKB_TS-1187A, F.Cu at (166.0, 62.0)
- added SW3: MASK, Button_Switch_SMD:SW_Push_1P1T_XKB_TS-1187A, F.Cu at (166.0, 68.6)
- added SW4: RECOVERY, Button_Switch_SMD:SW_Push_1P1T_XKB_TS-1187A, F.Cu at (166.0, 75.3)
- added U1: TPD4EUSB30, Package_SON:USON-10_2.5x1.0mm_P0.5mm, F.Cu at (128.9, 134.1)
- added U10: TPD4EUSB30, Package_SON:USON-10_2.5x1.0mm_P0.5mm, F.Cu at (134.7, 112.6)
- added U11: TPD4EUSB30, Package_SON:USON-10_2.5x1.0mm_P0.5mm, F.Cu at (143.5, 108.1)
- added U12: TPD4EUSB30, Package_SON:USON-10_2.5x1.0mm_P0.5mm, F.Cu at (146.4, 108.1)
- added U13: TPD4EUSB30, Package_SON:USON-10_2.5x1.0mm_P0.5mm, F.Cu at (149.3, 108.1)
- added U14: AP2331, Package_TO_SOT_SMD:SOT-23-3, F.Cu at (153.3, 108.3)
- added U15: LPJM4938GENL, Connector_RJ:RJ45_Wuerth_7499111446_Horizontal, F.Cu at (146.2, 118.4)
- added U16: TPD4EUSB30, Package_SON:USON-10_2.5x1.0mm_P0.5mm, F.Cu at (163.2, 135.7)
- added U17: TPD4EUSB30, Package_SON:USON-10_2.5x1.0mm_P0.5mm, F.Cu at (166.1, 135.7)
- added U18: TPD4EUSB30, Package_SON:USON-10_2.5x1.0mm_P0.5mm, F.Cu at (173.5, 106.7)
- added U19: TPD4EUSB30, Package_SON:USON-10_2.5x1.0mm_P0.5mm, F.Cu at (176.4, 106.7)
- added U2: TPD4EUSB30, Package_SON:USON-10_2.5x1.0mm_P0.5mm, F.Cu at (131.8, 134.1)
- added U20: TPS54331DR, TPS54331DR:SOIC127P599X175-8N, F.Cu at (108.7, 136.6)
- added U21: AP2127K-3.3, Package_TO_SOT_SMD:SOT-23-5, F.Cu at (109.1, 117.3)
- added U22: CH334F, Package_DFN_QFN:QFN-24-1EP_4x4mm_P0.5mm_EP2.6x2.6mm, F.Cu at (185.1, 65.0)
- added U3: TPD4EUSB30, Package_SON:USON-10_2.5x1.0mm_P0.5mm, F.Cu at (134.7, 134.1)
- added U4: FUSB302BMPX, Package_DFN_QFN:WQFN-14-1EP_2.5x2.5mm_P0.5mm_EP1.45x1.45mm, F.Cu at (135.0, 138.5)
- added U5: SY6280AAC, Package_TO_SOT_SMD:SOT-23-5, F.Cu at (130.0, 138.5)
- added U6: SY6280AAC, Package_TO_SOT_SMD:SOT-23-5, F.Cu at (130.0, 117.0)
- added U7: FUSB302BMPX, Package_DFN_QFN:WQFN-14-1EP_2.5x2.5mm_P0.5mm_EP1.45x1.45mm, F.Cu at (135.0, 117.0)
- added U8: TPD4EUSB30, Package_SON:USON-10_2.5x1.0mm_P0.5mm, F.Cu at (128.9, 112.6)
- added U9: TPD4EUSB30, Package_SON:USON-10_2.5x1.0mm_P0.5mm, F.Cu at (131.8, 112.6)
- added Y1: 25MHz, Crystal:Crystal_SMD_2016-4Pin_2.0x1.6mm, F.Cu at (108.5, 129.1)
- added Y2: 12MHz, Crystal:Crystal_SMD_2016-4Pin_2.0x1.6mm, F.Cu at (183.9, 69.9)
Other:
- board outline added: 52.2 x 62.2 mm
- copper layers 0 -> 2

Commit message: audio done
Parts:
- added C69: 10uF, Capacitor_SMD:C_0402_1005Metric, F.Cu at (93.2, 129.1)
- added R100: 18k, Resistor_SMD:R_0402_1005Metric, F.Cu at (166.6, 79.3)
- added R101: 18k, Resistor_SMD:R_0402_1005Metric, F.Cu at (166.6, 81.3)
- added R91: 510, Resistor_SMD:R_0402_1005Metric, F.Cu at (163.7, 77.3)
- added R92: 510, Resistor_SMD:R_0402_1005Metric, F.Cu at (163.7, 79.3)
- added R93: 24k, Resistor_SMD:R_0402_1005Metric, F.Cu at (163.7, 81.3)
- added R94: 510, Resistor_SMD:R_0402_1005Metric, F.Cu at (163.7, 83.2)
- added R95: 24k, Resistor_SMD:R_0402_1005Metric, F.Cu at (163.7, 85.2)
- added R96: 510, Resistor_SMD:R_0402_1005Metric, F.Cu at (163.7, 87.2)
- added R97: 24k, Resistor_SMD:R_0402_1005Metric, F.Cu at (166.6, 73.3)
- added R98: 510, Resistor_SMD:R_0402_1005Metric, F.Cu at (166.6, 75.3)
- added R99: 2k, Resistor_SMD:R_0402_1005Metric, F.Cu at (166.6, 77.3)
- C45, C46: footprint Capacitor_SMD:C_0402_1005Metric -> Capacitor_SMD:C_0603_1608Metric
- C50, C51: footprint Capacitor_SMD:C_1206_3216Metric -> Capacitor_SMD:C_0402_1005Metric
- C52: value 22uF -> 10uF; footprint Capacitor_SMD:C_0603_1608Metric -> Capacitor_SMD:C_0402_1005Metric
- C53: footprint Capacitor_SMD:C_0603_1608Metric -> Capacitor_SMD:C_0402_1005Metric
- R12, R13, R49, R8, R9: footprint Resistor_SMD:R_0402_1005Metric -> Resistor_SMD:R_0603_1608Metric
- R24: value 1.8k -> 18k
- R26, R29: value 1.8k -> 2k
- R33, R34, R36, R38, R40: value 499R -> 24k
- R35, R37, R39: value 499R -> 510
- R53, R54, R55, R56: value 560R -> 680R
- R65: value 13k -> 24k
- R66: value 13k -> 2k
- R68, R69: value NC -> 0R
- Y1, Y2: footprint Crystal:Crystal_SMD_2016-4Pin_2.0x1.6mm -> Crystal:Crystal_SMD_3225-4Pin_3.2x2.5mm
- moved J2 116.6 mm to (98.0, 146.5)
- moved J14 60.4 mm to (124.3, 115.4)
- moved U19 60.4 mm to (119.8, 127.9)
- moved U18 60.4 mm to (116.9, 127.9)
- moved R57 60.4 mm to (134.6, 110.0)
- moved R58 60.4 mm to (134.6, 112.0)
- moved R59 60.4 mm to (134.6, 114.0)
- moved R60 60.4 mm to (134.6, 116.0)
- moved R61 60.4 mm to (134.6, 118.0)
- moved R62 60.4 mm to (134.6, 120.0)
- moved C33 56.6 mm to (119.8, 143.0)
- moved C34 56.6 mm to (119.8, 145.0)
- moved R50 56.6 mm to (116.9, 143.1)
- moved J13 56.6 mm to (127.0, 137.0)
- moved R51 56.6 mm to (116.9, 145.0)
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Connections:
- D3 pad 1: unconnected-(R26-Pad1) -> Net-(R100-Pad1)
- R24 pad 1: unconnected-(R26-Pad1) -> Net-(R100-Pad1)
- R26 pad 1: unconnected-(R26-Pad1) -> Net-(R100-Pad1)
- R35 pad 1: /HDMI_TX/HDMI0_TX0N_PORT -> /HDMI_TX/HDMI0_TX3P_PORT
- R35 pad 2: Net-(Q7-D) -> Net-(Q6-D)
- R36 pad 1: /HDMI_TX/HDMI0_TX0P_PORT -> /HDMI_TX/HDMI0_TX0N_PORT
- R37 pad 1: /HDMI_TX/HDMI0_TX1N_PORT -> /HDMI_TX/HDMI0_TX0N_PORT
- R37 pad 2: Net-(Q8-D) -> Net-(Q7-D)
- R38 pad 1: /HDMI_TX/HDMI0_TX1P_PORT -> /HDMI_TX/HDMI0_TX0P_PORT
- R38 pad 2: Net-(Q8-D) -> Net-(Q7-D)
- R39 pad 1: /HDMI_TX/HDMI0_TX2N_PORT -> /HDMI_TX/HDMI0_TX0P_PORT
- R39 pad 2: Net-(Q9-D) -> Net-(Q7-D)
- R40 pad 1: /HDMI_TX/HDMI0_TX2P_PORT -> /HDMI_TX/HDMI0_TX1N_PORT
- R40 pad 2: Net-(Q9-D) -> Net-(Q8-D)

Commit message: work preparing for routing
Parts:
- removed C35, C36: 100nF, Capacitor_SMD:C_0402_1005Metric
- removed R55, R56: 680R, Resistor_SMD:R_0402_1005Metric
- removed U15: LPJM4938GENL, Connector_RJ:RJ45_Wuerth_7499111446_Horizontal
- added C70: 0.1uF, Capacitor_SMD:C_0402_1005Metric, F.Cu at (79.4, 119.4)
- added C71: 0.1uF, Capacitor_SMD:C_0402_1005Metric, F.Cu at (147.6, 127.3)
- added C72: 0.1uF, Capacitor_SMD:C_0402_1005Metric, F.Cu at (147.6, 129.3)
- added C73: 1uF, Capacitor_SMD:C_0402_1005Metric, F.Cu at (147.6, 131.2)
- added C74: 10uF, Capacitor_SMD:C_0402_1005Metric, F.Cu at (150.4, 127.3)
- added C75: 1uF, Capacitor_SMD:C_0402_1005Metric, F.Cu at (150.4, 129.3)
- added C76: 1uF, Capacitor_SMD:C_0402_1005Metric, F.Cu at (150.4, 131.2)
- added C77: 10uF, Capacitor_SMD:C_0402_1005Metric, F.Cu at (153.3, 127.3)
- added C78: 1uF, Capacitor_SMD:C_0402_1005Metric, F.Cu at (153.3, 129.3)
- added C79: 1uF, Capacitor_SMD:C_0402_1005Metric, F.Cu at (153.3, 131.2)
- added C80: 10uF, Capacitor_SMD:C_0402_1005Metric, F.Cu at (127.5, 70.6)
- added C81: 10uF, Capacitor_SMD:C_0402_1005Metric, F.Cu at (127.5, 72.6)
- added C82: 100nF, Capacitor_SMD:C_0402_1005Metric, F.Cu at (127.5, 74.5)
- added C83: 10uF, Capacitor_SMD:C_0402_1005Metric, F.Cu at (127.5, 76.5)
- added C84: 1uF, Capacitor_SMD:C_0402_1005Metric, F.Cu at (130.4, 70.6)
- added C85: 1nF, Capacitor_SMD:C_0402_1005Metric, F.Cu at (130.4, 72.6)
- added C86: 10pF, Capacitor_SMD:C_0402_1005Metric, F.Cu at (130.4, 74.5)
- added C87: 10uF, Capacitor_SMD:C_0402_1005Metric, F.Cu at (130.4, 76.5)
- added C88: 10uF, Capacitor_SMD:C_0402_1005Metric, F.Cu at (133.2, 70.6)
- added C89: 8.2nF, Capacitor_SMD:C_0402_1005Metric, F.Cu at (133.2, 72.6)
- added C90: 0.1uF, Capacitor_SMD:C_0402_1005Metric, F.Cu at (79.4, 121.3)
- added C91: 1uF, Capacitor_SMD:C_0402_1005Metric, F.Cu at (79.4, 123.3)
- added C92: 10uF, Capacitor_SMD:C_0402_1005Metric, F.Cu at (133.2, 74.5)
- added C93: 10uF, Capacitor_SMD:C_0402_1005Metric, F.Cu at (133.2, 76.5)
- added C94: 100nF/100V, Capacitor_SMD:C_0402_1005Metric, F.Cu at (126.4, 119.7)
- added C95: 100nF/100V, Capacitor_SMD:C_0402_1005Metric, F.Cu at (126.4, 121.7)
- added C96: 100nF/100V, Capacitor_SMD:C_0402_1005Metric, F.Cu at (126.4, 123.7)
- added C97: 100nF/100V, Capacitor_SMD:C_0402_1005Metric, F.Cu at (126.4, 125.6)
- added CN1: PJ-332A-6A (3.5mm Jack), Headphone_Jack:AUDIO-SMD_PJ-332A-6A, F.Cu at (142.1, 113.4)
- added D6: LESD8D5.0CB1T5G, Diode_SMD:D_SOD-882, F.Cu at (152.2, 109.7)
- added D7: LESD8D5.0CB1T5G, Diode_SMD:D_SOD-882, F.Cu at (152.2, 112.0)
- added D8: SS54, Diode_SMD:D_SMA, F.Cu at (138.7, 71.9)
- added J11: SYSTEM, 6P_05mm_FPC:FPC-SMD_6P-P0.50_XUNPU_FPC-05F-6PH20, F.Cu at (85.3, 130.1)
- added J21: 5V IN, Connector_JST:JST_GH_SM10B-GHS-TB_1x10-1MP_P1.25mm_Horizontal, F.Cu at (135.1, 43.7)
- added J22: BATTERY IN, Connector_JST:JST_GH_SM10B-GHS-TB_1x10-1MP_P1.25mm_Horizontal, F.Cu at (135.1, 51.1)
- added J23: L829-1J1T-JM, Ethernet:BEL_L829-1J1T-JM, F.Cu at (113.9, 122.5)
- added J3: RIGHT SPEAKERS, Connector_PinHeader_2.54mm:PinHeader_1x02_P2.54mm_Horizontal, F.Cu at (135.1, 120.7)
- added J4: LEFT SPEAKERS, Connector_PinHeader_2.54mm:PinHeader_1x02_P2.54mm_Horizontal, F.Cu at (135.1, 127.9)
- added J6: OLED EL POWER, 6P_05mm_FPC:FPC-SMD_6P-P0.50_XUNPU_FPC-05F-6PH20, F.Cu at (73.9, 147.8)
- added J9: Inner USB-C, USB-C:USB-C-SMD_TYPE-C-24P-QT, F.Cu at (162.3, 121.7)
- added L2: 3.3uH, Inductor_SMD:L_Vishay_IHLP-1616, F.Cu at (132.6, 80.3)
- added Q12: 2SK3018W, Package_TO_SOT_SMD:SOT-323_SC-70, F.Cu at (150.3, 116.1)
- added R102: 0R, Resistor_SMD:R_0402_1005Metric, F.Cu at (147.6, 119.3)
- added R103: 0R, Resistor_SMD:R_0402_1005Metric, F.Cu at (147.6, 121.3)
- added R104: 0R, Resistor_SMD:R_0402_1005Metric, F.Cu at (147.6, 123.3)
- added R105: 10k, Resistor_SMD:R_0402_1005Metric, F.Cu at (147.6, 125.3)
- added R106: 10k, Resistor_SMD:R_0402_1005Metric, F.Cu at (150.5, 119.3)
- added R107: 33R, Resistor_SMD:R_0402_1005Metric, F.Cu at (150.5, 121.3)
- added R108: 33R, Resistor_SMD:R_0402_1005Metric, F.Cu at (150.5, 123.3)
- added R109: 100k, Resistor_SMD:R_0402_1005Metric, F.Cu at (150.5, 125.3)
- added R110: 10k, Resistor_SMD:R_0402_1005Metric, F.Cu at (153.4, 119.3)
- added R111: 2.2k, Resistor_SMD:R_0402_1005Metric, F.Cu at (153.4, 121.3)
- added R112: 24k, Resistor_SMD:R_0402_1005Metric, F.Cu at (127.5, 78.5)
- added R113: 2k, Resistor_SMD:R_0402_1005Metric, F.Cu at (127.5, 80.5)
- added R114: 10k, Resistor_SMD:R_0402_1005Metric, F.Cu at (127.5, 82.5)
- added R115: 3.3k, Resistor_SMD:R_0402_1005Metric, F.Cu at (127.5, 84.5)
- added R116: 10k, Resistor_SMD:R_0402_1005Metric, F.Cu at (85.2, 115.5)
- added R117: 10k, Resistor_SMD:R_0402_1005Metric, F.Cu at (85.2, 117.5)
- added R118: 0R, Resistor_SMD:R_0402_1005Metric, F.Cu at (153.4, 123.3)
- added R119: 0R, Resistor_SMD:R_0402_1005Metric, F.Cu at (153.4, 125.3)
- added R120: 0R, Resistor_SMD:R_0402_1005Metric, F.Cu at (79.8, 146.4)
- added R121: 0R, Resistor_SMD:R_0402_1005Metric, F.Cu at (79.8, 148.4)
- added R122: 1M, Resistor_SMD:R_0402_1005Metric, F.Cu at (175.0, 125.4)
- added TP1: RJ45 ORANGE LED, TestPoint:TestPoint_Pad_D2.0mm, F.Cu at (127.0, 132.9)
- added U23: TPA2028D1YZFT, Audio_Amp:BGA9C50P3X3_162X162X63, F.Cu at (149.5, 109.9)
- added U24: SOT23 Hall Effect Sensor, Package_TO_SOT_SMD:SOT-23, F.Cu at (93.8, 115.6)
- added U25: TPA2028D1YZFT, Audio_Amp:BGA9C50P3X3_162X162X63, F.Cu at (149.5, 112.7)
- added U26: AMS1117-1.8, Package_TO_SOT_SMD:SOT-223-3_TabPin2, F.Cu at (131.0, 59.0)
- added U27: TPS54331DR, TPS54331DR:SOIC127P599X175-8N, F.Cu at (130.8, 66.4)
- added U28: SPI Flash, Package_SO:SOIC-8_3.9x4.9mm_P1.27mm, F.Cu at (94.0, 131.0)
- J5: value USB_C_Receptacle -> Outer USB-C
- J7: footprint Connector_RJ:RJ45_Wuerth_7499111446_Horizontal -> Connector_PinHeader_2.54mm:PinHeader_1x02_P2.54mm_Horizontal
- R53, R54: value 680R -> 1k
- moved SW1 114.5 mm to (73.7, 111.9)
- moved SW2 114.5 mm to (73.7, 118.5)
- moved SW3 114.5 mm to (73.7, 125.2)
- moved SW4 114.5 mm to (73.7, 131.8)
- moved C28 109.0 mm to (79.4, 109.5)
- moved C29 109.0 mm to (79.4, 111.5)
- moved C30 109.0 mm to (79.4, 113.5)
- moved C31 109.0 mm to (79.4, 115.4)
- moved C32 109.0 mm to (79.4, 117.4)
- moved J10 107.6 mm to (89.0, 110.9)
- moved J7 101.1 mm to (83.2, 122.8)
- moved R49 94.9 mm to (96.3, 125.6)
- moved R68 93.5 mm to (159.0, 62.1)
- moved R74 93.5 mm to (161.9, 62.1)
- moved C37 93.5 mm to (147.5, 52.1)
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Connections:
- net /UART2_TX_M0_DEBUG renamed /System/UART_TX
- net /eDP/VBAT renamed Net-(J6-Pin_4)
- net Net-(SW3-A) renamed /System/BOOT_SARADC
- C28 pad 1: /PWRON_L -> /System/PWRON_L
- C29 pad 1: /RESET_L -> /System/RESET_L
- C31 pad 1: /RECOVERY -> /System/RECOVERY
- C33 pad 2: (no net) -> unconnected-(C33-Pad2)
- C4 pad 1: (no net) -> /USBC0/IN_TX1-
- C5 pad 1: unconnected-(C5-Pad1) -> /USBC0/IN_TX1+
- C52 pad 1: /PCIE3.0-MKEY/+5v -> +5V
- C6 pad 1: unconnected-(C6-Pad1) -> /USBC0/IN_TX2-
- C69 pad 1: /PCIE3.0-MKEY/+5v -> +5V
- C7 pad 1: unconnected-(C7-Pad1) -> /USBC0/IN_TX2+
- CMC1 pad 1: (no net) -> /USBC0/IN_D-
- CMC1 pad 2: (no net) -> /USBC0/IN_D+
- J13 pad 14: (no net) -> unconnected-(R50-Pad1)
- J13 pad 23: (no net) -> unconnected-(R52-Pad2)
- J13 pad 35: (no net) -> unconnected-(C33-Pad2)
- J2 pad 10: /eDP/DP_1P -> /HDMI1_TX0P_PORT
- J2 pad 12: /eDP/DP_0N -> /HDMI1_TX_SBDN
- J2 pad 13: /eDP/DP_0P -> /HDMI1_TX_SBDP
- J2 pad 15: /eDP/AUX_P -> /HDMI1_TX3P_PORT
- J2 pad 16: /eDP/AUX_N -> /HDMI1_TX3N_PORT
- J2 pad 21: /eDP/BIST_EN -> Net-(J2-Pad21)
- J2 pad 25: /eDP/HPD -> Net-(J2-Pad25)
- J2 pad 3: /eDP/DP_3N -> /HDMI1_TX2N_PORT
- J2 pad 4: /eDP/DP_3P -> /HDMI1_TX2P_PORT
- J2 pad 6: /eDP/DP_2N -> /HDMI1_TX1N_PORT
- J2 pad 7: /eDP/DP_2P -> /HDMI1_TX1P_PORT
- J2 pad 9: /eDP/DP_1N -> /HDMI1_TX0N_PORT
- J20 pad 101: /RECOVERY -> /System/RECOVERY
- J20 pad 103: /HPR -> /Audio/R_AUDIO
- J20 pad 104: /HPL -> /Audio/L_AUDIO
- J20 pad 16: /RESET_L -> /System/RESET_L
- J20 pad 17: /PWRON_L -> /System/PWRON_L
- J20 pad 283: /GPIO1_A7 -> /Audio/SPK_EN
- J5 pad A10: unconnected-(R4-Pad1) -> /USBC0/IN_RX2-
- J5 pad A11: unconnected-(R5-Pad1) -> /USBC0/IN_RX2+
- J5 pad A2: unconnected-(C5-Pad1) -> /USBC0/IN_TX1+
- J5 pad A3: (no net) -> /USBC0/IN_TX1-
- J5 pad A6: (no net) -> /USBC0/IN_D+
- J5 pad A7: (no net) -> /USBC0/IN_D-
- J5 pad B10: unconnected-(R6-Pad1) -> /USBC0/IN_RX1-
- J5 pad B11: unconnected-(R7-Pad1) -> /USBC0/IN_RX1+
- J5 pad B2: unconnected-(C7-Pad1) -> /USBC0/IN_TX2+
- J5 pad B3: unconnected-(C6-Pad1) -> /USBC0/IN_TX2-
- J5 pad B6: (no net) -> /USBC0/IN_D+
- J5 pad B7: (no net) -> /USBC0/IN_D-
- R1 pad 1: (no net) -> unconnected-(R1-Pad1)
- R4 pad 1: unconnected-(R4-Pad1) -> /USBC0/IN_RX2-
- R41 pad 1: /PWRON_L -> /System/PWRON_L
- R41 pad 2: Net-(SW1-A) -> /System/PWRON_L
- R42 pad 1: /RESET_L -> /System/RESET_L
- R42 pad 2: Net-(SW2-A) -> /System/RESET_L
- R44 pad 1: /RECOVERY -> /System/RECOVERY
- R44 pad 2: Net-(SW4-A) -> /System/RECOVERY
- R5 pad 1: unconnected-(R5-Pad1) -> /USBC0/IN_RX2+
- R50 pad 1: (no net) -> unconnected-(R50-Pad1)
- R52 pad 2: (no net) -> unconnected-(R52-Pad2)
- R6 pad 1: unconnected-(R6-Pad1) -> /USBC0/IN_RX1-
- R7 pad 1: unconnected-(R7-Pad1) -> /USBC0/IN_RX1+
- SW1 pad 1: Net-(SW1-A) -> /System/PWRON_L
- SW2 pad 1: Net-(SW2-A) -> /System/RESET_L
- SW4 pad 1: Net-(SW4-A) -> /System/RECOVERY
- U1 pad 10: (no net) -> unconnected-(U1-NC-Pad10)
- U1 pad 6: (no net) -> unconnected-(U1-NC-Pad6)
- U1 pad 7: (no net) -> unconnected-(U1-NC-Pad7)
- U1 pad 9: (no net) -> unconnected-(U1-NC-Pad9)
- U20 pad 2: /PCIE3.0-MKEY/+5v -> +5V
- U22 pad 25: (no net) -> GND

Commit message: initial motherboard layout!
Parts:
- moved C44 280.8 mm to (-64.5, 233.0)
- moved C45 280.8 mm to (-43.6, 237.9)
- moved C46 280.8 mm to (-43.6, 240.4)
- moved C47 280.8 mm to (-64.5, 235.0)
- moved C48 280.8 mm to (-64.5, 237.0)
- moved C49 280.8 mm to (-64.5, 238.9)
- moved C50 280.8 mm to (-64.5, 240.9)
- moved C51 280.8 mm to (-64.5, 242.9)
- moved C52 280.8 mm to (-64.5, 244.8)
- moved C53 280.8 mm to (-61.6, 233.0)
- moved C54 280.8 mm to (-61.6, 235.0)
- moved C55 280.8 mm to (-61.6, 237.0)
- moved C56 280.8 mm to (-61.6, 238.9)
- moved C57 280.8 mm to (-61.6, 240.9)
- moved C58 280.8 mm to (-61.6, 242.9)
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Connections:
- U18 pad 1: /SD Card/D2 -> /SD Card/VDD
- U18 pad 10: unconnected-(U18-NC-Pad10) -> /SD Card/VDD
- U18 pad 2: /SD Card/D3 -> /SD Card/CMD
- U18 pad 4: /SD Card/CMD -> /SD Card/D3
- U18 pad 5: /SD Card/CLK -> /SD Card/D2
- U18 pad 6: unconnected-(U18-NC-Pad6) -> /SD Card/D2
- U18 pad 7: unconnected-(U18-NC-Pad7) -> /SD Card/D3
- U18 pad 9: unconnected-(U18-NC-Pad9) -> /SD Card/CMD
- U19 pad 1: /SD Card/D0 -> /SD Card/DET
- U19 pad 10: unconnected-(U19-NC-Pad10) -> /SD Card/DET
- U19 pad 4: /SD Card/DET -> /SD Card/D0
- U19 pad 5: /SD Card/VDD -> /SD Card/CLK
- U19 pad 6: unconnected-(U19-NC-Pad6) -> /SD Card/CLK
- U19 pad 7: unconnected-(U19-NC-Pad7) -> /SD Card/D0
- U19 pad 9: unconnected-(U19-NC-Pad9) -> /SD Card/D1
Routing:
- net /SD Card/D2: track 0.00 -> 5.83 mm
- net /SD Card/CMD: track 0.00 -> 5.44 mm
- net /SD Card/DET: track 0.00 -> 5.32 mm
- net /SD Card/D0: track 0.00 -> 5.03 mm
- net /SD Card/D1: track 0.00 -> 4.98 mm
- net /SD Card/D3: track 0.00 -> 4.56 mm
- net /SD Card/CLK: track 0.00 -> 4.18 mm
- net /SD Card/VDD: track 0.00 -> 2.62 mm
- added copper zone on B.Cu, net GND
- added copper zone on F.Cu, net GND
- added copper zone on In1.Cu, net GND
- added copper zone on In2.Cu, net GND
Other:
- board size 52.2 x 62.2 mm -> 177 x 88 mm
- copper layers 2 -> 4
