File: motherboard/audio.kicad_sch (KiCad schematic)
At the start: 27 parts, among them CN1 PJ-332A-6A (3.5mm Jack), J3 RIGHT SPEAKERS, J4 LEFT SPEAKERS, Q12 2SK3018W, U16 TPA2016D2RTJR

Commit message: v0.2 good routing checkpoint (217 unrouted)
Connections:
- net GND: now also C34.1, C35.1
Changed lines of the file:
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@@
 	)
 	(junction
+		(at 90.17 73.66)
+		(diameter 0)
+		(color 0 0 0 0)
+	)
+	(junction
 		(at 161.29 123.19)
 		(diameter 0)
@@
 	(wire
 		(pts
+			(xy 90.17 73.66) (xy 90.17 76.2)
+		)
+		(stroke
+			(width 0)
+			(type default)
+		)
+	)
+	(wire
+		(pts
 			(xy 161.29 123.19) (xy 161.29 132.08)
 		)
@@
 	(wire
 		(pts
+			(xy 74.93 76.2) (xy 74.93 73.66)
+		)
+		(stroke
+			(width 0)
+			(type default)
+		)
+	)
+	(wire
+		(pts
 			(xy 100.33 50.8) (xy 100.33 53.34)
 		)
@@
 	(wire
 		(pts
+			(xy 74.93 73.66) (xy 90.17 73.66)
+		)
+		(stroke
+			(width 0)
+			(type default)
+		)
+	)
+	(wire
+		(pts
 			(xy 100.33 48.26) (xy 100.33 50.8)
 		)
@@
 	(wire
 		(pts
-			(xy 90.17 71.12) (xy 90.17 76.2)
+			(xy 90.17 71.12) (xy 90.17 73.66)
 		)
 		(stroke
@@
 					(unit 1)
 				)
+			)
+		)
+	)
+	(symbol
+		(lib_id "power:GND")
+		(at 74.93 76.2 0)
+		(unit 1)
+		(exclude_from_sim no)
+		(in_bom yes)
+		(on_board yes)
+		(dnp no)
+		(fields_autoplaced yes)
+		(property "Reference" "#PWR0139"
+			(at 74.93 82.55 0)
+			(effects
+				(font
+					(size 1.27 1.27)
+				)
+				(hide yes)
+			)
+		)
+		(property "Value" "GND"
+			(at 74.93 81.28 0)
+			(effects
+				(font
+					(size 1.27 1.27)
+				)
+			)
+		)
+		(property "Footprint" ""
+			(at 74.93 76.2 0)
+			(effects
+				(font
+					(size 1.27 1.27)
+				)
+				(hide yes)
+			)
+		)
+		(property "Datasheet" ""
+			(at 74.93 76.2 0)
+			(effects
+				(font
+					(size 1.27 1.27)
+				)
+				(hide yes)
+			)
+		)
+		(property "Description" "Power symbol creates a global label with name \"GND\" , ground"
+			(at 74.93 76.2 0)
+			(effects
+				(font
+					(size 1.27 1.27)
+				)
+				(hide yes)
+			)
+		)
+		(pin "1"
+		)
+		(instances
+			(project "motherboard"
+				(path "/025fe4d1-0305-4b34-be04-f8d9818125a4/d168cefe-cdbf-401a-9d73-1a46286dd06c"
+					(reference "#PWR0139")
+					(unit 1)
+				)

Commit message: v0.2 75 routes left!
Parts:
- U16: footprint TPA2016:QFN50P400X400X80-21N -> TPA2016D2RTJR:QFN50P400X400X80-21N
Changed lines of the file:
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@@
 			)
 		)
-		(property "Footprint" "TPA2016:QFN50P400X400X80-21N"
+		(property "Footprint" "TPA2016D2RTJR:QFN50P400X400X80-21N"
 			(at 118.11 66.04 0)
 			(effects

Commit message: mainboard v0.3 + power WIP
Other:
- company: (none) -> Byran Huang
- title: (none) -> anyon e
Changed lines of the file:
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@@
 	(generator_version "8.99")
 	(paper "A4")
+	(title_block
+		(title "anyon e")
+		(date "2024-09-15")
+		(rev "V0.3")
+		(company "Byran Huang")
+		(comment 4 "Proof of concept board for feature verification")
+	)
 	(junction
 		(at 77.47 45.72)

Commit message: preparing for motherboard v1.1
Parts:
- renumbered C38 to C51, C37 to C52, C33 to C53, C34 to C54, C35 to C55, C36 to C56, C73 to C57, C72 to C58, C71 to C59, J4 to J17, J3 to J18, Q12 to Q3, R111 to R50, R109 to R51, R110 to R52, R102 to R53, R103 to R54, R104 to R55, R106 to R56, R105 to R57, R107 to R58, R108 to R59, U16 to U19
