File: motherboard/pcie30-mkey.kicad_sch (KiCad schematic)
At the start: 50 parts, among them IC1 PI6C557-05BLE, J15 Bus_M.2_Socket_M, U20 TPS54331DR, U21 AP2127K-3.3, Y1 25MHz

Commit message: created display evaluation board + layout modifications
Parts:
- IC1: footprint SOP65P640X120-20N:SOP65P640X120-20N -> SOP65P640X120-20N
Changed lines of the file:
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@@
 			)
 		)
-		(property "Footprint" "SOP65P640X120-20N:SOP65P640X120-20N"
+		(property "Footprint" "SOP65P640X120-20N"
 			(at 204.47 160.96 0)
 			(effects

Commit message: motherboard net labeling and impedance matching
Parts:
- IC1: footprint SOP65P640X120-20N -> SOP65P640X120-20N:SOP65P640X120-20N
Connections:
- net PCIE0_PORT0_REFCLKN_IN renamed PCIE0_PORT0_REFCLKN
- net PCIE0_PORT0_REFCLKP_IN renamed PCIE0_PORT0_REFCLKP
- net PCIE0_PORT1_REFCLKN_IN renamed PCIE0_PORT1_REFCLKN
- net PCIE0_PORT1_REFCLKP_IN renamed PCIE0_PORT1_REFCLKP
Changed lines of the file:
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@@
 		)
 	)
-	(hierarchical_label "PCIE0_PORT0_REFCLKN_IN"
+	(hierarchical_label "PCIE0_PORT0_REFCLKN"
 		(shape input)
 		(at 248.92 116.84 0)
@@
 		)
 	)
-	(hierarchical_label "PCIE0_PORT1_REFCLKN_IN"
+	(hierarchical_label "PCIE0_PORT1_REFCLKN"
 		(shape input)
 		(at 248.92 100.33 0)
@@
 		)
 	)
-	(hierarchical_label "PCIE0_PORT1_REFCLKP_IN"
+	(hierarchical_label "PCIE0_PORT1_REFCLKP"
 		(shape input)
 		(at 248.92 97.79 0)
@@
 		)
 	)
-	(hierarchical_label "PCIE0_PORT0_REFCLKP_IN"
+	(hierarchical_label "PCIE0_PORT0_REFCLKP"
 		(shape input)
 		(at 248.92 114.3 0)
@@
 			)
 		)
-		(property "Footprint" "SOP65P640X120-20N"
+		(property "Footprint" "SOP65P640X120-20N:SOP65P640X120-20N"
 			(at 204.47 160.96 0)
 			(effects

Commit message: added two more display eval test boards
Changed lines of the file:
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@@
+	)
+	(junction
+		(at 121.92 27.94)
+		(diameter 0)
+		(color 0 0 0 0)
 	)
 	(junction
@@
 	(wire
 		(pts
+			(xy 121.92 27.94) (xy 133.35 27.94)
+		)
+		(stroke
+			(width 0)
+			(type default)
+		)
+	)
+	(wire
+		(pts
 			(xy 137.16 129.54) (xy 139.7 129.54)
 		)
@@
 	(wire
 		(pts
-			(xy 121.92 27.94) (xy 133.35 27.94)
+			(xy 119.38 27.94) (xy 121.92 27.94)
 		)
 		(stroke
@@
 		)
 	)
-	(label "+3.3V_PCIE"
-		(at 121.92 27.94 0)
-		(fields_autoplaced yes)
-		(effects
-			(font
-				(size 1.27 1.27)
-			)
-			(justify left bottom)
-		)
-	)
 	(label "+3.3V_PI6C"
 		(at 153.67 81.28 0)
@@
 		)
 	)
+	(global_label "+3.3V_PCIE"
+		(shape input)
+		(at 119.38 27.94 180)
+		(fields_autoplaced yes)
+		(effects
+			(font
+				(size 1.27 1.27)
+			)
+			(justify right)
+		)
+		(property "Intersheetrefs" "${INTERSHEET_REFS}"
+			(at 105.4486 27.94 0)
+			(effects
+				(font
+					(size 1.27 1.27)
+				)
+				(justify right)
+				(hide yes)
+			)
+		)
+	)

Commit message: v0.2 layout
Parts:
- removed C49: 100nF, Capacitor_SMD:C_0402_1005Metric, symbol Device:C_Small
- removed C50, C52, C69: 10uF, Capacitor_SMD:C_0603_1608Metric, symbol Device:C_Small
- removed C51: 1uF, Capacitor_SMD:C_0402_1005Metric, symbol Device:C_Small
- removed C53: 8.2nF, Capacitor_SMD:C_0402_1005Metric, symbol Device:C_Small
- removed C54: 1nF, Capacitor_SMD:C_0402_1005Metric, symbol Device:C_Small
- removed C55: 10pF, Capacitor_SMD:C_0402_1005Metric, symbol Device:C_Small
- removed D5: SS54, Diode_SMD:D_SMA, symbol Device:D_Schottky
- removed L1: 3.3uH, Inductor_SMD:L_Vishay_IHLP-1616, symbol Device:L_Small
- removed R63: 10k, Resistor_SMD:R_0402_1005Metric, symbol Device:R_Small
- removed R64: 3.3k, Resistor_SMD:R_0402_1005Metric, symbol Device:R_Small
- removed R65: 24k, Resistor_SMD:R_0402_1005Metric, symbol Device:R_Small
- removed R66: 2k, Resistor_SMD:R_0402_1005Metric, symbol Device:R_Small
- removed U20: TPS54331DR, TPS54331DR:SOIC127P599X175-8N, symbol TPS54331DR:TPS54331DR

Commit message: mainboard v0.3 + power WIP
Parts:
- added D9: PI6C LED, LED_SMD:LED_0603_1608Metric, symbol Device:LED_Small
- added R91: 33k, Resistor_SMD:R_0402_1005Metric, symbol Device:R_Small
Connections:
- net +3.3V_PI6C: now also R91.2
- net GND: now also D9.1 (K)
- new net: D9.2 (A), R91.1
Changed lines of the file:
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@@
 	(title_block
 		(title "anyon e")
-		(date "2024-06-12")
-		(rev "V0.1")
+		(date "2024-09-15")
+		(rev "V0.3")
 		(company "Byran Huang")
 		(comment 4 "Proof of concept board for feature verification")
@@
 	)
 	(junction
+		(at 179.07 129.54)
+		(diameter 0)
+		(color 0 0 0 0)
+	)
+	(junction
 		(at 139.7 129.54)
 		(diameter 0)
@@
 	(wire
 		(pts
-			(xy 168.91 129.54) (xy 180.34 129.54)
+			(xy 168.91 129.54) (xy 179.07 129.54)
 		)
 		(stroke
@@
 	(wire
 		(pts
+			(xy 179.07 129.54) (xy 180.34 129.54)
+		)
+		(stroke
+			(width 0)
+			(type default)
+		)
+	)
+	(wire
+		(pts
 			(xy 55.88 20.32) (xy 66.04 20.32)
 		)
@@
 	)
 	(symbol
+		(lib_id "Device:LED_Small")
+		(at 179.07 137.16 90)
+		(unit 1)
+		(exclude_from_sim no)
+		(in_bom yes)
+		(on_board yes)
+		(dnp no)
+		(fields_autoplaced yes)
+		(property "Reference" "D9"
+			(at 181.61 135.8264 90)
+			(effects
+				(font
+					(size 1.27 1.27)
+				)
+				(justify right)
+			)
+		)
+		(property "Value" "PI6C LED"
+			(at 181.61 138.3664 90)
+			(effects
+				(font
+					(size 1.27 1.27)
+				)
+				(justify right)
+			)
+		)
+		(property "Footprint" "LED_SMD:LED_0603_1608Metric"
+			(at 179.07 137.16 90)
+			(effects
+				(font
+					(size 1.27 1.27)
+				)
+				(hide yes)
+			)
+		)
+		(property "Datasheet" "~"
+			(at 179.07 137.16 90)
+			(effects
+				(font
+					(size 1.27 1.27)
+				)
+				(hide yes)
+			)
+		)
+		(property "Description" "Light emitting diode, small symbol"
+			(at 179.07 137.16 0)
+			(effects
+				(font
+					(size 1.27 1.27)
+				)
+				(hide yes)
+			)
+		)
+		(pin "2"
+		)
+		(pin "1"
+		)
+		(instances
+			(project "motherboard"
+				(path "/025fe4d1-0305-4b34-be04-f8d9818125a4/8b9107a7-7899-4235-bab8-96db30f71454"
+					(reference "D9")
+					(unit 1)
+				)
+			)
+		)
+	)
+	(symbol
 		(lib_id "power:GND")
 		(at 238.76 106.68 0)
@@
 	)
 	(symbol
+		(lib_id "Device:R_Small")
+		(at 179.07 132.08 180)
+		(unit 1)
+		(exclude_from_sim no)
+		(in_bom yes)
+		(on_board yes)
+		(dnp no)
+		(fields_autoplaced yes)
+		(property "Reference" "R91"
+			(at 181.61 130.8099 0)
+			(effects
+				(font
+					(size 1.27 1.27)
+				)
+				(justify right)
+			)
+		)
+		(property "Value" "33k"
+			(at 181.61 133.3499 0)
+			(effects
+				(font
+					(size 1.27 1.27)
+				)
+				(justify right)
+			)
+		)
+		(property "Footprint" "Resistor_SMD:R_0402_1005Metric"
+			(at 179.07 132.08 0)
+			(effects
+				(font
+					(size 1.27 1.27)
+				)
+				(hide yes)
+			)
+		)
+		(property "Datasheet" "~"
+			(at 179.07 132.08 0)
+			(effects
+				(font
+					(size 1.27 1.27)
+				)
+				(hide yes)
+			)
+		)
+		(property "Description" "Resistor, small symbol"
+			(at 179.07 132.08 0)
+			(effects
+				(font
+					(size 1.27 1.27)
+				)
+				(hide yes)
+			)
+		)
+		(property "LCSC" "C25744"
+			(at 173.99 132.08 0)
+			(effects
+				(font
+					(size 1.27 1.27)
+				)
+				(hide yes)
+			)
+		)
+		(pin "2"
+		)
+		(pin "1"
+		)
+		(instances
+			(project "motherboard"
+				(path "/025fe4d1-0305-4b34-be04-f8d9818125a4/8b9107a7-7899-4235-bab8-96db30f71454"
+					(reference "R91")
+					(unit 1)
+				)
+			)
+		)
+	)
+	(symbol
 		(lib_id "power:+3.3V")
 		(at 148.59 127 0)
@@
 					(unit 1)
 				)
+			)
+		)
+	)
+	(symbol
+		(lib_id "power:GND")
+		(at 179.07 139.7 0)
+		(unit 1)
+		(exclude_from_sim no)
+		(in_bom yes)
+		(on_board yes)
+		(dnp no)
+		(fields_autoplaced yes)
+		(property "Reference" "#PWR0173"
+			(at 179.07 146.05 0)
+			(effects
+				(font
+					(size 1.27 1.27)
+				)
+				(hide yes)
+			)
+		)
+		(property "Value" "GND"
+			(at 179.07 144.78 0)
+			(effects
+				(font
+					(size 1.27 1.27)
+				)
+			)
+		)
+		(property "Footprint" ""
+			(at 179.07 139.7 0)
+			(effects
+				(font
+					(size 1.27 1.27)
+				)
+				(hide yes)
+			)
+		)
+		(property "Datasheet" ""
+			(at 179.07 139.7 0)
+			(effects
+				(font
+					(size 1.27 1.27)
+				)
+				(hide yes)
+			)
+		)
+		(property "Description" "Power symbol creates a global label with name \"GND\" , ground"
+			(at 179.07 139.7 0)
+			(effects
+				(font
+					(size 1.27 1.27)
+				)
+				(hide yes)
+			)
+		)
+		(pin "1"
+		)
+		(instances
+			(project "motherboard"
+				(path "/025fe4d1-0305-4b34-be04-f8d9818125a4/8b9107a7-7899-4235-bab8-96db30f71454"
+					(reference "#PWR0173")
+					(unit 1)
+				)

Commit message: preparing for motherboard v1.1
Parts:
- renumbered C46 to C73, C45 to C74, C47 to C75, C48 to C76, C57 to C77, C56 to C78, C60 to C79, C61 to C80, C58 to C81, C59 to C82, C63 to C83, C62 to C84, D9 to D8, J15 to J23, R74 to R60, R69 to R61, R75 to R62, R68 to R63, R76 to R64, R77 to R65, R67 to R66, R70 to R67, R71 to R68, R72 to R69, R78 to R70, R73 to R71, R79 to R72, R80 to R73, R81 to R74, R82 to R75, R83 to R76, R84 to R77, R85 to R78, R91 to R79, Y1 to Y2
