File: motherboard/eDP.kicad_sch (KiCad schematic)
At the start: 2 parts, among them J2 20455-040E-76 OLED IPEX, J6 OLED EL POWER

Commit message: mainboard v0.3 + power WIP
Parts:
- added C83, C84: 1uF, Capacitor_SMD:C_0402_1005Metric, symbol Device:C_Small
- added R56: 0R, Jumper:SolderJumper-2_P1.3mm_Open_TrianglePad1.0x1.5mm, symbol Device:R_Small
- added U25: TPS22917DBV, Package_TO_SOT_SMD:SOT-23-6, symbol Power_Management:TPS22917DBV
- J2: footprint 20455-040E-76:IPEX_20455-040E-76 -> eDP_Connector:IPEX_20455-040E-76
Connections:
- net +3.3V: now also C84.1, U25.1 (VIN); no longer J2.17, J2.18, J2.19
- net GND: now also C83.2, C84.2, U25.2 (GND)
- net at J6.4 (Pin_4), J6.5 (Pin_5), J6.6 (Pin_6): now also R56.1; no longer J2.10, J2.11, J2.12
- new net GPIO3_A7: U25.3 (ON)
- new net VCC_3.3V: C83.1, J2.17, J2.18, J2.19, U25.5 (QOD), U25.6 (VOUT)
- new net VDD: J2.10, J2.11, J2.12, R56.2
- no-connect marks 12 -> 13
Other:
- moved on the sheet: J6

Commit message: preparing for motherboard v1.1
Parts:
- renumbered C84 to C49, C83 to C50, J2 to J15, J6 to J16, R56 to R49, U25 to U18
Changed lines of the file:
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@@
 (kicad_sch
-	(version 20240417)
+	(version 20241004)
 	(generator "eeschema")
 	(generator_version "8.99")
@@
 		(on_board yes)
 		(dnp no)
-		(property "Reference" "#PWR0166"
+		(property "Reference" "#PWR0105"
 			(at 116.84 119.38 0)
 			(effects
@@
 			(project "motherboard"
 				(path "/025fe4d1-0305-4b34-be04-f8d9818125a4/41516588-89d4-4c4a-8d7d-a4354a401e31"
-					(reference "#PWR0166")
+					(reference "#PWR0105")
 					(unit 1)
 				)
@@
 		(on_board yes)
 		(dnp no)
-		(property "Reference" "#PWR064"
+		(property "Reference" "#PWR0104"
 			(at 104.14 109.22 0)
 			(effects
@@
 			(project "motherboard"
 				(path "/025fe4d1-0305-4b34-be04-f8d9818125a4/41516588-89d4-4c4a-8d7d-a4354a401e31"
-					(reference "#PWR064")
+					(reference "#PWR0104")
 					(unit 1)
 				)
@@
 		(dnp no)
 		(fields_autoplaced yes)
-		(property "Reference" "#PWR056"
+		(property "Reference" "#PWR0102"
 			(at 102.87 104.14 0)
 			(effects
@@
 			(project "motherboard"
 				(path "/025fe4d1-0305-4b34-be04-f8d9818125a4/41516588-89d4-4c4a-8d7d-a4354a401e31"
-					(reference "#PWR056")
+					(reference "#PWR0102")
 					(unit 1)
 				)
@@
 		(dnp no)
 		(fields_autoplaced yes)
-		(property "Reference" "#PWR057"
+		(property "Reference" "#PWR0106"
 			(at 138.43 134.62 0)
 			(effects
@@
 			(project ""
 				(path "/025fe4d1-0305-4b34-be04-f8d9818125a4/41516588-89d4-4c4a-8d7d-a4354a401e31"
-					(reference "#PWR057")
+					(reference "#PWR0106")
 					(unit 1)
 				)
@@
 		(dnp no)
 		(fields_autoplaced yes)
-		(property "Reference" "#PWR0145"
+		(property "Reference" "#PWR0107"
 			(at 109.22 139.7 0)
 			(effects
@@
 			(project "motherboard"
 				(path "/025fe4d1-0305-4b34-be04-f8d9818125a4/41516588-89d4-4c4a-8d7d-a4354a401e31"
-					(reference "#PWR0145")
+					(reference "#PWR0107")
 					(unit 1)
 				)
@@
 		(dnp no)
 		(fields_autoplaced yes)
-		(property "Reference" "#PWR0164"
+		(property "Reference" "#PWR0101"
 			(at 54.61 104.14 0)
 			(effects
@@
 			(project "motherboard"
 				(path "/025fe4d1-0305-4b34-be04-f8d9818125a4/41516588-89d4-4c4a-8d7d-a4354a401e31"
-					(reference "#PWR0164")
+					(reference "#PWR0101")
 					(unit 1)
 				)
@@
 		(dnp no)
 		(fields_autoplaced yes)
-		(property "Reference" "J6"
+		(property "Reference" "J16"
 			(at 101.6 125.3743 0)
 			(effects
@@
 			(project ""
 				(path "/025fe4d1-0305-4b34-be04-f8d9818125a4/41516588-89d4-4c4a-8d7d-a4354a401e31"
-					(reference "J6")
+					(reference "J16")
 					(unit 1)
 				)
@@
 		(dnp no)
 		(fields_autoplaced yes)
-		(property "Reference" "U25"
+		(property "Reference" "U18"
 			(at 82.55 85.09 0)
 			(effects
@@
 			(project ""
 				(path "/025fe4d1-0305-4b34-be04-f8d9818125a4/41516588-89d4-4c4a-8d7d-a4354a401e31"
-					(reference "U25")
+					(reference "U18")
 					(unit 1)
 				)
@@
 		(dnp no)
 		(fields_autoplaced yes)
-		(property "Reference" "#PWR0163"
+		(property "Reference" "#PWR0100"
 			(at 54.61 96.52 0)
 			(effects
@@
 			(project "motherboard"
 				(path "/025fe4d1-0305-4b34-be04-f8d9818125a4/41516588-89d4-4c4a-8d7d-a4354a401e31"
-					(reference "#PWR0163")
+					(reference "#PWR0100")
 					(unit 1)
 				)
@@
 		(dnp no)
 		(fields_autoplaced yes)
-		(property "Reference" "C84"
+		(property "Reference" "C49"
 			(at 57.15 93.9862 0)
 			(effects
@@
 			(project "motherboard"
 				(path "/025fe4d1-0305-4b34-be04-f8d9818125a4/41516588-89d4-4c4a-8d7d-a4354a401e31"
-					(reference "C84")
+					(reference "C49")
 					(unit 1)
 				)
@@
 		(dnp no)
 		(fields_autoplaced yes)
-		(property "Reference" "C83"
+		(property "Reference" "C50"
 			(at 105.41 93.9862 0)
 			(effects
@@
 			(project "motherboard"
 				(path "/025fe4d1-0305-4b34-be04-f8d9818125a4/41516588-89d4-4c4a-8d7d-a4354a401e31"
-					(reference "C83")
+					(reference "C50")
 					(unit 1)
 				)
@@
 		(dnp no)
 		(fields_autoplaced yes)
-		(property "Reference" "R56"
+		(property "Reference" "R49"
 			(at 113.03 115.57 90)
 			(effects
@@
 			(project "motherboard"
 				(path "/025fe4d1-0305-4b34-be04-f8d9818125a4/41516588-89d4-4c4a-8d7d-a4354a401e31"
-					(reference "R56")
+					(reference "R49")
 					(unit 1)
 				)
@@
 		(dnp no)
 		(fields_autoplaced yes)
-		(property "Reference" "#PWR0165"
+		(property "Reference" "#PWR0103"
 			(at 82.55 109.22 0)
 			(effects
@@
 			(project "motherboard"
 				(path "/025fe4d1-0305-4b34-be04-f8d9818125a4/41516588-89d4-4c4a-8d7d-a4354a401e31"
-					(reference "#PWR0165")
+					(reference "#PWR0103")
 					(unit 1)
 				)
@@
 		(dnp no)
 		(fields_autoplaced yes)
-		(property "Reference" "#PWR0111"
+		(property "Reference" "#PWR0108"
 			(at 153.67 160.02 0)
 			(effects
@@
 			(project "motherboard"
 				(path "/025fe4d1-0305-4b34-be04-f8d9818125a4/41516588-89d4-4c4a-8d7d-a4354a401e31"
-					(reference "#PWR0111")
+					(reference "#PWR0108")
 					(unit 1)
 				)
@@
 		(dnp no)
 		(fields_autoplaced yes)
-		(property "Reference" "J2"
+		(property "Reference" "J15"
 			(at 170.18 100.3299 0)
 			(effects
@@
 			(project ""
 				(path "/025fe4d1-0305-4b34-be04-f8d9818125a4/41516588-89d4-4c4a-8d7d-a4354a401e31"
-					(reference "J2")
+					(reference "J15")
 					(unit 1)
 				)

Commit message: v1.0 tapeout and more
Parts:
- removed J16: OLED EL POWER, 6P_05mm_FPC:FPC-SMD_6P-P0.50_XUNPU_FPC-05F-6PH20, symbol Connector_Generic_MountingPin:Conn_01x06_MountingPin
- removed R49: 0R, Jumper:SolderJumper-2_P1.3mm_Open_TrianglePad1.0x1.5mm, symbol Device:R_Small
- added TP2: HPD, TestPoint:TestPoint_Pad_D1.5mm, symbol Connector:TestPoint
Connections:
- net GPIO3_B7: now also TP2.1
