File: motherboard/ext_usb2.0.kicad_sch (KiCad schematic)
At the start: 15 parts, among them J25 USB-231-ARY, U24 SY6280AAC, U25 TVS2200DRV, U26 TPD4E02B04

Commit message: cleanup and final mainboard tapeout
Connections:
- net USB_N: now reaches CMC3.1, J25.2 (D-)
- net USB_P: now reaches CMC3.2, J25.3 (D+)
Changed lines of the file:
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@@
-	)
-	(junction
-		(at 171.45 97.79)
-		(diameter 0)
-		(color 0 0 0 0)
 	)
 	(junction
@@
 	(wire
 		(pts
-			(xy 171.45 97.79) (xy 180.34 97.79)
-		)
-		(stroke
-			(width 0)
-			(type default)
-		)
-	)
-	(wire
-		(pts
 			(xy 123.19 105.41) (xy 123.19 104.14)
 		)
@@
 		)
 	)
+	(label "USB_P"
+		(at 90.17 102.87 180)
+		(fields_autoplaced yes)
+		(effects
+			(font
+				(size 1.27 1.27)
+			)
+			(justify right bottom)
+		)
+	)
 	(label "VBUS"
 		(at 135.89 124.46 0)
@@
 			)
 			(justify left bottom)
+		)
+	)
+	(label "USB_N"
+		(at 87.63 105.41 180)
+		(fields_autoplaced yes)
+		(effects
+			(font
+				(size 1.27 1.27)
+			)
+			(justify right bottom)
 		)
 	)
@@
 		(fields_autoplaced yes)
 		(effects
-			(font
-				(size 1.27 1.27)
-			)
-			(justify left)
-		)
-	)
-	(hierarchical_label "VBUS"
-		(shape bidirectional)
-		(at 180.34 97.79 0)
-		(fields_autoplaced yes)
-		(effects
