File: motherboard/pcie20-ekey.kicad_sch (KiCad schematic)
At the start: 7 parts, among them J13 Bus_M.2_Socket_E

Commit message: preparing for motherboard v1.1
Parts:
- renumbered C54 to C21, C78 to C22, C79 to C23, J13 to J8, R51 to R17, R50 to R18, R52 to R19
Connections:
- net GPIO3_D5/PWM11_M3/LCD_2_BL: now reaches J8.54 (~{W_DISABLE2})
- net GPIO3_D5/PWM11_M3/LCD_2_BL: now also J8.70 (UIM_POWER_SRC/GPIO1/~{PEWAKE1})
- net GPIO4_C4/MIPI_CAM1_RESET_L: now reaches J8.56 (~{W_DISABLE1})
- no-connect marks 23 -> 20
Other:
- note removed: "connect to usb hub"
Changed lines of the file:
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@@
 (kicad_sch
-	(version 20240417)
+	(version 20241004)
 	(generator "eeschema")
 	(generator_version "8.99")
@@
 		(comment 4 "Proof of concept board for feature verification")
 	)
-	(text "connect to usb hub"
-		(exclude_from_sim no)
-		(at 74.422 98.806 0)
-		(effects
-			(font
-				(size 1.27 1.27)
-			)
-		)
-	)
 	(text "below 3 pins are from coolpi\nrest are from radxa definition"
 		(exclude_from_sim no)
@@
 	)
 	(no_connect
-		(at 170.18 92.71)
-	)
-	(no_connect
 		(at 170.18 146.05)
 	)
@@
 	)
 	(no_connect
-		(at 170.18 90.17)
-	)
-	(no_connect
 		(at 170.18 130.81)
 	)
@@
 	)
 	(no_connect
-		(at 119.38 115.57)
-	)
-	(no_connect
 		(at 119.38 90.17)
 	)
@@
 	(wire
 		(pts
+			(xy 170.18 90.17) (xy 182.88 90.17)
+		)
+		(stroke
+			(width 0)
+			(type default)
+		)
+	)
+	(wire
+		(pts
 			(xy 119.38 52.07) (xy 123.19 52.07)
 		)
@@
 	(wire
 		(pts
-			(xy 110.49 64.77) (xy 119.38 64.77)
+			(xy 102.87 64.77) (xy 119.38 64.77)
 		)
 		(stroke
@@
 	(wire
 		(pts
+			(xy 102.87 115.57) (xy 119.38 115.57)
+		)
+		(stroke
+			(width 0)
+			(type default)
+		)
+	)
+	(wire
+		(pts
 			(xy 102.87 133.35) (xy 119.38 133.35)
 		)
@@
 	(wire
 		(pts
+			(xy 182.88 92.71) (xy 170.18 92.71)
+		)
+		(stroke
+			(width 0)
+			(type default)
+		)
+	)
+	(wire
+		(pts
 			(xy 102.87 80.01) (xy 119.38 80.01)
 		)
@@
 	(wire
 		(pts
-			(xy 110.49 69.85) (xy 119.38 69.85)
+			(xy 102.87 69.85) (xy 119.38 69.85)
 		)
 		(stroke
@@
 	(wire
 		(pts
-			(xy 110.49 67.31) (xy 119.38 67.31)
+			(xy 102.87 67.31) (xy 119.38 67.31)
 		)
 		(stroke
@@
 	(hierarchical_label "GPIO4_A1{slash}PEWAKE0"
 		(shape output)
-		(at 110.49 69.85 180)
+		(at 102.87 69.85 180)
 		(fields_autoplaced yes)
 		(effects
@@
 		)
 	)
+	(hierarchical_label "GPIO3_D5{slash}PWM11_M3{slash}LCD_2_BL"
+		(shape output)
+		(at 182.88 92.71 0)
+		(fields_autoplaced yes)
+		(effects
+			(font
+				(size 1.27 1.27)
+			)
+			(justify left)
+		)
+	)
 	(hierarchical_label "PCIE20_1_REFCLKP"
 		(shape input)
 		(at 102.87 143.51 180)
+		(fields_autoplaced yes)
+		(effects
+			(font
+				(size 1.27 1.27)
+			)
+			(justify right)
+		)
+	)
+	(hierarchical_label "GPIO3_D5{slash}PWM11_M3{slash}LCD_2_BL"
+		(shape output)
+		(at 102.87 115.57 180)
 		(fields_autoplaced yes)
 		(effects
@@
 	(hierarchical_label "GPIO4_A0{slash}CLKREQ0"
 		(shape output)
-		(at 110.49 67.31 180)
+		(at 102.87 67.31 180)
 		(fields_autoplaced yes)
 		(effects
@@
 		(shape input)
 		(at 182.88 100.33 0)
+		(fields_autoplaced yes)
+		(effects
+			(font
+				(size 1.27 1.27)
+			)
+			(justify left)
+		)
+	)
+	(hierarchical_label "GPIO4_C4{slash}MIPI_CAM1_RESET_L"
+		(shape input)
+		(at 182.88 90.17 0)
 		(fields_autoplaced yes)
 		(effects
@@
 	(hierarchical_label "GPIO4_A2{slash}PERST0"
 		(shape output)
-		(at 110.49 64.77 180)
+		(at 102.87 64.77 180)
 		(fields_autoplaced yes)
 		(effects
@@
 		(dnp no)
 		(fields_autoplaced yes)
-		(property "Reference" "C78"
+		(property "Reference" "C22"
 			(at 116.84 48.2662 0)
 			(effects
@@
 			(project "motherboard"
 				(path "/025fe4d1-0305-4b34-be04-f8d9818125a4/4296e3bb-d60d-4db1-b6b7-692bdef698b7"
-					(reference "C78")
+					(reference "C22")
 					(unit 1)
 				)
@@
 		(dnp no)
 		(fields_autoplaced yes)
-		(property "Reference" "C79"
+		(property "Reference" "C23"
 			(at 125.73 48.2662 0)
 			(effects
@@
 			(project "motherboard"
 				(path "/025fe4d1-0305-4b34-be04-f8d9818125a4/4296e3bb-d60d-4db1-b6b7-692bdef698b7"
-					(reference "C79")
+					(reference "C23")
 					(unit 1)
 				)
@@
 		(on_board yes)
 		(dnp no)
-		(property "Reference" "C54"
+		(property "Reference" "C21"
 			(at 96.52 48.2662 0)
 			(effects
@@
 			(project "motherboard"
 				(path "/025fe4d1-0305-4b34-be04-f8d9818125a4/4296e3bb-d60d-4db1-b6b7-692bdef698b7"
-					(reference "C54")
+					(reference "C21")
 					(unit 1)
 				)
@@
 		(dnp no)
 		(fields_autoplaced yes)
-		(property "Reference" "R51"
+		(property "Reference" "R17"
 			(at 173.99 100.33 90)
 			(effects
@@
 			(project "motherboard"
 				(path "/025fe4d1-0305-4b34-be04-f8d9818125a4/4296e3bb-d60d-4db1-b6b7-692bdef698b7"
-					(reference "R51")
+					(reference "R17")
 					(unit 1)
 				)
@@
 		(dnp no)
 		(fields_autoplaced yes)
-		(property "Reference" "R52"
+		(property "Reference" "R19"
 			(at 111.76 133.35 90)
 			(effects
@@
 			(project "motherboard"
 				(path "/025fe4d1-0305-4b34-be04-f8d9818125a4/4296e3bb-d60d-4db1-b6b7-692bdef698b7"
-					(reference "R52")
+					(reference "R19")
 					(unit 1)
 				)
@@
 		(dnp no)
 		(fields_autoplaced yes)
-		(property "Reference" "#PWR072"
+		(property "Reference" "#PWR044"
 			(at 144.78 162.56 0)
 			(effects
@@
 			(project ""
 				(path "/025fe4d1-0305-4b34-be04-f8d9818125a4/4296e3bb-d60d-4db1-b6b7-692bdef698b7"
-					(reference "#PWR072")
+					(reference "#PWR044")
 					(unit 1)
 				)
@@
 		(dnp no)
 		(fields_autoplaced yes)
-		(property "Reference" "J13"
+		(property "Reference" "J8"
 			(at 146.9741 57.15 0)
 			(effects
@@
 		)
 		(pin "20"
+		)
+		(instances
+			(project "motherboard"
+				(path "/025fe4d1-0305-4b34-be04-f8d9818125a4/4296e3bb-d60d-4db1-b6b7-692bdef698b7"
+					(reference "J8")
+					(unit 1)
+				)
+			)
 		)
 	)
@@
 		(dnp no)
 		(fields_autoplaced yes)
-		(property "Reference" "R50"
+		(property "Reference" "R18"
 			(at 179.07 102.87 90)
 			(effects
@@
 			(project "motherboard"
 				(path "/025fe4d1-0305-4b34-be04-f8d9818125a4/4296e3bb-d60d-4db1-b6b7-692bdef698b7"
-					(reference "R50")
+					(reference "R18")
 					(unit 1)
 				)
@@
 		(dnp no)
 		(fields_autoplaced yes)
-		(property "Reference" "#PWR0131"
+		(property "Reference" "#PWR043"
 			(at 119.38 58.42 0)
 			(effects
@@
 			(project "motherboard"
 				(path "/025fe4d1-0305-4b34-be04-f8d9818125a4/4296e3bb-d60d-4db1-b6b7-692bdef698b7"
-					(reference "#PWR0131")
+					(reference "#PWR043")
 					(unit 1)
 				)

Commit message: about to present!
about to present!
Other:
- note added: "BT_REG_ON_H"
- note added: "BT_WAKE_L"
- note added: "W_DISABLE"
Changed lines of the file:
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@@
+		)
+	)
+	(text "BT_REG_ON_H"
+		(exclude_from_sim no)
+		(at 220.218 75.184 0)
+		(effects
+			(font
+				(size 1.27 1.27)
+			)
 		)
 	)
@@
 		)
 	)
+	(text "W_DISABLE"
+		(exclude_from_sim no)
+		(at 222.758 90.424 0)
+		(effects
+			(font
+				(size 1.27 1.27)
+			)
+		)
+	)
+	(text "BT_WAKE_L"
+		(exclude_from_sim no)
+		(at 61.468 115.824 0)
+		(effects
+			(font
+				(size 1.27 1.27)
+			)
+		)
+	)
+	(text "BT_WAKE_L"
+		(exclude_from_sim no)
+		(at 223.012 92.964 0)
+		(effects
+			(font
+				(size 1.27 1.27)
+			)
+		)
+	)
