File: motherboard/sdcard.kicad_sch (KiCad schematic)
At the start: 9 parts, among them J14 Micro_SD_Card_Det1, U18 TPD4E02B04, U19 TPD4E02B04

Commit message: mainboard v0.3 + power WIP
Other:
- company: (none) -> Byran Huang
- title: (none) -> anyon e
Changed lines of the file:
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@@
 	(generator_version "8.99")
 	(paper "A4")
+	(title_block
+		(title "anyon e")
+		(date "2024-09-15")
+		(rev "V0.3")
+		(company "Byran Huang")
+		(comment 4 "Proof of concept board for feature verification")
+	)
 	(wire
 		(pts

Commit message: preparing for motherboard v1.1
Parts:
- renumbered J14 to J24, R57 to R80, R58 to R81, R59 to R82, R60 to R83, R61 to R84, R62 to R85, U18 to U22, U19 to U23
Changed lines of the file:
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@@
 (kicad_sch
-	(version 20240417)
+	(version 20241004)
 	(generator "eeschema")
 	(generator_version "8.99")
@@
 		(dnp no)
 		(fields_autoplaced yes)
-		(property "Reference" "#PWR079"
+		(property "Reference" "#PWR0156"
 			(at 101.6 144.78 0)
 			(effects
@@
 			(project "motherboard"
 				(path "/025fe4d1-0305-4b34-be04-f8d9818125a4/2b07758b-0d60-456c-9b9b-614b30378eb3"
-					(reference "#PWR079")
+					(reference "#PWR0156")
 					(unit 1)
 				)
@@
 		(dnp no)
 		(fields_autoplaced yes)
-		(property "Reference" "R58"
+		(property "Reference" "R81"
 			(at 114.3 71.12 90)
 			(effects
@@
 			(project "motherboard"
 				(path "/025fe4d1-0305-4b34-be04-f8d9818125a4/2b07758b-0d60-456c-9b9b-614b30378eb3"
-					(reference "R58")
+					(reference "R81")
 					(unit 1)
 				)
@@
 		(dnp no)
 		(fields_autoplaced yes)
-		(property "Reference" "R57"
+		(property "Reference" "R80"
 			(at 119.38 68.58 90)
 			(effects
@@
 			(project ""
 				(path "/025fe4d1-0305-4b34-be04-f8d9818125a4/2b07758b-0d60-456c-9b9b-614b30378eb3"
-					(reference "R57")
+					(reference "R80")
 					(unit 1)
 				)
@@
 		(dnp no)
 		(fields_autoplaced yes)
-		(property "Reference" "R62"
+		(property "Reference" "R85"
 			(at 113.03 91.44 90)
 			(effects
@@
 			(project "motherboard"
 				(path "/025fe4d1-0305-4b34-be04-f8d9818125a4/2b07758b-0d60-456c-9b9b-614b30378eb3"
-					(reference "R62")
+					(reference "R85")
 					(unit 1)
 				)
@@
 		(dnp no)
 		(fields_autoplaced yes)
-		(property "Reference" "J14"
+		(property "Reference" "J24"
 			(at 151.765 62.23 0)
 			(effects
@@
 			(project ""
 				(path "/025fe4d1-0305-4b34-be04-f8d9818125a4/2b07758b-0d60-456c-9b9b-614b30378eb3"
-					(reference "J14")
+					(reference "J24")
 					(unit 1)
 				)
@@
 		(dnp no)
 		(fields_autoplaced yes)
-		(property "Reference" "R61"
+		(property "Reference" "R84"
 			(at 107.95 86.36 90)
 			(effects
@@
 			(project "motherboard"
 				(path "/025fe4d1-0305-4b34-be04-f8d9818125a4/2b07758b-0d60-456c-9b9b-614b30378eb3"
-					(reference "R61")
+					(reference "R84")
 					(unit 1)
 				)
@@
 		(dnp no)
 		(fields_autoplaced yes)
-		(property "Reference" "R60"
+		(property "Reference" "R83"
 			(at 113.03 83.82 90)
 			(effects
@@
 			(project "motherboard"
 				(path "/025fe4d1-0305-4b34-be04-f8d9818125a4/2b07758b-0d60-456c-9b9b-614b30378eb3"
-					(reference "R60")
+					(reference "R83")
 					(unit 1)
 				)
@@
 		(dnp no)
 		(fields_autoplaced yes)
-		(property "Reference" "U19"
+		(property "Reference" "U23"
 			(at 148.59 113.03 0)
 			(effects
@@
 			(project "motherboard"
 				(path "/025fe4d1-0305-4b34-be04-f8d9818125a4/2b07758b-0d60-456c-9b9b-614b30378eb3"
-					(reference "U19")
+					(reference "U23")
 					(unit 1)
 				)
@@
 		(dnp no)
 		(fields_autoplaced yes)
-		(property "Reference" "#PWR077"
+		(property "Reference" "#PWR0154"
 			(at 123.19 106.68 0)
 			(effects
@@
 			(project ""
 				(path "/025fe4d1-0305-4b34-be04-f8d9818125a4/2b07758b-0d60-456c-9b9b-614b30378eb3"
-					(reference "#PWR077")
+					(reference "#PWR0154")
 					(unit 1)
 				)
@@
 		(dnp no)
 		(fields_autoplaced yes)
-		(property "Reference" "#PWR080"
+		(property "Reference" "#PWR0157"
 			(at 148.59 144.78 0)
 			(effects
@@
 			(project "motherboard"
 				(path "/025fe4d1-0305-4b34-be04-f8d9818125a4/2b07758b-0d60-456c-9b9b-614b30378eb3"
-					(reference "#PWR080")
+					(reference "#PWR0157")
 					(unit 1)
 				)
@@
 		(dnp no)
 		(fields_autoplaced yes)
-		(property "Reference" "#PWR078"
+		(property "Reference" "#PWR0155"
 			(at 171.45 106.68 0)
 			(effects
@@
 			(project "motherboard"
 				(path "/025fe4d1-0305-4b34-be04-f8d9818125a4/2b07758b-0d60-456c-9b9b-614b30378eb3"
-					(reference "#PWR078")
+					(reference "#PWR0155")
 					(unit 1)
 				)
@@
 		(dnp no)
 		(fields_autoplaced yes)
-		(property "Reference" "R59"
+		(property "Reference" "R82"
 			(at 109.22 73.66 90)
 			(effects
@@
 			(project "motherboard"
 				(path "/025fe4d1-0305-4b34-be04-f8d9818125a4/2b07758b-0d60-456c-9b9b-614b30378eb3"
-					(reference "R59")
+					(reference "R82")
 					(unit 1)
 				)
@@
 		(dnp no)
 		(fields_autoplaced yes)
-		(property "Reference" "U18"
+		(property "Reference" "U22"
 			(at 101.6 113.03 0)
 			(effects
@@
 			(project "motherboard"
 				(path "/025fe4d1-0305-4b34-be04-f8d9818125a4/2b07758b-0d60-456c-9b9b-614b30378eb3"
-					(reference "U18")
+					(reference "U22")
 					(unit 1)
 				)
