File: haptic/haptic.kicad_sch (KiCad schematic)
At the start: 0 parts

Commit message: haptics wip, created encoder pcb
Parts:
- added C1, C3, C4: 10uF, Capacitor_SMD:C_0805_2012Metric, symbol Device:C_Small
- added C11: 22uF, Capacitor_SMD:C_0805_2012Metric, symbol Device:C_Small
- added C12, C13, C18, C2, C20, C5: 0.1uF, Capacitor_SMD:C_0603_1608Metric, symbol Device:C_Small
- added C7: 1uF, Capacitor_SMD:C_0603_1608Metric, symbol Device:C_Small
- added J1: USB_C_Receptacle_USB2.0, GCT_USB:USB4510_NoPaste, symbol Connector:USB_C_Receptacle_USB2.0
- added J3: BLDC, Molex:532610371, symbol Connector:Conn_01x03_Male
- added Q1: UMH3N, Package_TO_SOT_SMD:SOT-363_SC-70-6, symbol Transistor_BJT:UMH3N
- added R1, R2: 5.1k, Resistor_SMD:R_0603_1608Metric, symbol Device:R_Small
- added R10, R13, R7, R9: 2.2k, Resistor_SMD:R_0603_1608Metric, symbol Device:R_Small
- added R11, R12, R3, R4, R5, R6, R8: 10k, Resistor_SMD:R_0603_1608Metric, symbol Device:R_Small
- added TP1: 5V, Modified:TestPoint_Pad_D2.0mm_ValueSilk, symbol Connector:TestPoint_Small
- added TP10: U, Modified:TestPoint_Pad_D2.0mm_ValueSilk, symbol Connector:TestPoint_Small
- added TP11: V, Modified:TestPoint_Pad_D2.0mm_ValueSilk, symbol Connector:TestPoint_Small
- added TP12: W, Modified:TestPoint_Pad_D2.0mm_ValueSilk, symbol Connector:TestPoint_Small
- added TP2: 3.3v, Modified:TestPoint_Pad_D2.0mm_ValueSilk, symbol Connector:TestPoint_Small
- added TP3: GND, Modified:TestPoint_Pad_D2.0mm_ValueSilk, symbol Connector:TestPoint_Small
- added TP4: TX, Modified:TestPoint_Pad_D2.0mm_ValueSilk, symbol Connector:TestPoint_Small
- added TP5: RX, Modified:TestPoint_Pad_D2.0mm_ValueSilk, symbol Connector:TestPoint_Small
- added TP6: EN, Modified:TestPoint_Pad_D2.0mm_ValueSilk, symbol Connector:TestPoint_Small
- added TP7: BOOT, Modified:TestPoint_Pad_D2.0mm_ValueSilk, symbol Connector:TestPoint_Small
- added TP8: SDA, Modified:TestPoint_Pad_D2.0mm_ValueSilk, symbol Connector:TestPoint_Small
- added TP9: SCL, Modified:TestPoint_Pad_D2.0mm_ValueSilk, symbol Connector:TestPoint_Small
- added U1: AP2114HA-3.3, Modified:SOT-223-3_TabPin2_InGndOut, symbol Regulator_Linear:AP7361C-33E
- added U2: TS1117BCW33_RPG, Modified:SOT-223-3_TabPin2_GndOutIn, symbol Regulator_Linear:TS1117BCW33_RPG
- added U3: T-Micro32_Plus, lilygo_micro32:T-Micro32, symbol lilygo_micro32:T-Micro32_Plus
- added U4: CH340C, Package_SO:SOIC-16_3.9x9.9mm_P1.27mm, symbol Interface_USB:CH340C
- added U7: TMC6300, Modified:QFN-20-1EP_3x3mm_P0.4mm_EP1.65x1.65mm_ThermalVias_LargerViaHoles, symbol Trinamic:TMC6300
Connections:
- new net: J3.1 (Pin_1), TP12.1, U7.1 (W)
- new net: J3.2 (Pin_2), TP11.1, U7.17 (V)
- new net: C20.1, U7.13 (1V8OUT)
- new net: J3.3 (Pin_3), TP10.1, U7.15 (U)
- new net: C13.2, U7.2 (VCP)
- new net +3V3: C1.1, C18.1, C2.1, C4.1, C5.1, R10.2, R13.1, R5.1, R7.1, R9.1, TP2.1, U1.3 (VO), U2.2 (Output), U3.2 (3V3), U4.16 (VCC), U4.4 (V3), U7.11 (VIO/~{STDBY})
- new net +5V: C11.1, C12.1, C13.1, C3.1, J1.A4 (VBUS), J1.A9 (VBUS), J1.B4 (VBUS), J1.B9 (VBUS), TP1.1, U1.1 (VI), U2.3 (Input), U7.18 (VS)
- new net DTR: Q1.2 (B1), Q1.4 (E2), U4.13 (~{DTR})
- new net ESP32_BOOT: Q1.3 (C2), TP7.1, U3.25 (IO0)
- new net ESP32_EN: C7.1, Q1.6 (C1), R5.2, TP6.1, U3.3 (EN)
- new net GND: C1.2, C11.2, C12.2, C18.2, C2.2, C20.2, C3.2, C4.2, C5.2, C7.2, J1.A1 (GND), J1.A12 (GND), J1.B1 (GND), J1.B12 (GND), J1.S1 (SHIELD), R1.2, R11.2, R12.2, R2.2, R3.2, R4.2, R6.2, R8.2, TP3.1, U1.2 (GND), U2.1 (GND), U3.1 (GND), U3.15 (GND), U3.38 (GND), U4.1 (GND), U7.14 (GND), U7.16 (BRUV), U7.20 (BRW), U7.8 (GND), U7.9 (GND), U7.PAD
- new net LCD_BACKLIGHT: U3.31 (IO19)
- new net LCD_CMD: U3.36 (IO22)
- new net LCD_CS: U3.33 (IO21)
- new net LCD_DATA: U3.29 (IO5)
- new net LCD_RST: U3.26 (IO4)
- new net LCD_SCK: U3.28 (IO20)
- new net LED_DATA_3V3: U3.21 (IO7)
- new net MAG_CLK: R10.1, U3.16 (IO13)
- new net MAG_CSN: U3.13 (IO14)
- new net MAG_DO: R9.2, U3.17 (IO37)
- new net RTS: Q1.1 (E1), Q1.5 (B2), U4.14 (~{RTS})
- new net SCL: R13.2, TP9.1, U3.22 (IO8)
- new net SDA: R7.2, TP8.1, U3.23 (IO15)
- new net STRAIN_DO: U3.18 (IO38)
- new net STRAIN_SCK: U3.24 (IO2)
- new net TMC_DIAG: U3.4 (IO36/SVP), U7.12 (DIAG)
- new net TMC_UH: R3.1, U3.11 (IO26), U7.3 (UH)
- new net TMC_UL: R8.1, U3.10 (IO25), U7.6 (UL)
- new net TMC_VH: R4.1, U3.12 (IO27), U7.4 (VH)
- new net TMC_VL: R12.1, U3.8 (IO32), U7.10 (VL)
- new net TMC_WH: R6.1, U3.14 (IO12), U7.5 (WH)
- new net TMC_WL: R11.1, U3.9 (IO33), U7.7 (WL)
- new net USB_CC1: J1.A5 (CC1), R1.1
- new net USB_CC2: J1.B5 (CC2), R2.1
- new net USB_D+: J1.A6 (D+), J1.B6 (D+), U4.5 (UD+)
- new net USB_D-: J1.A7 (D-), J1.B7 (D-), U4.6 (UD-)
- new net USB_SERIAL_RXI: TP4.1, U3.35 (TXD), U4.3 (RXD)
- new net USB_SERIAL_TXO: TP5.1, U3.34 (RXD), U4.2 (TXD)
- no-connect marks 0 -> 11
Other:
- note added: "Could put a sense resistor and sense amplifier here"
- note added: "GPIO12=MTDI. Should be 0 on boot for 3.3v built-in flash/psram on ESP32-PICO-v3-02"
- note added: "IO2 must be 0 to enter UART download mode"
- note added: "If your voltage regulator follows the 5V-GND-3V3 pinout (AP2114HA) populate your regulator on the footprint labled U6. If your regulator follows the pinout of GND-3V3-5V (TS1117BCW33) populate your regulator on the footprint labaled U9)."
- note added: "MCU - ESP32 (T-MICRO32 PLUS)"
- note added: "MOTOR DRIVER"
- note added: "POWER"
- note added: "PULLUPS, PULLDOWNS"
- note added: "Pull-ups on MT6701 allow for I2C (though we'll primarily use SSI)"
- note added: "Recommended 1uF-10uF on EN for auto-reset circuitry, per Espressif design notes."
- note added: "Reset/Boot via USB serial"
- note added: "USB"
- note added: "Use either U6 or U9, but not both!"
