File: keyboard/keyboard.kicad_pcb (KiCad board)
At the start: 0 parts

Commit message: keyboard v1 halfway routed
Parts:
- added AE1: Antenna, Mikoto-Footprints:2.4GHz-meander-antenna-v2, F.Cu at (134.7, 146.2)
- added C1: 4.7uF, Capacitor_SMD:C_0402_1005Metric, F.Cu at (134.9, 136.9)
- added C10: 1.5pF, Capacitor_SMD:C_0402_1005Metric, F.Cu at (141.6, 146.8)
- added C11: 1pF, Capacitor_SMD:C_0402_1005Metric, F.Cu at (141.6, 145.8)
- added C12: 1pF, Capacitor_SMD:C_0402_1005Metric, F.Cu at (142.5, 144.8)
- added C13: 4.7uF, Capacitor_SMD:C_0402_1005Metric, F.Cu at (136.7, 134.0)
- added C14: 1uF, Capacitor_SMD:C_0402_1005Metric, F.Cu at (127.8, 139.0)
- added C15: 1uF, Capacitor_SMD:C_0402_1005Metric, F.Cu at (125.8, 142.7)
- added C16: 100nF, Capacitor_SMD:C_0402_1005Metric, F.Cu at (147.6, 133.8)
- added C17: 100nF, Capacitor_SMD:C_0402_1005Metric, F.Cu at (147.9, 141.3)
- added C18: 100nF, Capacitor_SMD:C_0402_1005Metric, F.Cu at (135.0, 142.1)
- added C19: 4.7uF, Capacitor_SMD:C_0402_1005Metric, F.Cu at (135.5, 133.9)
- added C2: 1uF, Capacitor_SMD:C_0402_1005Metric, F.Cu at (144.4, 146.2)
- added C20: 1uF, Capacitor_SMD:C_0402_1005Metric, F.Cu at (135.0, 139.5)
- added C21: 15pF, Capacitor_SMD:C_0402_1005Metric, F.Cu at (147.8, 146.1)
- added C22: 15pF, Capacitor_SMD:C_0402_1005Metric, F.Cu at (148.0, 142.3)
- added C23: 10nF, Capacitor_SMD:C_0402_1005Metric, F.Cu at (130.0, 140.1)
- added C24: 1000pF/NC, Capacitor_SMD:C_0402_1005Metric, F.Cu at (273.3, 49.7)
- added C3: 47nF, Capacitor_SMD:C_0402_1005Metric, F.Cu at (148.4, 137.6)
- added C4: 4.7uF, Capacitor_SMD:C_0402_1005Metric, F.Cu at (134.9, 135.8)
- added C5: 1nF, Capacitor_SMD:C_0402_1005Metric, F.Cu at (135.0, 143.3)
- added C6: 100pF, Capacitor_SMD:C_0402_1005Metric, F.Cu at (145.4, 146.2)
- added C7: 100nF, Capacitor_SMD:C_0402_1005Metric, F.Cu at (146.4, 133.8)
- added C8: 15pF, Capacitor_SMD:C_0402_1005Metric, F.Cu at (144.7, 133.9)
- added C9: 15pF, Capacitor_SMD:C_0402_1005Metric, F.Cu at (140.9, 133.9)
- added D1: CHG, LED_SMD:LED_0603_1608Metric, F.Cu at (274.3, 45.4)
- added D10: D, Diode_SMD:D_SOD-523, F.Cu at (144.3, 47.2)
- added D11: D, Diode_SMD:D_SOD-523, F.Cu at (162.3, 47.2)
- added D12: D, Diode_SMD:D_SOD-523, F.Cu at (180.3, 47.2)
- added D13: D, Diode_SMD:D_SOD-523, F.Cu at (198.3, 47.2)
- added D14: D, Diode_SMD:D_SOD-523, F.Cu at (216.3, 47.2)
- added D15: D, Diode_SMD:D_SOD-523, F.Cu at (234.3, 47.2)
- added D16: D, Diode_SMD:D_SOD-523, F.Cu at (252.3, 47.2)
- added D18: D, Diode_SMD:D_SOD-523, F.Cu at (27.0, 65.2)
- added D19: D, Diode_SMD:D_SOD-523, F.Cu at (45.0, 65.2)
- added D2: B5819W SL, Diode_SMD:D_SOD-323, F.Cu at (121.7, 142.8)
- added D20: D, Diode_SMD:D_SOD-523, F.Cu at (63.0, 65.2)
- added D21: D, Diode_SMD:D_SOD-523, F.Cu at (81.0, 65.2)
- added D22: D, Diode_SMD:D_SOD-523, F.Cu at (99.0, 65.2)
- added D23: D, Diode_SMD:D_SOD-523, F.Cu at (117.0, 65.2)
- added D24: D, Diode_SMD:D_SOD-523, F.Cu at (135.0, 65.2)
- added D25: D, Diode_SMD:D_SOD-523, F.Cu at (153.0, 65.2)
- added D26: D, Diode_SMD:D_SOD-523, F.Cu at (171.0, 65.2)
- added D27: D, Diode_SMD:D_SOD-523, F.Cu at (189.0, 65.2)
- added D28: D, Diode_SMD:D_SOD-523, F.Cu at (207.0, 65.2)
- added D29: D, Diode_SMD:D_SOD-523, F.Cu at (225.0, 65.2)
- added D3: BLUE, LED_SMD:LED_0603_1608Metric, F.Cu at (272.5, 45.4)
- added D30: D, Diode_SMD:D_SOD-523, F.Cu at (243.0, 65.2)
- added D31: D, Diode_SMD:D_SOD-523, F.Cu at (265.5, 65.2)
- added D32: D, Diode_SMD:D_SOD-523, F.Cu at (31.7, 83.2)
- added D33: D, Diode_SMD:D_SOD-523, F.Cu at (54.2, 83.2)
- added D34: D, Diode_SMD:D_SOD-523, F.Cu at (72.2, 83.2)
- added D35: D, Diode_SMD:D_SOD-523, F.Cu at (90.2, 83.2)
- added D36: D, Diode_SMD:D_SOD-523, F.Cu at (108.2, 83.2)
- added D37: D, Diode_SMD:D_SOD-523, F.Cu at (126.2, 83.2)
- added D38: D, Diode_SMD:D_SOD-523, F.Cu at (144.2, 83.2)
- added D39: D, Diode_SMD:D_SOD-523, F.Cu at (162.2, 83.2)
- added D4: D, Diode_SMD:D_SOD-523, F.Cu at (31.8, 47.2)
- added D40: D, Diode_SMD:D_SOD-523, F.Cu at (180.2, 83.2)
- added D41: D, Diode_SMD:D_SOD-523, F.Cu at (198.2, 83.2)
- added D42: D, Diode_SMD:D_SOD-523, F.Cu at (216.2, 83.2)
- added D43: D, Diode_SMD:D_SOD-523, F.Cu at (234.2, 83.2)
- added D44: D, Diode_SMD:D_SOD-523, F.Cu at (252.2, 83.2)
- added D45: D, Diode_SMD:D_SOD-523, F.Cu at (270.2, 83.2)
- added D46: D, Diode_SMD:D_SOD-523, F.Cu at (34.2, 101.2)
- added D47: D, Diode_SMD:D_SOD-523, F.Cu at (59.0, 101.2)
- added D48: D, Diode_SMD:D_SOD-523, F.Cu at (77.0, 101.2)
- added D49: D, Diode_SMD:D_SOD-523, F.Cu at (95.0, 101.2)
- added D5: D, Diode_SMD:D_SOD-523, F.Cu at (54.3, 47.2)
- added D50: D, Diode_SMD:D_SOD-523, F.Cu at (113.0, 101.2)
- added D51: D, Diode_SMD:D_SOD-523, F.Cu at (130.9, 101.2)
- added D52: D, Diode_SMD:D_SOD-523, F.Cu at (148.9, 101.2)
- added D53: D, Diode_SMD:D_SOD-523, F.Cu at (166.9, 101.2)
- added D54: D, Diode_SMD:D_SOD-523, F.Cu at (184.9, 101.2)
- added D55: D, Diode_SMD:D_SOD-523, F.Cu at (202.9, 101.2)
- added D56: D, Diode_SMD:D_SOD-523, F.Cu at (220.9, 101.2)
- added D57: D, Diode_SMD:D_SOD-523, F.Cu at (238.9, 101.2)
- added D58: D, Diode_SMD:D_SOD-523, F.Cu at (263.7, 101.2)
- added D59: D, Diode_SMD:D_SOD-523, F.Cu at (38.6, 119.2)
- added D6: D, Diode_SMD:D_SOD-523, F.Cu at (72.3, 47.2)
- added D60: D, Diode_SMD:D_SOD-523, F.Cu at (67.8, 119.2)
- added D61: D, Diode_SMD:D_SOD-523, F.Cu at (85.8, 119.2)
- added D62: D, Diode_SMD:D_SOD-523, F.Cu at (103.8, 119.2)
- added D63: D, Diode_SMD:D_SOD-523, F.Cu at (121.8, 119.2)
- added D64: D, Diode_SMD:D_SOD-523, F.Cu at (139.8, 119.2)
- added D65: D, Diode_SMD:D_SOD-523, F.Cu at (157.8, 119.2)
- added D66: D, Diode_SMD:D_SOD-523, F.Cu at (175.8, 119.2)
- added D67: D, Diode_SMD:D_SOD-523, F.Cu at (193.8, 119.2)
- added D68: D, Diode_SMD:D_SOD-523, F.Cu at (211.8, 119.2)
- added D69: D, Diode_SMD:D_SOD-523, F.Cu at (229.8, 119.2)
- added D7: D, Diode_SMD:D_SOD-523, F.Cu at (90.3, 47.2)
- added D70: D, Diode_SMD:D_SOD-523, F.Cu at (247.8, 119.2)
- added D71: D, Diode_SMD:D_SOD-523, F.Cu at (268.1, 119.2)
- added D72: D, Diode_SMD:D_SOD-523, F.Cu at (27.2, 137.2)
- added D73: D, Diode_SMD:D_SOD-523, F.Cu at (45.2, 137.2)
- added D74: D, Diode_SMD:D_SOD-523, F.Cu at (63.2, 137.2)
- added D75: D, Diode_SMD:D_SOD-523, F.Cu at (83.5, 137.2)
- added D76: D, Diode_SMD:D_SOD-523, F.Cu at (113.0, 137.2)
- added D77: D, Diode_SMD:D_SOD-523, F.Cu at (166.8, 137.2)
- added D78: D, Diode_SMD:D_SOD-523, F.Cu at (196.2, 137.2)
- added D79: D, Diode_SMD:D_SOD-523, F.Cu at (216.5, 137.2)
- added D8: D, Diode_SMD:D_SOD-523, F.Cu at (108.3, 47.2)
- added D80: D, Diode_SMD:D_SOD-523, F.Cu at (234.5, 137.2)
- added D81: D, Diode_SMD:D_SOD-523, F.Cu at (252.5, 137.2)
- added D82: D, Diode_SMD:D_SOD-523, F.Cu at (270.5, 137.2)
- added D9: D, Diode_SMD:D_SOD-523, F.Cu at (126.3, 47.2)
- added F1: 500mA, Fuse:Fuse_0402_1005Metric, F.Cu at (124.4, 142.7)
- added J1: Pico-EZmate, Connector_Molex:Molex_Pico-EZmate_78171-0002_1x02-1MP_P1.20mm_Vertical, B.Cu at (125.7, 132.8)
- added J2: USB2.0, Connector_USB:USB_C_Receptacle_HRO_TYPE-C-31-M-12, F.Cu at (266.1, 47.8)
- added J3: Debug, Connector_PinHeader_2.54mm:PinHeader_1x04_P2.54mm_Vertical, B.Cu at (181.1, 145.0)
- added K1: Esc, Cherry_ULP:Cherry_ULP_SMD, F.Cu at (31.3, 50.2)
- added K10: F9, Cherry_ULP:Cherry_ULP_SMD, F.Cu at (197.8, 50.2)
- added K11: F10, Cherry_ULP:Cherry_ULP_SMD, F.Cu at (215.8, 50.2)
- added K12: F11, Cherry_ULP:Cherry_ULP_SMD, F.Cu at (233.8, 50.2)
- added K13: F12, Cherry_ULP:Cherry_ULP_SMD, F.Cu at (251.8, 50.2)
- added K15: ~~,`, Cherry_ULP:Cherry_ULP_SMD, F.Cu at (26.8, 68.2)
- added K16: !,1, Cherry_ULP:Cherry_ULP_SMD, F.Cu at (44.8, 68.2)
- added K17: @,2, Cherry_ULP:Cherry_ULP_SMD, F.Cu at (62.8, 68.2)
- added K18: #,3, Cherry_ULP:Cherry_ULP_SMD, F.Cu at (80.8, 68.2)
- added K19: $,4, Cherry_ULP:Cherry_ULP_SMD, F.Cu at (98.8, 68.2)
- added K2: F1, Cherry_ULP:Cherry_ULP_SMD, F.Cu at (53.8, 50.2)
- added K20: %,5, Cherry_ULP:Cherry_ULP_SMD, F.Cu at (116.8, 68.2)
- added K21: ^,6, Cherry_ULP:Cherry_ULP_SMD, F.Cu at (134.8, 68.2)
- added K22: &,7, Cherry_ULP:Cherry_ULP_SMD, F.Cu at (152.8, 68.2)
- added K23: *,8, Cherry_ULP:Cherry_ULP_SMD, F.Cu at (170.8, 68.2)
- added K24: (,9, Cherry_ULP:Cherry_ULP_SMD, F.Cu at (188.8, 68.2)
- added K25: ),0, Cherry_ULP:Cherry_ULP_SMD, F.Cu at (206.8, 68.2)
- added K26: _,-, Cherry_ULP:Cherry_ULP_SMD, F.Cu at (224.8, 68.2)
- added K27: +,=, Cherry_ULP:Cherry_ULP_SMD, F.Cu at (242.8, 68.2)
- added K28: Backspace, Cherry_ULP:Cherry_ULP_SMD, F.Cu at (265.3, 68.2)
- added K29: Tab, Cherry_ULP:Cherry_ULP_SMD, F.Cu at (31.3, 86.2)
- added K3: F2, Cherry_ULP:Cherry_ULP_SMD, F.Cu at (71.8, 50.2)
- added K30: Q, Cherry_ULP:Cherry_ULP_SMD, F.Cu at (53.8, 86.2)
- added K31: W, Cherry_ULP:Cherry_ULP_SMD, F.Cu at (71.8, 86.2)
- added K32: E, Cherry_ULP:Cherry_ULP_SMD, F.Cu at (89.8, 86.2)
- added K33: R, Cherry_ULP:Cherry_ULP_SMD, F.Cu at (107.8, 86.2)
- added K34: T, Cherry_ULP:Cherry_ULP_SMD, F.Cu at (125.8, 86.2)
- added K35: Y, Cherry_ULP:Cherry_ULP_SMD, F.Cu at (143.8, 86.2)
- added K36: U, Cherry_ULP:Cherry_ULP_SMD, F.Cu at (161.8, 86.2)
- added K37: I, Cherry_ULP:Cherry_ULP_SMD, F.Cu at (179.8, 86.2)
- added K38: O, Cherry_ULP:Cherry_ULP_SMD, F.Cu at (197.8, 86.2)
- added K39: P, Cherry_ULP:Cherry_ULP_SMD, F.Cu at (215.8, 86.2)
- added K4: F3, Cherry_ULP:Cherry_ULP_SMD, F.Cu at (89.8, 50.2)
- added K40: {,[, Cherry_ULP:Cherry_ULP_SMD, F.Cu at (233.8, 86.2)
- added K41: },], Cherry_ULP:Cherry_ULP_SMD, F.Cu at (251.8, 86.2)
- added K42: |,\, Cherry_ULP:Cherry_ULP_SMD, F.Cu at (269.8, 86.2)
- added K43: Caps Lock, Cherry_ULP:Cherry_ULP_SMD, F.Cu at (33.5, 104.2)
- added K44: A, Cherry_ULP:Cherry_ULP_SMD, F.Cu at (58.3, 104.2)
- added K45: S, Cherry_ULP:Cherry_ULP_SMD, F.Cu at (76.3, 104.2)
- added K46: D, Cherry_ULP:Cherry_ULP_SMD, F.Cu at (94.3, 104.2)
- added K47: F, Cherry_ULP:Cherry_ULP_SMD, F.Cu at (112.3, 104.2)
- added K48: G, Cherry_ULP:Cherry_ULP_SMD, F.Cu at (130.3, 104.2)
- added K49: H, Cherry_ULP:Cherry_ULP_SMD, F.Cu at (148.3, 104.2)
- added K5: F4, Cherry_ULP:Cherry_ULP_SMD, F.Cu at (107.8, 50.2)
- added K50: J, Cherry_ULP:Cherry_ULP_SMD, F.Cu at (166.3, 104.2)
- added K51: K, Cherry_ULP:Cherry_ULP_SMD, F.Cu at (184.3, 104.2)
- added K52: L, Cherry_ULP:Cherry_ULP_SMD, F.Cu at (202.3, 104.2)
- added K53: :,;, Cherry_ULP:Cherry_ULP_SMD, F.Cu at (220.3, 104.2)
- added K54: ",', Cherry_ULP:Cherry_ULP_SMD, F.Cu at (238.3, 104.2)
- added K55: Enter, Cherry_ULP:Cherry_ULP_SMD, F.Cu at (263.1, 104.2)
- added K56: Shift, Cherry_ULP:Cherry_ULP_SMD, F.Cu at (38.0, 122.2)
- added K57: Z, Cherry_ULP:Cherry_ULP_SMD, F.Cu at (67.3, 122.2)
- added K58: X, Cherry_ULP:Cherry_ULP_SMD, F.Cu at (85.3, 122.2)
- added K59: C, Cherry_ULP:Cherry_ULP_SMD, F.Cu at (103.3, 122.2)
- added K6: F5, Cherry_ULP:Cherry_ULP_SMD, F.Cu at (125.8, 50.2)
- added K60: V, Cherry_ULP:Cherry_ULP_SMD, F.Cu at (121.3, 122.2)
- added K61: B, Cherry_ULP:Cherry_ULP_SMD, F.Cu at (139.3, 122.2)
- added K62: N, Cherry_ULP:Cherry_ULP_SMD, F.Cu at (157.3, 122.2)
- added K63: M, Cherry_ULP:Cherry_ULP_SMD, F.Cu at (175.3, 122.2)
- added K64: <,,, Cherry_ULP:Cherry_ULP_SMD, F.Cu at (193.3, 122.2)
- added K65: >,., Cherry_ULP:Cherry_ULP_SMD, F.Cu at (211.3, 122.2)
- added K66: ?,/, Cherry_ULP:Cherry_ULP_SMD, F.Cu at (229.3, 122.2)
- added K67: ↑, Cherry_ULP:Cherry_ULP_SMD, F.Cu at (247.3, 122.2)
- added K68: Shift, Cherry_ULP:Cherry_ULP_SMD, F.Cu at (267.6, 122.2)
- added K69: Fn, Cherry_ULP:Cherry_ULP_SMD, F.Cu at (26.8, 140.2)
- added K7: F6, Cherry_ULP:Cherry_ULP_SMD, F.Cu at (143.8, 50.2)
- added K70: Ctrl, Cherry_ULP:Cherry_ULP_SMD, F.Cu at (44.8, 140.2)
- added K71: Alt, Cherry_ULP:Cherry_ULP_SMD, F.Cu at (62.8, 140.2)
- added K72: Meta, Cherry_ULP:Cherry_ULP_SMD, F.Cu at (83.0, 140.2)
- added K73: Space, Cherry_ULP:Cherry_ULP_SMD, F.Cu at (112.5, 140.2)
- added K74: Space, Cherry_ULP:Cherry_ULP_SMD, F.Cu at (166.1, 140.2)
- added K75: Meta, Cherry_ULP:Cherry_ULP_SMD, F.Cu at (195.6, 140.2)
- added K76: Alt, Cherry_ULP:Cherry_ULP_SMD, F.Cu at (215.8, 140.2)
- added K77: ←, Cherry_ULP:Cherry_ULP_SMD, F.Cu at (233.8, 140.2)
- added K78: ↓, Cherry_ULP:Cherry_ULP_SMD, F.Cu at (251.8, 140.2)
- added K79: →, Cherry_ULP:Cherry_ULP_SMD, F.Cu at (269.8, 140.2)
- added K8: F7, Cherry_ULP:Cherry_ULP_SMD, F.Cu at (161.8, 50.2)
- added K9: F8, Cherry_ULP:Cherry_ULP_SMD, F.Cu at (179.8, 50.2)
- added L1: 15nH, Inductor_SMD:L_0402_1005Metric, F.Cu at (149.9, 137.1)
- added L2: 10uH, Inductor_SMD:L_0603_1608Metric, F.Cu at (149.3, 135.8)
- added L3: 10uH, Inductor_SMD:L_0603_1608Metric, F.Cu at (138.8, 134.1)
- added L4: 3.9nH, Inductor_SMD:L_0402_1005Metric, F.Cu at (140.4, 144.7)
- added NT1: NetTie_2, Mikoto-Footprints:net-tie-2-tiny, F.Cu at (142.8, 142.0)
- added R1: 0R, Resistor_SMD:R_0402_1005Metric, F.Cu at (139.9, 146.3)
- added R10: 10M, Resistor_SMD:R_0402_1005Metric, F.Cu at (130.0, 141.2)
- added R11: 1M, Resistor_SMD:R_0402_1005Metric, F.Cu at (272.2, 49.7)
- added R2: 10k, Resistor_SMD:R_0402_1005Metric, F.Cu at (127.4, 137.4)
- added R3: 10k, Resistor_SMD:R_0402_1005Metric, F.Cu at (122.7, 140.0)
- added R4: 10k, Resistor_SMD:R_0402_1005Metric, F.Cu at (127.8, 140.1)
- added R5: 1.5k, Resistor_SMD:R_0402_1005Metric, F.Cu at (272.8, 47.9)
- added R6: 5.1k, Resistor_SMD:R_0402_1005Metric, F.Cu at (272.9, 52.0)
- added R7: 5.1k, Resistor_SMD:R_0402_1005Metric, F.Cu at (272.8, 55.8)
- added R8: 2M, Resistor_SMD:R_0402_1005Metric, F.Cu at (128.4, 137.4)
- added R9: 2M, Resistor_SMD:R_0402_1005Metric, F.Cu at (130.0, 139.0)
- added SW1: Reset, Button_Switch_SMD:SW_Push_1P1T_XKB_TS-1187A, F.Cu at (266.0, 57.2)
- added U1: BQ21040DBVR, BQ21040:SOT95P280X145-6N, F.Cu at (125.1, 138.9)
- added U2: nRF52840, Package_DFN_QFN:Nordic_AQFN-73-1EP_7x7mm_P0.5mm, F.Cu at (141.3, 139.5)
- added U3: ESDR0502NMUTAG, Mikoto-Footprints:UDFN-6_1.2x1.0mm_P0.4mm, F.Cu at (272.6, 53.9)
- added Y1: 32.768 kHz, Crystal:Crystal_SMD_2012-2Pin_2.0x1.2mm, F.Cu at (142.8, 133.9)
- added Y2: 32MHz, Crystal:Crystal_SMD_2016-4Pin_2.0x1.6mm, F.Cu at (147.6, 144.2)
Routing:
- net VBUS: track 0.00 -> 253.0 mm, vias 0 -> 3
- net /Key Matrix/Row_2: track 0.00 -> 249.9 mm, vias 0 -> 14
- net /Key Matrix/Row_1: track 0.00 -> 248.7 mm, vias 0 -> 14
- net /Key Matrix/Row_3: track 0.00 -> 244.2 mm, vias 0 -> 13
- net /Key Matrix/Row_4: track 0.00 -> 244.1 mm, vias 0 -> 13
- net /Key Matrix/Row_0: track 0.00 -> 231.3 mm, vias 0 -> 13
- net /Key Matrix/Row_5: track 0.00 -> 201.2 mm, vias 0 -> 11
- net /Key Matrix/Col_8: track 0.00 -> 143.4 mm, vias 0 -> 2
- net /Key Matrix/Col_10: track 0.00 -> 143.3 mm, vias 0 -> 2
- net /Key Matrix/Col_7: track 0.00 -> 142.2 mm, vias 0 -> 2
- net /Key Matrix/Col_6: track 0.00 -> 141.9 mm, vias 0 -> 2
- net /Key Matrix/Col_9: track 0.00 -> 141.8 mm, vias 0 -> 2
- net /Key Matrix/Col_5: track 0.00 -> 136.6 mm, vias 0 -> 2
- net /Key Matrix/Col_3: track 0.00 -> 120.2 mm
- net /Key Matrix/Col_2: track 0.00 -> 119.6 mm
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- added copper zone on B.Cu, net GND
- added copper zone on F.Cu, net GND
Other:
- copper layers 0 -> 2

Commit message: fully routed and fixed
Parts:
- removed J2: USB2.0, Connector_USB:USB_C_Receptacle_HRO_TYPE-C-31-M-12
- added P1: USB-C, Connector_USB:USB_C_Receptacle_HRO_TYPE-C-31-M-12, F.Cu at (266.1, 47.8)
- moved R7 11.3 mm to (261.7, 53.8), turned to 180 degrees
- moved D2 10.3 mm to (123.9, 132.7)
- moved AE1 4.58 mm to (130.3, 145.1)
- moved C10 4.21 mm to (137.4, 146.5)
- moved R1 2.82 mm to (137.4, 145.0), turned to 180 degrees
- moved C9 2.31 mm to (142.7, 132.5), turned to 180 degrees
- moved C13 1.96 mm to (138.6, 134.2), turned to 180 degrees
- moved C3 1.68 mm to (146.8, 137.1)
- moved C23 1.62 mm to (128.8, 141.2)
- moved R10 1.55 mm to (128.8, 142.2)
- moved L3 1.28 mm to (138.3, 132.9)
- moved C11 1.24 mm to (140.4, 146.1)
- moved R9 1.20 mm to (129.5, 137.9), turned to -90 degrees
- moved C1 1.08 mm to (135.8, 136.3)
- moved SW1 1.04 mm to (265.0, 57.5)
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Connections:
- U2 pad B13: BAT_VOLT -> unconnected-(U2-AIN1/P0.03-PadB13)
- U2 pad J1: /Key Matrix/Col_0 -> BAT_VOLT
- U2 pad U1: unconnected-(U2-TRACEDATA1/P0.12-PadU1) -> /Key Matrix/Col_0
Routing:
- net BLUE_LED: track 0.00 -> 257.2 mm, vias 0 -> 2
- net RESET: track 0.00 -> 242.3 mm, vias 0 -> 6
- net USB_D+: track 0.00 -> 242.3 mm, vias 0 -> 2
- net USB_D-: track 0.00 -> 241.1 mm, vias 0 -> 4
- net /Key Matrix/Col_13: track 19.9 -> 260.9 mm, vias 0 -> 4
- net Net-(D1-K): track 0.00 -> 240.2 mm, vias 0 -> 4
- net Net-(D1-A): track 0.00 -> 239.7 mm, vias 0 -> 4
- net /Key Matrix/Col_10: track 143.3 -> 308.0 mm, vias 2 -> 6
- net /Key Matrix/Col_11: track 85.0 -> 242.8 mm, vias 0 -> 4
- net /Key Matrix/Col_12: track 86.0 -> 232.6 mm, vias 0 -> 2
- net /Key Matrix/Col_0: track 101.2 -> 221.6 mm, vias 0 -> 2
- net /Key Matrix/Col_1: track 116.3 -> 227.8 mm, vias 0 -> 2
- net SWC: track 0.00 -> 110.7 mm, vias 0 -> 4
- net /Key Matrix/Row_0: track 231.3 -> 340.6 mm
- net SWD: track 0.00 -> 103.5 mm, vias 0 -> 4
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
Commit message: trackpad solutions
Parts:
- moved U3 3.40 mm to (276.0, 53.9)
- moved C24 3.24 mm to (276.5, 49.2)
- moved R6 3.01 mm to (275.9, 52.2)
- moved R11 2.96 mm to (275.1, 49.1)
- moved D3 2.40 mm to (274.9, 45.4)
- moved R5 2.32 mm to (275.1, 47.6)
- moved D1 2.20 mm to (276.5, 45.4)
Routing:
- net Net-(P1-SHIELD): track 20.0 -> 23.5 mm
- net VBUS: track 283.6 -> 287.0 mm
- net USB_D+: track 242.3 -> 245.7 mm
- net USB_D-: track 241.1 -> 244.5 mm
- net /nRF52840/CC1: track 6.80 -> 9.72 mm
- net BLUE_LED: track 257.2 -> 259.6 mm
- net Net-(D1-A): track 239.7 -> 241.1 mm
- net Net-(D1-K): track 240.2 -> 241.1 mm
- net GND: vias 20 -> 99

Commit message: implemented most features
Changed lines of the file:
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@@
+	)
+	(segment
+		(start 140.25 143.540581)
+		(end 140.25 133.792209)
+		(width 0.2)
+		(layer "B.Cu")
+		(net 44)
 	)
 	(segment
@@
 	)
 	(segment
-		(start 139.848737 137.751263)
-		(end 140.027 137.573)
-		(width 0.2)
-		(layer "B.Cu")
-		(net 44)
-	)
-	(segment
-		(start 140.027 133.569209)
-		(end 139.9 133.442209)
-		(width 0.2)
-		(layer "B.Cu")
-		(net 44)
-	)
-	(segment
 		(start 172.2 116.3)
 		(end 209.8 116.3)
@@
 	)
 	(segment
-		(start 140.232182 143.558399)
-		(end 140.232182 138.134708)
+		(start 140.17154 143.619041)
+		(end 140.25 143.540581)
 		(width 0.2)
 		(layer "B.Cu")
@@
 	)
 	(segment
-		(start 140.027 137.573)
-		(end 140.027 133.569209)
+		(start 140.25 133.792209)
+		(end 139.9 133.442209)
 		(width 0.2)
 		(layer "B.Cu")
@@
 		(width 0.2)
 		(layer "B.Cu")
-		(net 44)
-	)
-	(segment
-		(start 140.17154 143.619041)
-		(end 140.232182 143.558399)
-		(width 0.2)
-		(layer "B.Cu")
-		(net 44)
-	)
-	(segment
-		(start 140.232182 138.134708)
-		(end 139.848737 137.751263)
-		(width 0.2)
-		(layer "B.Cu")

Commit message: CAD work + documentation
Routing:
- net GND: track 30.3 -> 30.9 mm, vias 99 -> 104
Other:
- board outline added: 258.4 x 104.6 mm

Commit message: keyboard battery and pogo pin system
Parts:
- added J2: USB POGO, Connector_PinHeader_2.54mm:PinHeader_1x04_P2.54mm_Vertical, F.Cu at (274.5, 101.0)
- J1: value Pico-EZmate -> BATT; footprint Connector_Molex:Molex_Pico-EZmate_78171-0002_1x02-1MP_P1.20mm_Vertical -> Connector_PinHeader_2.54mm:PinHeader_1x02_P2.54mm_Vertical; moved to F.Cu
- J3: moved to F.Cu
- R3: value 10k -> 2.7k
- moved J1 23.9 mm to (103.3, 141.3), turned to 180 degrees
- moved SW1 4.03 mm to (268.9, 58.5)
- moved D2 3.72 mm to (122.8, 136.2), turned to 90 degrees
- moved U3 1.30 mm to (274.7, 53.9)
- turned J3 to 180 degrees
Connections:
- P1 pad B6: (no net) -> USB_D+
- P1 pad B7: (no net) -> USB_D-
Routing:
- net VBUS: track 287.0 -> 345.7 mm, vias 7 -> 6
- net /Key Matrix/Col_1: track 227.8 -> 257.2 mm
- net /Key Matrix/Col_12: track 232.6 -> 259.8 mm
- net /Key Matrix/Col_10: track 308.0 -> 334.3 mm, vias 6 -> 8
- net /Key Matrix/Col_6: track 166.3 -> 191.3 mm
- net /Key Matrix/Col_8: track 218.6 -> 243.1 mm
- net VBAT: track 26.2 -> 49.8 mm, vias 3 -> 2
- net /Key Matrix/Col_13: track 260.9 -> 280.9 mm, vias 4 -> 2
- net /Key Matrix/Col_2: track 216.6 -> 229.7 mm, vias 2 -> 4
- net /Key Matrix/Col_3: track 200.8 -> 211.9 mm, vias 2 -> 4
- net /Key Matrix/Col_4: track 171.8 -> 182.4 mm, vias 2 -> 4
- net USB_D+: track 245.7 -> 255.8 mm
- net USB_D-: track 244.5 -> 251.1 mm
- net Net-(D2-K): track 11.7 -> 6.12 mm
- net /Key Matrix/Col_9: track 242.8 -> 245.1 mm, vias 9 -> 10
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Other:
- outline, holes or cut-outs redrawn
- board text added: "BATTERY >"
- board text added: "PROTECTOR"
