File: keyboard/key_matrix.kicad_sch (KiCad schematic)
At the start: 156 parts, among them K1 Esc, K10 F9, K11 F10, K12 F11, K13 F12, K15 ~~,`, K16 !,1, K17 @,2, K18 #,3, K19 $,4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

Commit message: TAPEOUT: keyboard + protector, display + halls switch eval
Parts:
- D10, D11, D12, D13, D14, D15, D16, D18, D19, D20, D21, D22, D23, D24, D25, D26, D27, D28, D29, D30, D31, D32, D33, D34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: LCSC (none) -> C7420320
