File: keyboard/nRF52840.kicad_sch (KiCad schematic)
At the start: 54 parts, among them J1 Pico-EZmate, J2 USB2.0, J3 Debug, SW1 Reset, U1 BQ21040DBVR, U2 nRF52840, U3 ESDR0502NMUTAG, Y1 32.768 kHz, Y2 32MHz

Commit message: fully routed and fixed
Parts:
- removed J2: USB2.0, Connector_USB:USB_C_Receptacle_HRO_TYPE-C-31-M-12, symbol mikoto:USB_C_Receptacle_USB2.0
- added P1: USB-C, Connector_USB:USB_C_Receptacle_HRO_TYPE-C-31-M-12, symbol Connector:USB_C_Plug_USB2.0
Connections:
- net BAT_VOLT: now also U2.J1 (AIN2/P0.04); no longer U2.B13 (AIN1/P0.03)
- net CC1: now also P1.A5 (CC)
- net CC2: now also P1.B5 (VCONN)
- net Col_0: now also U2.U1 (TRACEDATA1/P0.12); no longer U2.J1 (AIN2/P0.04)
- net GND: now also P1.A1 (GND), P1.A12 (GND), P1.B1 (GND), P1.B12 (GND)
- net USB_D+: now also P1.A6 (D+)
- net USB_D-: now also P1.A7 (D-)
- net VBUS: now also P1.A4 (VBUS), P1.A9 (VBUS), P1.B4 (VBUS), P1.B9 (VBUS)
- net at C24.1, R11.2: now also P1.S1 (SHIELD)
- no-connect marks 25 -> 23
Other:
- moved on the sheet: C24, R11, R6, R7

Commit message: keyboard battery and pogo pin system
Parts:
- added J2: USB POGO, Connector_PinHeader_2.54mm:PinHeader_1x04_P2.54mm_Vertical, symbol Connector_Generic:Conn_01x04
- J1: value Pico-EZmate -> BATT; footprint Connector_Molex:Molex_Pico-EZmate_78171-0002_1x02-1MP_P1.20mm_Vertical -> Connector_PinHeader_2.54mm:PinHeader_1x02_P2.54mm_Vertical; now not fitted; now left out of the parts list
- J3: now not fitted; now left out of the parts list
- R3: value 10k -> 2.7k
Connections:
- net GND: now also J2.4 (Pin_4)
- net USB_D+: now also P1.B6 (D+), J2.2 (Pin_2)
- net USB_D-: now also P1.B7 (D-), J2.3 (Pin_3)
- net VBUS: now also J2.1 (Pin_1)
Other:
- note added: "ISET: 540/2700 = 200mA"
- note removed: "ISET: 54mA"
Changed lines of the file:
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@@
 		)
 	)
-	(text "ISET: 54mA"
+	(text "ISET: 540/2700 = 200mA"
 		(exclude_from_sim no)
-		(at 266.192 141.224 0)
+		(at 260.096 141.732 0)
 		(effects
 			(font
@@
 		)
 	)
+	(global_label "USB_D-"
+		(shape input)
+		(at 326.39 179.07 180)
+		(fields_autoplaced yes)
+		(effects
+			(font
+				(size 1.27 1.27)
+			)
+			(justify right)
+		)
+		(property "Intersheetrefs" "${INTERSHEET_REFS}"
+			(at 315.7848 179.07 0)
+			(effects
+				(font
+					(size 1.27 1.27)
+				)
+				(justify right)
+				(hide yes)
+			)
+		)
+	)
 	(global_label "SWC"
 		(shape input)
@@
 		)
 	)
+	(global_label "VBUS"
+		(shape input)
+		(at 326.39 173.99 180)
+		(fields_autoplaced yes)
+		(effects
+			(font
+				(size 1.27 1.27)
+			)
+			(justify right)
+		)
+		(property "Intersheetrefs" "${INTERSHEET_REFS}"
+			(at 318.5062 173.99 0)
+			(effects
+				(font
+					(size 1.27 1.27)
+				)
+				(justify right)
+				(hide yes)
+			)
+		)
+	)
 	(global_label "VBAT"
 		(shape input)
@@
 		)
 	)
+	(global_label "USB_D+"
+		(shape input)
+		(at 326.39 176.53 180)
+		(fields_autoplaced yes)
+		(effects
+			(font
+				(size 1.27 1.27)
+			)
+			(justify right)
+		)
+		(property "Intersheetrefs" "${INTERSHEET_REFS}"
+			(at 315.7848 176.53 0)
+			(effects
+				(font
+					(size 1.27 1.27)
+				)
+				(justify right)
+				(hide yes)
+			)
+		)
+	)
 	(global_label "BAT_VOLT"
 		(shape input)
@@
 			)
 		)
-		(property "Value" "10k"
+		(property "Value" "2.7k"
 			(at 276.098 137.16 0)
 			(effects
@@
 	)
 	(symbol
+		(lib_id "Connector_Generic:Conn_01x04")
+		(at 331.47 176.53 0)
+		(unit 1)
+		(exclude_from_sim no)
+		(in_bom no)
+		(on_board yes)
+		(dnp yes)
+		(fields_autoplaced yes)
+		(property "Reference" "J2"
+			(at 334.01 176.5299 0)
+			(effects
+				(font
+					(size 1.27 1.27)
+				)
+				(justify left)
+			)
+		)
+		(property "Value" "USB POGO"
+			(at 334.01 179.0699 0)
+			(effects
+				(font
+					(size 1.27 1.27)
+				)
+				(justify left)
+			)
+		)
+		(property "Footprint" "Connector_PinHeader_2.54mm:PinHeader_1x04_P2.54mm_Vertical"
+			(at 331.47 176.53 0)
+			(effects
+				(font
+					(size 1.27 1.27)
+				)
+				(hide yes)
+			)
+		)
+		(property "Datasheet" "~"
+			(at 331.47 176.53 0)
+			(effects
+				(font
+					(size 1.27 1.27)
+				)
+				(hide yes)
+			)
+		)
+		(property "Description" "Generic connector, single row, 01x04, script generated (kicad-library-utils/schlib/autogen/connector/)"
+			(at 331.47 176.53 0)
+			(effects
+				(font
+					(size 1.27 1.27)
+				)
+				(hide yes)
+			)
+		)
+		(pin "1"
+		)
+		(pin "2"
+		)
+		(pin "3"
+		)
+		(pin "4"
+		)
+		(instances
+			(project "keyboard"
+				(path "/b7d3f851-0752-4e3e-bd6d-3affc9fb3bff/8a7a807d-1631-4def-b093-3afd7da15c20"
+					(reference "J2")
+					(unit 1)
+				)
+			)
+		)
+	)
+	(symbol
 		(lib_id "Device:R_Small")
 		(at 332.74 125.73 270)
@@
 		(unit 1)
 		(exclude_from_sim no)
-		(in_bom yes)
+		(in_bom no)
 		(on_board yes)
-		(dnp no)
+		(dnp yes)
 		(fields_autoplaced yes)
 		(property "Reference" "J3"
@@
 	(symbol
 		(lib_id "power:GND")
+		(at 326.39 181.61 0)
+		(unit 1)
+		(exclude_from_sim no)
+		(in_bom yes)
+		(on_board yes)
+		(dnp no)
+		(fields_autoplaced yes)
+		(property "Reference" "#PWR020"
+			(at 326.39 187.96 0)
+			(effects
+				(font
+					(size 1.27 1.27)
+				)
+				(hide yes)
+			)
+		)
+		(property "Value" "GND"
+			(at 326.39 186.69 0)
+			(effects
+				(font
+					(size 1.27 1.27)
+				)
+			)
+		)
+		(property "Footprint" ""
+			(at 326.39 181.61 0)
+			(effects
+				(font
+					(size 1.27 1.27)
+				)
+				(hide yes)
+			)
+		)
+		(property "Datasheet" ""
+			(at 326.39 181.61 0)
+			(effects
+				(font
+					(size 1.27 1.27)
+				)
+				(hide yes)
+			)
+		)
+		(property "Description" "Power symbol creates a global label with name \"GND\" , ground"
+			(at 326.39 181.61 0)
+			(effects
+				(font
+					(size 1.27 1.27)
+				)
+				(hide yes)
+			)
+		)
+		(pin "1"
+		)
+		(instances
+			(project "keyboard"
+				(path "/b7d3f851-0752-4e3e-bd6d-3affc9fb3bff/8a7a807d-1631-4def-b093-3afd7da15c20"
+					(reference "#PWR020")
+					(unit 1)
+				)
+			)
+		)
+	)
+	(symbol
+		(lib_id "power:GND")
 		(at 161.29 54.61 0)
 		(unit 1)
@@
 		(pin "A12"
 		)
+		(pin "B6"
+		)
+		(pin "B7"
+		)
 		(instances
 			(project ""
@@
 		(unit 1)
 		(exclude_from_sim no)
-		(in_bom yes)
+		(in_bom no)
 		(on_board yes)
-		(dnp no)
+		(dnp yes)
 		(fields_autoplaced yes)
 		(property "Reference" "J1"
@@
 			)
 		)
-		(property "Value" "Pico-EZmate"
+		(property "Value" "BATT"
 			(at 281.94 113.0299 0)
 			(effects
@@
 			)
 		)
-		(property "Footprint" "Connector_Molex:Molex_Pico-EZmate_78171-0002_1x02-1MP_P1.20mm_Vertical"
+		(property "Footprint" "Connector_PinHeader_2.54mm:PinHeader_1x02_P2.54mm_Vertical"
 			(at 279.4 110.49 0)
 			(effects

Commit message: TAPEOUT: keyboard + protector, display + halls switch eval
Parts:
- removed F1: 500mA, Fuse:Fuse_0402_1005Metric, symbol Device:Polyfuse_Small
- removed J1: BATT, Connector_PinHeader_2.54mm:PinHeader_1x02_P2.54mm_Vertical, symbol Connector_Generic:Conn_01x02
- added TP5: VBAT, symbol Connector:TestPoint
- added TP6: BAT GND, symbol Connector:TestPoint
- C1, C13, C19, C4: Digikey 1276-1784-1-ND -> (none); JLC Part C23733 -> (none); LCSC (none) -> C23733; LCSC Part C368809 -> (none)
- C10: Digikey 1276-1658-1-ND -> (none); JLC Part C1552 -> (none); LCSC (none) -> C1552; LCSC Part C170150 -> (none)
- C11, C12: Digikey 1276-1595-1-ND -> (none); JLC Part C1550 -> (none); LCSC (none) -> C1550; LCSC Part C371977 -> (none)
- C14, C15, C2, C20: Digikey 1276-1067-1-ND -> (none); JLC Part C52923 -> (none); LCSC (none) -> C52923; LCSC Part C52923 -> (none)
- C16, C17, C18, C7: Digikey 1276-6720-1-ND -> (none); JLC Part C1525 -> (none); LCSC (none) -> C307331; LCSC Part C1525 -> (none)
- C21, C22, C8, C9: JLC Part C1548 -> (none); LCSC (none) -> C1548; LCSC Part C307341 -> (none)
- C23: Digikey 1276-1499-1-ND -> (none); JLC Part C15195 -> (none); LCSC (none) -> C15195; LCSC Part C15195 -> (none)
- C3: Digikey 1276-1077-1-ND -> (none); JLC Part C26403 -> (none); LCSC (none) -> C272875; LCSC Part C307434 -> (none)
- C5: Digikey 1276-1032-1-ND -> (none); JLC Part C1523 -> (none); LCSC (none) -> C1523; LCSC Part C14442 -> (none)
- C6: Digikey 478-1082-1-ND -> (none); JLC Part C1546 -> (none); LCSC (none) -> C1546; LCSC Part C26409 -> (none)
- D1: JLC Part C72038 -> (none); LCSC (none) -> C72038; LCSC Part C160478 -> (none)
- D2: JLC Part C50704 -> (none); LCSC (none) -> C8598; LCSC Part C50704 -> (none)
- D3: JLC Part C72041 -> (none); LCSC (none) -> C2290; LCSC Part C146215 -> (none)
- L1: JLC Part C27143 -> (none); LCSC (none) -> C27143; LCSC Part C76763 -> (none)
- L2, L3: JLC Part C1035 -> (none); LCSC (none) -> C285968; LCSC Part C76732 -> (none)
- L4: JLC Part C14033 -> (none); LCSC (none) -> C14033; LCSC Part C76775 -> (none)
- P1: LCSC (none) -> C165948
- R1: JLC Part C17168 -> (none); LCSC (none) -> C17168; LCSC Part C106231 -> (none)
- R10: JLC Part C26082 -> (none); LCSC (none) -> C26082; LCSC Part C138067 -> (none)
- R11: LCSC (none) -> C26083
- R2, R4: JLC Part C25744 -> (none); LCSC (none) -> C25744; LCSC Part C60490 -> (none)
- R3: footprint Resistor_SMD:R_0402_1005Metric -> Resistor_SMD:R_0603_1608Metric; JLC Part C25744 -> (none); LCSC (none) -> C13167; LCSC Part C60490 -> (none)
- R5: JLC Part C25867 -> (none); LCSC (none) -> C25867; LCSC Part C114759 -> (none)
- R6, R7: JLC Part C25905 -> (none); LCSC (none) -> C25905; LCSC Part C105872 -> (none)
- R8, R9: footprint Resistor_SMD:R_0402_1005Metric -> Resistor_SMD:R_0603_1608Metric; JLC Part C138014 -> (none); LCSC (none) -> C22976; LCSC Part C138014 -> (none)
- SW1: LCSC (none) -> C318884
- U1: LCSC (none) -> C202311
- U2: Digikey 1490-1071-1-ND -> (none); JLC Part C1851953 -> (none); LCSC (none) -> C190794; LCSC Part C1851953 -> (none)
- U3: JLC Part C327480 -> (none); LCSC (none) -> C327480; LCSC Part C327480 -> (none)
- Y1: Digikey 728-1075-1-ND -> (none); JLC Part C93231 -> (none); LCSC (none) -> C99009; LCSC Part C97607 -> (none)
- Y2: Digikey 490-XRCGB32M000F1S1DR0CT-ND‎ -> (none); JLC Part C255896 -> (none); LCSC (none) -> C2965584; LCSC Part C2965584 -> (none)
Connections:
- net GND: now also TP6.1
- net VBAT: now also TP5.1
- net at D2.1 (K): now also C15.1, U1.6 (VIN)

Commit message: keyboard TAPEOUT and plate file finalization
Parts:
- TP5, TP6: footprint (none) -> TestPoint:TestPoint_Pad_2.5x2.5mm
Changed lines of the file:
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@@
 			)
 		)
-		(property "Footprint" ""
+		(property "Footprint" "TestPoint:TestPoint_Pad_2.5x2.5mm"
 			(at 274.32 118.11 0)
 			(effects
@@
 			)
 		)
-		(property "Footprint" ""
+		(property "Footprint" "TestPoint:TestPoint_Pad_2.5x2.5mm"
 			(at 279.4 110.49 0)
 			(effects
