File: keyboard/protector/protector.kicad_sch (KiCad schematic)
At the start: 10 parts, among them Q1 CSD16301Q2, Q2 CSD16301Q2, U1 BQ29707

Commit message: TAPEOUT: keyboard + protector, display + halls switch eval
Parts:
- C1: LCSC (none) -> C307331
- Q1, Q2: LCSC (none) -> C140340
- R1: LCSC (none) -> C25104
- R2: LCSC (none) -> C25879
- U1: LCSC (none) -> C2864878
Changed lines of the file:
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@@
+			)
+		)
+		(property "LCSC" "C140340"
+			(at 113.03 92.71 0)
+			(effects
+				(font
+					(size 1.27 1.27)
+				)
+				(hide yes)
 			)
 		)
@@
 			)
 		)
+		(property "LCSC" "C25104"
+			(at 162.56 69.8499 0)
+			(effects
+				(font
+					(size 1.27 1.27)
+				)
+				(hide yes)
+			)
+		)
 		(pin "1"
 		)
@@
 		(property "Description" "Resistor, small symbol"
 			(at 99.06 83.82 0)
+			(effects
+				(font
+					(size 1.27 1.27)
+				)
+				(hide yes)
+			)
+		)
+		(property "LCSC" "C25879"
+			(at 101.6 82.5499 0)
 			(effects
 				(font
@@
 			)
 		)
+		(property "LCSC" "C307331"
+			(at 162.56 76.2062 0)
+			(effects
+				(font
+					(size 1.27 1.27)
+				)
+				(hide yes)
+			)
+		)
 		(pin "2"
 		)
@@
 			)
 		)
+		(property "LCSC" "C140340"
+			(at 128.27 92.71 0)
+			(effects
+				(font
+					(size 1.27 1.27)
+				)
+				(hide yes)
+			)
+		)
 		(pin "1"
 		)
@@
 			(effects
 				(font
+					(size 1.27 1.27)
+				)
+				(hide yes)
+			)
+		)
+		(property "LCSC" "C2864878"
+			(at 142.24 67.31 0)
+			(effects
+				(font
