File: keyboard/protector/protector.kicad_pcb (KiCad board)
At the start: 2 copper layers, 32.2 x 4.4 mm, 10 parts, among them Q1 CSD16301Q2, Q2 CSD16301Q2, U1 BQ29707

Commit message: TAPEOUT: keyboard + protector, display + halls switch eval
Parts:
- TP1, TP2, TP3, TP4: moved to B.Cu
- turned TP1 to 180 degrees
- turned TP2 to 180 degrees
- turned TP3 to 180 degrees
- turned TP4 to 180 degrees
Routing:
- net Net-(Q2-G): track 1.77 -> 2.35 mm, vias 0 -> 2
Other:
- board text added: "anyon_e"
- board text added: "v1"
- board text removed: "_V1.0"

Commit message: keyboard TAPEOUT and plate file finalization
Routing:
- net /OUT_N: vias 20 -> 28
- net /CELL_P: vias 30 -> 38
Other:
- board size 32.2 x 4.4 mm -> 32.2 x 15.4 mm
Changed lines of the file:
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@@
 		)
 	)
-	(gr_rect
-		(start 117.5 94.05)
+	(gr_line
+		(start 149.7 89.41)
 		(end 149.7 98.45)
 		(stroke
@@
 			(type default)
 		)
-		(fill none)
+		(layer "Edge.Cuts")
+	)
+	(gr_line
+		(start 123.98 98.45)
+		(end 123.98 104.77)
+		(stroke
+			(width 0.05)
+			(type default)
+		)
+		(layer "Edge.Cuts")
+	)
+	(gr_line
+		(start 149.7 98.45)
+		(end 123.98 98.45)
+		(stroke
+			(width 0.05)
+			(type default)
+		)
+		(layer "Edge.Cuts")
+	)
+	(gr_line
+		(start 123.98 104.77)
+		(end 117.5 104.77)
+		(stroke
+			(width 0.05)
+			(type default)
+		)
+		(layer "Edge.Cuts")
+	)
+	(gr_line
+		(start 117.5 94.05)
+		(end 143.13 94.05)
+		(stroke
+			(width 0.05)
+			(type default)
+		)
+		(layer "Edge.Cuts")
+	)
+	(gr_line
+		(start 117.5 104.77)
+		(end 117.5 94.05)
+		(stroke
+			(width 0.05)
+			(type default)
+		)
+		(layer "Edge.Cuts")
+	)
+	(gr_line
+		(start 143.13 94.05)
+		(end 143.13 89.41)
+		(stroke
+			(width 0.05)
+			(type default)
+		)
+		(layer "Edge.Cuts")
+	)
+	(gr_line
+		(start 143.13 89.41)
+		(end 149.7 89.41)
+		(stroke
+			(width 0.05)
+			(type default)
+		)
 		(layer "Edge.Cuts")
 	)
@@
 	)
 	(via
+		(at 119.61 98.6)
+		(size 0.6)
+		(drill 0.3)
+		(layers "F.Cu" "B.Cu")
+		(net 4)
+	)
+	(via
 		(at 118.25 96.25)
 		(size 0.6)
@@
 	)
 	(via
+		(at 118.86 98.6)
+		(size 0.6)
+		(drill 0.3)
+		(layers "F.Cu" "B.Cu")
+		(net 4)
+	)
+	(via
+		(at 122.61 98.61)
+		(size 0.6)
+		(drill 0.3)
+		(layers "F.Cu" "B.Cu")
+		(net 4)
+	)
+	(via
 		(at 118.25 97)
 		(size 0.6)
@@
 	)
 	(via
+		(at 120.36 98.6)
+		(size 0.6)
+		(drill 0.3)
+		(layers "F.Cu" "B.Cu")
+		(net 4)
+	)
+	(via
 		(at 118.25 95.5)
 		(size 0.6)
@@
 	(via
 		(at 119 95.5)
+		(size 0.6)
+		(drill 0.3)
+		(layers "F.Cu" "B.Cu")
+		(net 4)
+	)
+	(via
+		(at 118.11 98.6)
+		(size 0.6)
+		(drill 0.3)
+		(layers "F.Cu" "B.Cu")
+		(net 4)
+	)
+	(via
+		(at 121.86 98.61)
+		(size 0.6)
+		(drill 0.3)
+		(layers "F.Cu" "B.Cu")
+		(net 4)
+	)
+	(via
+		(at 121.11 98.6)
+		(size 0.6)
+		(drill 0.3)
+		(layers "F.Cu" "B.Cu")
+		(net 4)
+	)
+	(via
+		(at 123.36 98.61)
 		(size 0.6)
 		(drill 0.3)
@@
 	)
 	(via
+		(at 146.86 93.6)
+		(size 0.6)
+		(drill 0.3)
+		(layers "F.Cu" "B.Cu")
+		(net 6)
+	)
+	(via
+		(at 148.36 93.61)
+		(size 0.6)
+		(drill 0.3)
+		(layers "F.Cu" "B.Cu")
+		(net 6)
+	)
+	(via
 		(at 148.25 96.25)
 		(size 0.6)
@@
 	)
 	(via
+		(at 147.61 93.61)
+		(size 0.6)
+		(drill 0.3)
+		(layers "F.Cu" "B.Cu")
+		(net 6)
+	)
+	(via
 		(at 149 96.25)
 		(size 0.6)
@@
 	)
 	(via
+		(at 149.11 93.61)
+		(size 0.6)
+		(drill 0.3)
+		(layers "F.Cu" "B.Cu")
+		(net 6)
+	)
+	(via
 		(at 142.75 96.25)
 		(size 0.6)
@@
 	)
 	(via
+		(at 143.81 93.61)
+		(size 0.6)
+		(drill 0.3)
+		(layers "F.Cu" "B.Cu")
+		(net 6)
+	)
+	(via
 		(at 146 97)
 		(size 0.6)
@@
 	)
 	(via
+		(at 146.11 93.6)
+		(size 0.6)
+		(drill 0.3)
+		(layers "F.Cu" "B.Cu")
+		(net 6)
+	)
+	(via
 		(at 139.75 97)
 		(size 0.6)
@@
 	)
 	(via
+		(at 144.56 93.61)
+		(size 0.6)
+		(drill 0.3)
+		(layers "F.Cu" "B.Cu")
+		(net 6)
+	)
+	(via
 		(at 149 95.5)
 		(size 0.6)
@@
 	(via
 		(at 139.75 95.5)
+		(size 0.6)
+		(drill 0.3)
+		(layers "F.Cu" "B.Cu")
+		(net 6)
+	)
+	(via
+		(at 145.36 93.6)
 		(size 0.6)
 		(drill 0.3)
@@
 		(polygon
 			(pts
-				(xy 136.1 97.1) (xy 136.1 98.5) (xy 149.8 98.5) (xy 149.8 94) (xy 139.1 94) (xy 139.1 97.1)
+				(xy 136.1 97.1) (xy 136.1 98.5) (xy 149.8 98.5) (xy 149.82 92.97) (xy 139.12 92.97) (xy 139.1 97.1)
 			)
 		)
@@
 		(polygon
 			(pts
-				(xy 117.4 94) (xy 117.4 98.5) (xy 132 98.5) (xy 132 95.9) (xy 130 95.9) (xy 130 97.2) (xy 123.7 97.2)
+				(xy 117.4 94) (xy 117.4 99.65) (xy 132 99.65) (xy 132 95.9) (xy 130 95.9) (xy 130 97.2) (xy 123.7 97.2)
 				(xy 123.7 94)
 			)
@@
 		(polygon
 			(pts
-				(xy 139.1 94) (xy 139 98.5) (xy 149.8 98.5) (xy 149.8 94)
-			)
-		)
+				(xy 139.12 92.98) (xy 139 98.5) (xy 149.8 98.5) (xy 149.82 92.98)
+			)
+		)
