File: motherboard/display_eval/display_eval.kicad_sch (KiCad schematic)
At the start: 30 parts, among them J1 20455-040E-76 OLED IPEX, J2 OLED PWR, J3 0472720024, J4 HDMI mux'ed to DP1.4a, J5 DEBUG, J6 Hall Sensor, J7 Hall Sensor, J8 Hall Sensor, U1 Hall Switch Testing, U2 Hall Switch Testing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

Commit message: added two more display eval test boards
Parts:
- removed C1, C3, C5: 0.1uF, Capacitor_SMD:C_0402_1005Metric, symbol Device:C_Small
- removed C2, C4, C6: 1uF, Capacitor_SMD:C_0402_1005Metric, symbol Device:C_Small
- removed H1, H2: M3, MountingHole:MountingHole_3.2mm_M3_Pad_Via, symbol Mechanical:MountingHole
- removed J6, J7, J8: Hall Sensor, Connector_PinHeader_2.54mm:PinHeader_1x03_P2.54mm_Vertical, symbol Connector_Generic:Conn_01x03
- removed R5, R6, R7: 5.1k, Resistor_SMD:R_0603_1608Metric, symbol Device:R_Small
- removed TP11: ~, TestPoint:TestPoint_Pad_D1.0mm, symbol Connector:TestPoint_Small
- removed U1, U2, U3: Hall Switch Testing, Package_TO_SOT_SMD:SOT-23, symbol Sensor_Magnetic:SM351LT
- R1: now fitted; now in the parts list
