File: power/power.kicad_sch (KiCad schematic)
At the start: 0 parts

Commit message: major power work
Parts:
- added C12, C13, C14: 10uF, symbol Device:C_Small
- added C15, C16: 22uF, symbol Device:C_Small
- added C17, C20, C21: 0.1uF, symbol Device:C_Small
- added C18, C19: 330pF, symbol Device:C_Small
- added J6: USB C, symbol Connector:USB_C_Receptacle_USB2.0_14P
- added R10, R5, R6, R7, R8, R9: 10k, symbol Device:R_Small
- added R25: 1M, symbol Device:R_Small
- added R3, R4: 2.2k, symbol Device:R_Small
- added SW1: USB SELECT, symbol Switch:SW_SPST
- added U1: TPS25750DRJKR, TPS25750DRJKR:IC_TPS25750DRJKR, symbol TPS25750D:TPS25750DRJKR
- added U3: CAT24C256, Package_SO:SOIC-8_3.9x4.9mm_P1.27mm, symbol Memory_EEPROM:CAT24C256
- added U4: TS3USB30ERSWR, Package_DFN_QFN:UQFN-10_1.4x1.8mm_P0.4mm, symbol Interface_USB:TS3USB30ERSWR
Connections:
- new net: R9.2, U4.8 (~{OE})
- new net: J6.S1 (SHIELD), R25.1
- new net: U1.15 (DRAIN), U1.30 (DRAIN), U1.40 (EXP_DRAIN)
- new net: R5.2, U3.1 (A0)
- new net: R8.2, U3.7 (WP)
- new net: R6.2, U3.2 (A1)
- new net: R7.2, U3.3 (A2)
- new net CC1: C18.1, J6.A5 (CC1), U1.28 (CC1)
- new net CC2: C19.1, J6.B5 (CC2), U1.29 (CC2)
- new net GND: C12.2, C13.2, C14.2, C15.2, C16.2, C17.2, C18.2, C19.2, C20.2, C21.2, J6.A1 (GND), J6.A12 (GND), J6.B1 (GND), J6.B12 (GND), R10.1, R25.2, R5.1, R6.1, R7.1, R8.1, R9.1, U1.10 (~{I2CS_IRQ}), U1.11 (GND), U1.12 (GND), U1.14 (GND), U1.18 (~{I2CM_IRQ}), U1.31 (GND), U1.39 (EXP_GND), U3.4 (GND), U4.4 (GND)
- new net I2CM_SCL: R4.2, U1.17 (I2CM_SCL), U3.6 (SCL)
- new net I2CM_SDA: R3.2, U1.16 (I2CM_SDA), U3.5 (SDA)
- new net I2CS_SCL: U1.9 (I2CS_SCL)
- new net I2CS_SDA: U1.8 (I2CS_SDA)
- new net LDO_1V5: C12.1, U1.2 (ADCIN1), U1.3 (ADCIN2), U1.4 (LDO_1V5)
- new net LDO_3V3: C13.1, C20.1, C21.1, R3.1, R4.1, SW1.2 (B), U1.1 (LDO_3V3), U3.8 (VCC), U4.9 (VCC)
- new net MAIN_USB_N: U4.6 (D2-)
- new net MAIN_USB_P: U4.2 (D2+)
- new net OUT_USB_N: J6.A7 (D-), J6.B7 (D-), U4.5 (D-)
- new net OUT_USB_P: J6.A6 (D+), J6.B6 (D+), U4.3 (D+)
- new net PP5V: U1.34_35 (PP5V)
- new net PPHV: C15.1, C16.1, C17.1, U1.20_22 (PPHV)
- new net S: R10.2, SW1.1 (A), U4.10 (S)
- new net TPS_USB_N: U4.7 (D1-)
- new net TPS_USB_P: U4.1 (D1+)
- new net USB_N: U1.27 (GPIO5(USB_N))
- new net USB_P: U1.26 (GPIO4(USB_P))
- new net VBUS: J6.A4 (VBUS), J6.A9 (VBUS), J6.B4 (VBUS), J6.B9 (VBUS), U1.23_25 (VBUS_IN), U1.32_33 (VBUS)
- new net VIN_3V3: C14.1, U1.38 (VIN_3V3)
- no-connect marks 0 -> 7
Other:
- added sheet BQ25798 (BQ25798.kicad_sch)
- added sheet LTC2943 (LTC2943.kicad_sch)
- added sheet TPS54531 (TPS54531.kicad_sch)
- added sheet TPS55289 (TPS55289.kicad_sch)

Commit message: powertrain schematic init
Parts:
- removed C12, C13, C14: 10uF, symbol Device:C_Small
- removed C15, C16: 22uF, symbol Device:C_Small
- removed C17, C20, C21: 0.1uF, symbol Device:C_Small
- removed C18, C19: 330pF, symbol Device:C_Small
- removed J6: USB C, symbol Connector:USB_C_Receptacle_USB2.0_14P
- removed R10, R5, R6, R7, R8, R9: 10k, symbol Device:R_Small
- removed R25: 1M, symbol Device:R_Small
- removed R4: 2.2k, symbol Device:R_Small
- removed SW1: USB SELECT, symbol Switch:SW_SPST
- removed U1: TPS25750DRJKR, TPS25750DRJKR:IC_TPS25750DRJKR, symbol TPS25750D:TPS25750DRJKR
- removed U3: CAT24C256, Package_SO:SOIC-8_3.9x4.9mm_P1.27mm, symbol Memory_EEPROM:CAT24C256
- removed U4: TS3USB30ERSWR, Package_DFN_QFN:UQFN-10_1.4x1.8mm_P0.4mm, symbol Interface_USB:TS3USB30ERSWR
- added C1: 1uF, symbol Device:C_Small
- added J1: USB-C Power + USB2.0, symbol Connector:USB_C_Receptacle_USB2.0_16P
- added R1: 1M, Resistor_SMD:R_0402_1005Metric, symbol Device:R_Small
- added R2: 10R, symbol Device:R_Small
- added U1: HUSB238, husb238:DFN-10_L3.0-W3.0-P0.50-BL-EP2.5, symbol HUSB238:HUSB238_002DD
- added U2: LTC2943, DFN-8_DD_LIT, symbol LTC2943:LTC2943IDD-PBF
- added U3: BQ7791501PWR, BQ7791501PWR:SOP65P640X120-24N, symbol BQ77915:BQ7791501PWR
- added U4: BQ25713RSNR, RSN0032B, symbol BQ25713:BQ25713RSNR
- added U5: RP2040, Package_DFN_QFN:QFN-56-1EP_7x7mm_P0.4mm_EP3.2x3.2mm, symbol MCU_RaspberryPi:RP2040
- R3: value 2.2k -> 5.1k
Connections:
- net CC1: now also J1.A5 (CC1), U1.4 (CC1)
- net CC2: now also J1.B5 (CC2), U1.5 (CC2)
- net GND: now also C1.2, J1.A1 (GND), J1.A12 (GND), J1.B1 (GND), J1.B12 (GND), R1.2, U1.11 (GND), U2.2 (GND), U2.3 (GND), U2.7 (GND), U2.9 (EPAD)
- net I2CM_SDA: no longer names the net of R3.2
- net LDO_3V3: no longer names the net of R3.1
- new net: J1.A4 (VBUS), J1.A9 (VBUS), J1.B4 (VBUS), J1.B9 (VBUS), R2.1
- new net: C1.1, R2.2, U1.1 (VIN)
- new net: U5.1 (IOVDD), U5.10 (IOVDD), U5.22 (IOVDD), U5.33 (IOVDD), U5.42 (IOVDD), U5.49 (IOVDD)
- new net: U5.23 (DVDD), U5.50 (DVDD)
- new net: J1.S1 (SHIELD), R1.1
- new net D+: J1.A6 (D+), J1.B6 (D+), U1.2 (D+)
- new net D-: J1.A7 (D-), J1.B7 (D-), U1.3 (D-)
- new net SCL: U1.7 (SCL)
- new net SDA: U1.6 (SDA)
- no-connect marks 7 -> 2
Other:
- removed sheet BQ25798
- removed sheet LTC2943
- removed sheet TPS54531
- removed sheet TPS55289

Commit message: mainboard v0.3 + power WIP
Parts:
- removed U5: RP2040, Package_DFN_QFN:QFN-56-1EP_7x7mm_P0.4mm_EP3.2x3.2mm, symbol MCU_RaspberryPi:RP2040
- added BT1: Cell 1, Connector_PinHeader_2.54mm:PinHeader_1x02_P2.54mm_Vertical, symbol Device:Battery_Cell
- added BT2: Cell 2, Connector_PinHeader_2.54mm:PinHeader_1x02_P2.54mm_Vertical, symbol Device:Battery_Cell
- added BT3: Cell 3, Connector_PinHeader_2.54mm:PinHeader_1x02_P2.54mm_Vertical, symbol Device:Battery_Cell
- added BT4: Cell 4, Connector_PinHeader_2.54mm:PinHeader_1x02_P2.54mm_Vertical, symbol Device:Battery_Cell
- added C10, C26: 100nF, Capacitor_SMD:C_0603_1608Metric, symbol Device:C_Small
- added C11, C12, C13, C14, C15, C16, C17, C23, C27, C46, C48, C6, C7: 1uF, Capacitor_SMD:C_0603_1608Metric, symbol Device:C_Small
- added C18, C19, C20, C21, C22, C5, C55: 0.1uF, Capacitor_SMD:C_0603_1608Metric, symbol Device:C_Small
- added C2, C24, C25, C28, C29, C3, C30, C31, C32, C33, C4, C40, C41, C42, C43, C44, C45, C56, C8, C9: 10uF, Capacitor_SMD:C_0603_1608Metric, symbol Device:C_Small
- added C34, C35: 33nF, Capacitor_SMD:C_0603_1608Metric, symbol Device:C_Small
- added C36: 470nF, Capacitor_SMD:C_0603_1608Metric, symbol Device:C_Small
- added C37: 10nF, Capacitor_SMD:C_0603_1608Metric, symbol Device:C_Small
- added C38, C39: 47nF, Capacitor_SMD:C_0603_1608Metric, symbol Device:C_Small
- added C47: 2.2uF, Capacitor_SMD:C_0603_1608Metric, symbol Device:C_Small
- added C49: 680pF, Capacitor_SMD:C_0603_1608Metric, symbol Device:C_Small
- added C50: 15pF, Capacitor_SMD:C_0603_1608Metric, symbol Device:C_Small
- added C51: 33pF, Capacitor_SMD:C_0603_1608Metric, symbol Device:C_Small
- added C52: 1800pF, Capacitor_SMD:C_0603_1608Metric, symbol Device:C_Small
- added C53, C54: 100pF, Capacitor_SMD:C_0603_1608Metric, symbol Device:C_Small
- added C57: 0.1uF, Resistor_SMD:R_0603_1608Metric, symbol Device:C_Small
- added D1: MMSZ5248B, Diode_SMD:D_SOD-123, symbol Device:D_Zener_Small_Filled
- added D2: BAS316, Diode_SMD:D_SOD-323, symbol Diode:BAS316
- added D3: SMBJ26A-13-F, Diode_SMD:D_SMB, symbol Diode:SMAJ26A
- added D4: LED1, LED_SMD:LED_0603_1608Metric, symbol Device:LED_Small
- added D5: LED2, LED_SMD:LED_0603_1608Metric, symbol Device:LED_Small
- added D6: LED3, LED_SMD:LED_0603_1608Metric, symbol Device:LED_Small
- added D7: LED4, LED_SMD:LED_0603_1608Metric, symbol Device:LED_Small
- added D8: LED5, LED_SMD:LED_0603_1608Metric, symbol Device:LED_Small
- added J2: USB, FPC:FPC-SMD_6P-P0.50_XUNPU_FPC-05F-6PH20, symbol Connector_Generic_MountingPin:Conn_01x06_MountingPin
- added L1: MWSA0603S-100MT, Inductor_SMD:L_Sunlord_MWSA0603S, symbol Device:L_Small
- added L2: MWSA0603S-2R2MT, Inductor_SMD:L_Sunlord_MWSA0603S, symbol Device:L_Small
- added Q1: SI7617DN-T1-GE3, Package_SO:Vishay_PowerPAK_1212-8_Single, symbol Transistor_FET:Si7617DN
- added Q2, Q3, Q4, Q5, Q6, Q7, Q8: CSD18534Q5A, Package_TO_SOT_SMD:TDSON-8-1, symbol Transistor_FET:CSD18534Q5A
- added R10, R15, R16, R17, R18: 33R, Resistor_SMD:R_0603_1608Metric, symbol Device:R_Small
- added R11: 7.5k, Resistor_SMD:R_0603_1608Metric, symbol Device:R_Small
- added R12: 24k, Resistor_SMD:R_0603_1608Metric, symbol Device:R_Small
- added R13: 56k, Resistor_SMD:R_0603_1608Metric, symbol Device:R_Small
- added R14, R30, R31, R32, R47, R48, R49, R50, R51, R52, R58, R59, R60, R61, R62, R63: 10k, Resistor_SMD:R_0603_1608Metric, symbol Device:R_Small
- added R19, R57: 1k, Resistor_SMD:R_0603_1608Metric, symbol Device:R_Small
- added R20: 15mΩ SHUNT RLP25FEER015, Resistor_SMD:R_Shunt_Vishay_WSK2512_6332Metric_T1.19mm, symbol Device:R_Shunt
- added R21, R22: 100R, Resistor_SMD:R_0603_1608Metric, symbol Device:R_Small
- added R23, R24: 5.1k, Resistor_SMD:R_0603_1608Metric, symbol Device:R_Small
- added R25: 10M, Resistor_SMD:R_0603_1608Metric, symbol Device:R_Small
- added R26: 3M, Resistor_SMD:R_0603_1608Metric, symbol Device:R_Small
- added R27: 1M, Resistor_SMD:R_0603_1608Metric, symbol Device:R_Small
- added R28, R41: 470k, Resistor_SMD:R_0603_1608Metric, symbol Device:R_Small
- added R29: 100k, Resistor_SMD:R_0603_1608Metric, symbol Device:R_Small
- added R33: 2.2R, Resistor_SMD:R_0603_1608Metric, symbol Device:R_Small
- added R34, R37: 10mΩ SHUNT FMF25FPJR010-LH, Resistor_SMD:R_Shunt_Vishay_WSK2512_6332Metric_T1.19mm, symbol Device:R_Shunt
- added R35, R36: 5.1R, Resistor_SMD:R_0603_1608Metric, symbol Device:R_Small
- added R38, R39, R44: 10R, Resistor_SMD:R_0603_1608Metric, symbol Device:R_Small
- added R4: 49.9k, Resistor_SMD:R_0603_1608Metric, symbol Device:R_Small
- added R40: 130k, Resistor_SMD:R_0603_1608Metric, symbol Device:R_Small
- added R42: 390k, Resistor_SMD:R_0603_1608Metric, symbol Device:R_Small
- added R43: 220k, Resistor_SMD:R_0603_1608Metric, symbol Device:R_Small
- added R45: 2M, Resistor_SMD:R_0603_1608Metric, symbol Device:R_Small
- added R46: 300k, Resistor_SMD:R_0603_1608Metric, symbol Device:R_Small
- added R5, R6: DNP, Resistor_SMD:R_0603_1608Metric, symbol Device:R_Small
- added R53: 40.2k, Resistor_SMD:R_0603_1608Metric, symbol Device:R_Small
- added R54: 200R, Resistor_SMD:R_0603_1608Metric, symbol Device:R_Small
- added R55: 110k, Resistor_SMD:R_0603_1608Metric, symbol Device:R_Small
- added R56: 27k, Resistor_SMD:R_0603_1608Metric, symbol Device:R_Small
- added R7: 0R, Resistor_SMD:R_0603_1608Metric, symbol Device:R_Small
- added R8: 2.2k, Resistor_SMD:R_0603_1608Metric, symbol Device:R_Small
- added R9: 50mΩ SHUNT LR122WF500MT4E, Resistor_SMD:R_Shunt_Vishay_WSK2512_6332Metric_T1.19mm, symbol Device:R_Shunt
- added SW1: RST, Button_Switch_SMD:SW_Push_1P1T_XKB_TS-1187A, symbol Switch:SW_SPST
- added SW2: BOOT, Button_Switch_SMD:SW_Push_1P1T_XKB_TS-1187A, symbol Switch:SW_SPST
- added TH1: 103AT 10k, Connector_PinHeader_2.54mm:PinHeader_1x02_P2.54mm_Vertical, symbol Device:Thermistor_NTC
- added TP1: CCFG, TestPoint:TestPoint_Pad_2.0x2.0mm, symbol Connector:TestPoint
- added TP2: CMPIN, TestPoint:TestPoint_Pad_2.0x2.0mm, symbol Connector:TestPoint
- added TP3: CMPOUT, TestPoint:TestPoint_Pad_2.0x2.0mm, symbol Connector:TestPoint
- added U5: ESP32-S3-MINI-1, RF_Module:ESP32-S2-MINI-1, symbol RF_Module:ESP32-S3-MINI-1
- added U6: TVS2200DRV, Package_SON:WSON-6-1EP_2x2mm_P0.65mm_EP1x1.6mm, symbol Power_Protection:TVS2200DRV
- added U7: TPS560200, Package_TO_SOT_SMD:SOT-23-5, symbol Regulator_Switching:TPS560200
- added U8: CP2102N-Axx-xQFN28, Package_DFN_QFN:QFN-28-1EP_5x5mm_P0.5mm_EP3.35x3.35mm, symbol Interface_USB:CP2102N-Axx-xQFN28
- C1: footprint (none) -> Capacitor_SMD:C_0603_1608Metric
- J1: footprint (none) -> Connector_USB:USB_C_Receptacle_HRO_TYPE-C-31-M-12
- R1: footprint Resistor_SMD:R_0402_1005Metric -> Resistor_SMD:R_0603_1608Metric
- R2, R3: footprint (none) -> Resistor_SMD:R_0603_1608Metric
- U1: footprint husb238:DFN-10_L3.0-W3.0-P0.50-BL-EP2.5 -> HUSB238:DFN-10_L3.0-W3.0-P0.50-BL-EP2.5
- U2: footprint DFN-8_DD_LIT -> LTC2943:DFN-8_DD_LIT
- U3: footprint BQ7791501PWR:SOP65P640X120-24N -> BQ77915:SOP65P640X120-24N
- U4: footprint RSN0032B -> BQ25713:RSN0032B
Connections:
- net GND: now also U4.10 (PSYS), U4.27 (PGND), U4.33 (PAD), C10.2, C2.2, C22.2, C27.2, C28.2, C29.2, C3.2, C30.2, C31.2, C32.2, C33.2, C34.2, C35.2, C36.2, C37.2, C4.2, C40.2, C41.2, C42.2, C43.2, C44.2, C45.2, C46.2, C47.2, C48.2, C49.2, C5.2, C50.2, C51.2, C52.2, C53.1, C54.1, C56.1, C57.1, C6.2, C7.1, C8.2, C9.2, D1.2 (A), D4.1 (K), D5.1 (K), D6.1 (K), D7.1 (K), D8.1 (K), J2.6 (Pin_6), J2.MP (MountPin), Q3.1 (S), Q3.2 (S), Q3.3 (S), Q5.1 (S), Q5.2 (S), Q5.3 (S), Q6.1 (S), Q6.2 (S), Q6.3 (S), R11.1, R14.1, R26.1, R28.1, R41.1, R43.1, R46.1, R5.2, R56.1, R6.2, R7.2, SW1.2 (B), SW2.2 (B), U5.1 (GND), U5.2 (GND), U5.42 (GND), U5.43 (GND), U5.46 (GND), U5.47 (GND), U5.48 (GND), U5.49 (GND), U5.50 (GND), U5.51 (GND), U5.52 (GND), U5.53 (GND), U5.54 (GND), U5.55 (GND), U5.56 (GND), U5.57 (GND), U5.58 (GND), U5.59 (GND), U5.60 (GND), U5.61 (GND), U5.62 (GND), U5.63 (GND), U5.64 (GND), U5.65 (GND), U6.1 (GND), U6.2 (GND), U6.3 (GND), U6.7 (GND), U7.2 (GND), U8.29 (GND), U8.3 (GND)
- net SCL: now also U2.5 (SDA), U4.13 (SCL), R50.1, U5.5 (IO1)
- net SDA: now also U2.4 (SCL), U4.12 (SDA), R51.1, U5.6 (IO2)
- net at J1.A4 (VBUS), J1.A9 (VBUS), J1.B4 (VBUS)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: now also Q1.1 (S), Q1.2 (S), Q1.3 (S), R4.2
- net at U2.1 (SENSE+): now also R9.2
- net ~{ALCC}: now reaches U2.6 (*ALCC)
- net ~{ALCC}: now also R8.1, U5.7 (IO3)
- net at U2.8 (SENSE-): now also R9.3
- net VBUS: now reaches U4.1 (VBUS)
- net VBUS: now also C10.1, C28.1, C29.1, C30.1, C31.1, C32.1, C33.1, C36.1, C8.1, C9.1, Q1.5 (D), R33.2, R34.4, U6.4 (IN), U6.5 (IN), U6.6 (IN)
- net PROCHOT_N: now reaches U4.11 (PROCHOT_N)
- net PROCHOT_N: now also R54.1, U5.8 (IO4)
- net at U4.14 (CMPIN): now also R45.1, R46.2, TP2.1
- net CMPOUT: now reaches U4.15 (CMPOUT)
- net CMPOUT: now also R45.2, R47.1, TP3.1, U5.11 (IO7)
- net COMP1: now reaches U4.16 (COMP1)
- net COMP1: now also C51.1, R53.2
- net COMP2: now reaches U4.17 (COMP2)
- net COMP2: now also C50.1, R52.2
- net CELL_BATPRES: now reaches U4.18 (CELL_BATPRES)
- net CELL_BATPRES: now also R40.1, R41.2
- net SRN: now reaches U4.19 (SRN)
- net SRN: now also U3.11 (SRN), C18.1, C20.1, R21.2, R39.1
- net at U4.2 (ACN): now also R36.1
- net SRP: now reaches U4.20 (SRP)
- net SRP: now also U3.10 (SRP), C18.2, C19.1, R22.2, R38.1
- net BATDRV_N: now reaches U4.21 (BATDRV_N)
- net BATDRV_N: now also Q8.4 (G)
- net VSYS: now reaches U4.22 (VSYS)
- net VSYS: now also C40.1, C41.1, C42.1, C43.1, C44.1, C45.1, Q7.5 (D), Q8.1 (S), Q8.2 (S), Q8.3 (S)
- net SW2: now reaches U4.23 (SW2)
- net SW2: now also C39.1, L2.2, Q6.5 (D), Q7.1 (S), Q7.2 (S), Q7.3 (S)
- net HIDRV2: now reaches U4.24 (HIDRV2)
- net HIDRV2: now also Q7.4 (G)
- net BTST2: now reaches U4.25 (BTST2)
- net BTST2: now also C39.2
- net LODRV2: now reaches U4.26 (LODRV2)
- net LODRV2: now also Q6.4 (G)
- net REGN: now reaches U4.28 (REGN)
- net REGN: now also C47.1, R44.2
- net LODRV1: now reaches U4.29 (LODRV1)
- net LODRV1: now also Q5.4 (G)
- net at U4.3 (ACP): now also R35.1
- net BTST1: now reaches U4.30 (BTST1)
- net BTST1: now also C38.2
- net HIDRV1: now reaches U4.31 (HIDRV1)
- net HIDRV1: now also Q4.4 (G)
- net SW1: now reaches U4.32 (SW1)
- net SW1: now also C38.1, L2.1, Q4.1 (S), Q4.2 (S), Q4.3 (S), Q5.5 (D)
- net CHRG_OK: now reaches U4.4 (CHRG_OK)
- net CHRG_OK: now also R48.1, U5.9 (IO5)
- net EN_OTG: now reaches U4.5 (EN_OTG)
- net EN_OTG: now also R49.1, U5.10 (IO6)
- net ILIM_HIZ: now reaches U4.6 (ILIM_HIZ)
- net ILIM_HIZ: now also R42.1, R43.2
- net VDDA: now reaches U4.7 (VDDA)
- net VDDA: now also C48.1, R40.2, R42.2, R44.1
- net IADPT: now reaches U4.8 (IADPT)
- net IADPT: now also C54.2, R55.2, U5.14 (IO10)
- net IBAT: now reaches U4.9 (IBAT)
- net IBAT: now also C53.2, U5.15 (IO11)
- net at U1.10 (GATE): now also R3.1
- net at U1.8 (VSET): now also R6.1, R7.1
- net at U1.9 (ISET): now also R5.1
- net at U3.1 (VDD): now also U3.20 (CCFG), C11.1, R19.2, TP1.1
- net at U3.12 (DSG): now also R24.1
- net at U3.13 (CHG): now also R23.1
- net LD: now reaches U3.14 (LD)
- net LD: now also R28.2
- net CBI: now reaches U3.16 (CBI)
- net CBI: now also R32.1, U5.13 (IO9)
- net at U3.17 (OCDP): now also R29.1
- net at U3.18 (TS): now also R31.2, TH1.1
- net at U3.19 (VTB): now also R31.1
- net at U3.2 (AVDD): now also C12.1
- net PRES: now reaches U3.22 (PRES)
- net PRES: now also R30.1, U5.12 (IO8)
- net GNDPWR: now reaches U3.23 (CTRC)
- net GNDPWR: now also U3.24 (CTRD), U3.9 (VSS), BT4.2 (-), C11.2, C12.2, C17.2, C19.2, C20.2, C23.2, C24.2, C25.2, C26.2, D3.2 (A2), R18.1, R20.1, R29.2, R32.2, TH1.2
- net VC4: now reaches U3.3 (VC5)
- net VC4: now also U3.4 (VC4), C13.1, D3.1 (A1), R10.2
- net VC3: now reaches U3.5 (VC3)
- net VC3: now also C13.2, C14.1, R15.2
- net VC2: now reaches U3.6 (VC2)
- net VC2: now also C14.2, C15.1, R16.2
- net VC1: now reaches U3.7 (VC1)
- net VC1: now also C15.2, C16.1, C23.1, R17.2
- net VC0: now reaches U3.8 (VC0)
- net VC0: now also C16.2, C17.1, R18.2
- net at R3.2: now also Q1.4 (G), R4.1
- new net: R20.3, R22.1
- new net: BT3.2 (-), BT4.1 (+), R17.1
- new net: BT2.2 (-), BT3.1 (+), R16.1
- new net: C21.1, Q2.1 (S), Q2.2 (S), Q2.3 (S), R20.4, R25.1
- new net: Q2.5 (D), Q3.5 (D)
- new net: D4.2 (A), R59.2
- new net: BT1.2 (-), BT2.1 (+), R15.1
- new net: R13.1, R14.2, U7.1 (EN)
- new net: C37.1, Q4.5 (D), R34.1
- new net: C46.1, C55.1, R37.3, R38.2
- new net: C55.2, R37.2, R39.2
- new net: C49.1, R52.1
- new net: L1.1, U7.3 (PH)
- new net: C35.1, R34.2, R36.2
- new net: C34.1, R34.3, R35.2
- new net: C27.1, R33.1
- new net: C52.1, R53.1
- new net: R55.1, R56.2
- new net: D2.2 (A), R24.2, R27.1
- new net: D8.2 (A), R63.2
- new net: D5.2 (A), R60.2
- new net: Q8.5 (D), R37.4
- new net: R20.2, R21.1
- new net: D6.2 (A), R61.2
- new net: R57.1, U8.9 (~{RST})
- new net: D7.2 (A), R62.2
- new net: C21.2, C22.1
- new net +3.3V: C2.1, C3.1, C56.2, C57.2, C6.1, L1.2, R12.2, R47.2, R48.2, R49.2, R50.2, R51.2, R54.2, R57.2, R58.2, R8.2, U5.3 (3V3), U8.6 (VDD), U8.7 (VREGIN)
- new net CHG: Q2.4 (G), R23.2, R25.2
- new net DSG: D1.1 (K), D2.1 (K), Q3.4 (G), R26.2, R27.2
- new net EN: C7.2, R58.1, SW1.1 (A), U5.45 (EN)
- new net FB: R11.2, R12.1, U7.5 (FB)
- new net IO0: SW2.1 (A), U5.4 (IO0)
- new net LED1: R59.1, U5.16 (IO12)
- new net LED2: R60.1, U5.17 (IO13)
- new net LED3: R61.1, U5.18 (IO14)
- new net LED4: R62.1, U5.19 (IO15)
- new net LED5: R63.1, U5.20 (IO16)
- new net PACK+: BT1.1 (+), C24.1, C25.1, C26.1, R10.1, R19.1, R30.2, R37.1, R9.1
- new net RXD0: U5.40 (RXD0), U8.26 (TXD)
- new net TXD0: U5.39 (TXD0), U8.25 (RXD)
- new net USB_D+: J2.3 (Pin_3), U8.5 (D-)
- new net USB_D-: J2.2 (Pin_2), U8.4 (D+)
- new net USB_VBUS: J2.1 (Pin_1), U8.8 (VBUS)
- new net VDD: C4.1, C5.1, R13.2, R9.4, U7.4 (VIN)
- no-connect marks 2 -> 24
Other:
- note added: "78% w.r.t VDDA"
- note added: "@TODO check shunts"
- note added: "CCFG tie to AVDD for 4 cell"
- note added: "ILIM = 2.9A"
- note added: "hystersis"
- moved on the sheet: R3, U4

Commit message: power v0.1 layout done
Parts:
- L1: value MWSA0603S-100MT -> FTC252012S100MBCA; footprint Inductor_SMD:L_Sunlord_MWSA0603S -> Inductor_SMD:L_1008_2520Metric
Changed lines of the file:
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@@
 	)
 	(symbol
-		(lib_id "RF_Module:ESP32-S3-MINI-1")
-		(at 5.08 54.61 0)
-		(unit 1)
-		(exclude_from_sim no)
-		(in_bom yes)
-		(on_board yes)
-		(dnp no)
-		(fields_autoplaced yes)
-		(property "Reference" "U5"
-			(at 7.2741 21.59 0)
-			(effects
-				(font
-					(size 1.27 1.27)
-				)
-				(justify left)
-			)
-		)
-		(property "Value" "ESP32-S3-MINI-1"
-			(at 7.2741 24.13 0)
-			(effects
-				(font
-					(size 1.27 1.27)
-				)
-				(justify left)
-			)
-		)
-		(property "Footprint" "RF_Module:ESP32-S2-MINI-1"
-			(at 20.32 83.82 0)
-			(effects
-				(font
-					(size 1.27 1.27)
-				)
-				(hide yes)
-			)
-		)
-		(property "Datasheet" "https://www.espressif.com/sites/default/files/documentation/esp32-s3-mini-1_mini-1u_datasheet_en.pdf"
-			(at 5.08 13.97 0)
-			(effects
-				(font
-					(size 1.27 1.27)
-				)
-				(hide yes)
-			)
-		)
-		(property "Description" "RF Module, ESP32-S3 SoC, Wi-Fi 802.11b/g/n, Bluetooth, BLE, 32-bit, 3.3V, SMD, onboard antenna"
-			(at 5.08 11.43 0)
-			(effects
-				(font
-					(size 1.27 1.27)
-				)
-				(hide yes)
-			)
-		)
-		(pin "12"
-		)
-		(pin "13"
-		)
-		(pin "14"
-		)
-		(pin "11"
-		)
-		(pin "10"
-		)
-		(pin "15"
-		)
-		(pin "16"
-		)
-		(pin "17"
-		)
-		(pin "18"
-		)
-		(pin "19"
-		)
-		(pin "2"
-		)
-		(pin "20"
-		)
-		(pin "21"
-		)
-		(pin "22"
-		)
-		(pin "23"
-		)
-		(pin "24"
-		)
-		(pin "25"
-		)
-		(pin "26"
-		)
-		(pin "27"
-		)
-		(pin "28"
-		)
-		(pin "29"
-		)
-		(pin "3"
-		)
-		(pin "30"
-		)
-		(pin "31"
-		)
-		(pin "32"
-		)
-		(pin "33"
-		)
-		(pin "34"
-		)
-		(pin "35"
-		)
-		(pin "36"
-		)
-		(pin "37"
-		)
-		(pin "38"
-		)
-		(pin "39"
-		)
-		(pin "4"
-		)
-		(pin "40"
-		)
-		(pin "41"
-		)
-		(pin "42"
-		)
-		(pin "43"
-		)
-		(pin "44"
-		)
-		(pin "45"
-		)
-		(pin "46"
-		)
-		(pin "47"
-		)
-		(pin "48"
-		)
-		(pin "49"
-		)
-		(pin "5"
-		)
-		(pin "50"
-		)
-		(pin "51"
-		)
-		(pin "52"
-		)
-		(pin "53"
-		)
-		(pin "54"
-		)
-		(pin "55"
-		)
-		(pin "56"
-		)
-		(pin "57"
-		)
-		(pin "58"
-		)
-		(pin "59"
-		)
-		(pin "6"
-		)
-		(pin "60"
-		)
-		(pin "61"
-		)
-		(pin "62"
-		)
-		(pin "63"
-		)
-		(pin "64"
-		)
-		(pin "65"
-		)
-		(pin "7"
-		)
-		(pin "8"
-		)
-		(pin "9"
-		)
-		(pin "1"
-		)
-		(instances
-			(project ""
-				(path "/f6ef1cf7-e202-4cf7-a9a2-de51d726791c"
-					(reference "U5")
-					(unit 1)
-				)
-			)
-		)
-	)
-	(symbol
 		(lib_id "power:GND")
 		(at -58.42 69.85 0)
@@
 			)
 		)
-		(property "Value" "MWSA0603S-100MT"
+		(property "Value" "FTC252012S100MBCA"
 			(at 73.66 128.27 90)
 			(effects
@@
 			)
 		)
-		(property "Footprint" "Inductor_SMD:L_Sunlord_MWSA0603S"
+		(property "Footprint" "Inductor_SMD:L_1008_2520Metric"
 			(at 73.66 130.81 0)
 			(effects
@@
 					(unit 1)
 				)
+			)
+		)
+	)
+	(symbol
+		(lib_id "RF_Module:ESP32-S3-MINI-1")
+		(at 5.08 54.61 0)
+		(unit 1)
+		(exclude_from_sim no)
+		(in_bom yes)
+		(on_board yes)
+		(dnp no)
+		(fields_autoplaced yes)
+		(property "Reference" "U5"
+			(at 7.2741 21.59 0)
+			(effects
+				(font
+					(size 1.27 1.27)
+				)
+				(justify left)
+			)
+		)
+		(property "Value" "ESP32-S3-MINI-1"
+			(at 7.2741 24.13 0)
+			(effects
+				(font
+					(size 1.27 1.27)
+				)
+				(justify left)
+			)
+		)
+		(property "Footprint" "RF_Module:ESP32-S2-MINI-1"
+			(at 20.32 83.82 0)
+			(effects
+				(font
+					(size 1.27 1.27)
+				)
+				(hide yes)
+			)
+		)
+		(property "Datasheet" "https://www.espressif.com/sites/default/files/documentation/esp32-s3-mini-1_mini-1u_datasheet_en.pdf"
+			(at 5.08 13.97 0)
+			(effects
+				(font
+					(size 1.27 1.27)
+				)
+				(hide yes)
+			)
+		)
+		(property "Description" "RF Module, ESP32-S3 SoC, Wi-Fi 802.11b/g/n, Bluetooth, BLE, 32-bit, 3.3V, SMD, onboard antenna"
+			(at 5.08 11.43 0)
+			(effects
+				(font
+					(size 1.27 1.27)
+				)
+				(hide yes)
+			)
+		)
+		(pin "13"
+		)
+		(pin "53"
+		)
+		(pin "54"
+		)
+		(pin "5"
+		)
+		(pin "50"
+		)
+		(pin "51"
+		)
+		(pin "52"
+		)
+		(pin "49"
+		)
+		(pin "36"
+		)
+		(pin "26"
+		)
+		(pin "55"
+		)
+		(pin "56"
+		)
+		(pin "57"
+		)
+		(pin "58"
+		)
+		(pin "59"
+		)
+		(pin "44"
+		)
+		(pin "45"
+		)
+		(pin "46"
+		)
+		(pin "47"
+		)
+		(pin "48"
+		)
+		(pin "22"
+		)
+		(pin "33"
+		)
+		(pin "2"
+		)
+		(pin "19"
+		)
+		(pin "37"
+		)
+		(pin "38"
+		)
+		(pin "39"
+		)
+		(pin "4"
+		)
+		(pin "40"
+		)
+		(pin "41"
+		)
+		(pin "42"
+		)
+		(pin "43"
+		)
+		(pin "34"
+		)
+		(pin "35"
+		)
+		(pin "6"
+		)
+		(pin "60"
+		)
+		(pin "61"
+		)
+		(pin "31"
+		)
+		(pin "32"
+		)
+		(pin "28"
+		)
+		(pin "29"
+		)
+		(pin "3"
+		)
+		(pin "12"
+		)
+		(pin "30"
+		)
+		(pin "16"
+		)
+		(pin "27"
+		)
+		(pin "20"
+		)
+		(pin "7"
+		)
+		(pin "8"
+		)
+		(pin "9"
+		)
+		(pin "62"
+		)
+		(pin "63"
+		)
+		(pin "14"
+		)
+		(pin "23"
+		)
+		(pin "15"
+		)
+		(pin "64"
+		)
+		(pin "65"
+		)
+		(pin "11"
+		)
+		(pin "10"
+		)
+		(pin "17"
+		)
+		(pin "25"
+		)
+		(pin "18"
+		)
+		(pin "24"
+		)
+		(pin "21"
+		)
+		(pin "1"
+		)
+		(instances
+			(project ""
+				(path "/f6ef1cf7-e202-4cf7-a9a2-de51d726791c"
+					(reference "U5")
+					(unit 1)
+				)

Commit message: power sub 50 routes
Parts:
- added J3: BATTERY OUT, Connector_Molex:Molex_PicoBlade_53261-1071_1x10-1MP_P1.25mm_Horizontal, symbol Connector_Generic_MountingPin:Conn_01x10_MountingPin
- added J4: BACKUP, Connector_PinHeader_2.54mm:PinHeader_1x02_P2.54mm_Vertical, symbol Connector_Generic:Conn_01x02
Connections:
- net GND: now also J3.10 (Pin_10), J3.6 (Pin_6), J3.7 (Pin_7), J3.8 (Pin_8), J3.9 (Pin_9), J3.MP (MountPin)
- net SRN: no longer C18.1, C20.1, R21.2, U3.11 (SRN)
- net SRP: no longer C18.2, C19.1, R22.2, U3.10 (SRP)
- net VDD: now also J3.1 (Pin_1), J3.2 (Pin_2), J3.3 (Pin_3), J3.4 (Pin_4), J3.5 (Pin_5)
- net at U5.21 (IO17): now also J4.2 (Pin_2)
- net at U5.22 (IO18): now also J4.1 (Pin_1)
- new net BMS_SRN: C18.1, C20.1, R21.2, U3.11 (SRN)
- new net BMS_SRP: C18.2, C19.1, R22.2, U3.10 (SRP)
- no-connect marks 24 -> 42
