File: power/power.kicad_pcb (KiCad board)
At the start: 4 copper layers, 64 x 45.4 mm, 178 parts, among them J1 USB-C Power + USB2.0, J2 USB, J3 BATTERY OUT, J4 BACKUP, J5 I2C, Q1 SI7617DN-T1-GE3, Q2 CSD18534Q5A, Q3 CSD18534Q5A, Q4 CSD18534Q5A, Q5 CSD18534Q5A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

Commit message: powertrain v2
Parts:
- removed U8: CP2102N-Axx-xQFN28, Package_DFN_QFN:QFN-28-1EP_5x5mm_P0.5mm_EP3.35x3.35mm
- added C58: 100nF, Capacitor_SMD:C_0402_1005Metric, F.Cu at (173.6, 134.4)
- added R72: 12k, Resistor_SMD:R_0402_1005Metric, F.Cu at (170.0, 136.0)
- C4: value 10uF -> 100nF; footprint Capacitor_SMD:C_0603_1608Metric -> Capacitor_SMD:C_0402_1005Metric
- C5: value 0.1uF -> 22uF
- C6: value 1uF -> 22uF
- L1: value FTC252012S100MBCA -> SLO0530H3R3MTT; footprint Inductor_SMD:L_1008_2520Metric -> Inductor_SMD:L_Chilisin_BMRA00050530
- R11: value 7.5k -> 47k; footprint Resistor_SMD:R_0603_1608Metric -> Resistor_SMD:R_0402_1005Metric
- R12: value 24k -> 10k; footprint Resistor_SMD:R_0603_1608Metric -> Resistor_SMD:R_0402_1005Metric
- R13: value 56k -> 49.9k; footprint Resistor_SMD:R_0603_1608Metric -> Resistor_SMD:R_0402_1005Metric
- R14: value 10k -> 510k; footprint Resistor_SMD:R_0603_1608Metric -> Resistor_SMD:R_0402_1005Metric
- R57: value 1k -> 10k; footprint Resistor_SMD:R_0603_1608Metric -> Resistor_SMD:R_0402_1005Metric
- R71: value 1k -> 47k; footprint Resistor_SMD:R_0603_1608Metric -> Resistor_SMD:R_0402_1005Metric
- R9: value 50mΩ SHUNT LR122WF500MT4E -> 10mΩ SHUNT FMF25FPJR010-LH
- U7: value TPS560200 -> TPS564257DRLR; footprint Package_TO_SOT_SMD:SOT-23-5 -> TPS564257:SOT50P160X60-6N
- moved R57 14.3 mm to (170.0, 135.0), turned to 180 degrees
- moved C6 11.8 mm to (173.5, 132.6), turned to 0 degrees
- moved R11 11.6 mm to (173.6, 136.4)
- moved R13 9.70 mm to (172.5, 136.4), turned to -90 degrees
- moved D14 9.62 mm to (173.4, 139.0), turned to 90 degrees
- moved C3 8.09 mm to (163.8, 136.1), turned to -90 degrees
- moved R14 8.05 mm to (171.5, 135.5), turned to -90 degrees
- moved C5 8.03 mm to (173.5, 131.0), turned to 0 degrees
- moved C2 6.47 mm to (165.4, 136.1), turned to -90 degrees
- moved SW1 6.26 mm to (176.9, 126.3), turned to 90 degrees
- moved R71 5.10 mm to (167.2, 137.5)
- moved R12 4.54 mm to (172.5, 134.4), turned to 90 degrees
- moved C4 3.95 mm to (163.9, 133.4), turned to 90 degrees
- moved L1 3.30 mm to (168.3, 131.4), turned to 0 degrees
- moved C7 3.01 mm to (178.3, 131.0), turned to 180 degrees
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Connections:
- C2 pad 1: +3.3V -> VDD
- C3 pad 1: +3.3V -> VDD
- C5 pad 1: VDD -> +3.3V
- L1 pad 1: Net-(U7-PH) -> /3V3_SW
- R11 pad 1: GND -> Net-(D14-A)
- R11 pad 2: /FB -> +3.3V
- R12 pad 1: /FB -> Net-(U7-PG)
- R13 pad 1: Net-(U7-EN) -> Net-(U7-FB)
- R13 pad 2: VDD -> +3.3V
- R14 pad 1: GND -> Net-(U7-FB)
- R14 pad 2: Net-(U7-EN) -> +3.3V
- R57 pad 1: Net-(U8-~{RST}) -> GND
- R57 pad 2: +3.3V -> Net-(U7-FB)
- R71 pad 1: +3.3V -> Net-(U7-EN)
- R71 pad 2: Net-(D14-A) -> VDD
- R9 pad 1: /C4 -> VDD
- R9 pad 4: VDD -> /C4
- U2 pad 4: /SDA -> /SCL
- U2 pad 5: /SCL -> /SDA
- U5 pad 23: unconnected-(U5-IO19-Pad23) -> /USB_D-
- U5 pad 24: unconnected-(U5-IO20-Pad24) -> /USB_D+
- U7 pad 1: Net-(U7-EN) -> VDD
- U7 pad 2: GND -> /3V3_SW
- U7 pad 3: Net-(U7-PH) -> GND
- U7 pad 4: VDD -> Net-(U7-PG)
- U7 pad 5: /FB -> Net-(U7-EN)
Routing:
- net +3.3V: track 87.6 -> 42.2 mm, vias 7 -> 5
- net Net-(U8-~{RST}): track 17.3 -> 0.00 mm, vias 2 -> 0
- net /EN: track 16.6 -> 0.00 mm
- net /IO0: track 28.4 -> 14.7 mm
- net VDD: track 62.1 -> 49.6 mm
- net /USB_D+: track 9.98 -> 0.00 mm, vias 2 -> 0
- net /USB_D-: track 9.82 -> 0.00 mm, vias 2 -> 0
- net /RXD0: track 8.79 -> 0.00 mm
- net /FB: track 7.44 -> 0.00 mm, vias 2 -> 0
- net /USB_VBUS: track 6.69 -> 0.00 mm
- net Net-(U2-SENSE+): track 8.55 -> 2.20 mm
- net GNDPWR: track 36.9 -> 30.9 mm
- net /~{ALCC}: track 72.8 -> 67.0 mm
- net /TXD0: track 5.28 -> 0.00 mm
- net Net-(U7-EN): track 3.55 -> 0.00 mm
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Other:
- board text added: "V2"
